File: untitled.kicad_sch (KiCad schematic)
At the start: 17 parts, among them J1 1147330000, J2 1147330000, J3 1147330000, K1 G2RL-1-H, K2 G2RL-1-H, K3 G2RL-1-H

Commit message: 13-jul-26_6pm
Changed lines of the file:
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@@
 	(wire
 		(pts
-			(xy 134.62 86.36) (xy 134.62 87.63)
+			(xy 138.43 83.82) (xy 138.43 85.09)
 		)
 		(stroke
@@
 			(type default)
 			(color 255 73 219 1)
+		)
+	)
+	(wire
+		(pts
+			(xy 138.43 83.82) (xy 133.35 83.82)
+		)
+		(stroke
+			(width 0)
+			(type default)
 		)
 	)
@@
 		(on_board yes)
 		(dnp no)
-		(property "Reference" "#PWR02"
+		(property "Reference" "#PWR0102"
 			(at 99.06 64.77 0)
 			(effects
@@
 			(project ""
 				(path "/38a2da3c-ed29-422f-ab41-066ccf490e61/2e698a92-0ed9-457a-8ea3-5be56f6a1bd4"
-					(reference "#PWR02")
+					(reference "#PWR0102")
 					(unit 1)
 				)
@@
 	(symbol
 		(lib_id "power:GNDREF")
-		(at 134.62 87.63 0)
+		(at 138.43 85.09 0)
 		(unit 1)
 		(exclude_from_sim no)
@@
 		(dnp no)
 		(fields_autoplaced yes)
-		(property "Reference" "#PWR03"
-			(at 134.62 93.98 0)
+		(property "Reference" "#PWR0103"
+			(at 138.43 91.44 0)
 			(effects
 				(font
@@
 		)
 		(property "Value" "GND"
-			(at 134.62 92.71 0)
+			(at 138.43 90.17 0)
 			(effects
 				(font
@@
 		)
 		(property "Footprint" ""
-			(at 134.62 87.63 0)
+			(at 138.43 85.09 0)
 			(effects
 				(font
@@
 		)
 		(property "Datasheet" ""
-			(at 134.62 87.63 0)
+			(at 138.43 85.09 0)
 			(effects
 				(font
@@
 		)
 		(property "Description" "Power symbol creates a global label with name \"GNDREF\" , reference supply ground"
-			(at 134.62 87.63 0)
+			(at 138.43 85.09 0)
 			(effects
 				(font
@@
 			(project ""
 				(path "/38a2da3c-ed29-422f-ab41-066ccf490e61/2e698a92-0ed9-457a-8ea3-5be56f6a1bd4"
-					(reference "#PWR03")
+					(reference "#PWR0103")
 					(unit 1)
 				)
