File: SALIDA 1.kicad_sch (KiCad schematic)
At the start: 45 parts, among them IC13 VNI4140K, J5 1728840000, J6 1728840000, U7 TSB582IYQ2T, U8 ULN2003, U9 ULN2003

Commit message: 7-may-26 346
se esta trabajando en los reles esquematico y pcb
Parts:
- renumbered C25 to C30, C24 to C31, C23 to C32, C35 to C33, C33 to C35, D14 to D17, D15 to D18, D16 to D19, D17 to D20, R14 to R28, R13 to R29, R15 to R30, R16 to R31, R18 to R32, R19 to R33, R17 to R34, R20 to R35, R21 to R36, R22 to R37, R23 to R38, R24 to R39, R25 to R40, R40 to R41, R41 to R42, R42 to R43, R43 to R44, R36 to R45, R37 to R46, R38 to R47, R39 to R48, R44 to R49, R45 to R50, R46 to R51, R47 to R52, U9 to U10, U7 to U8, U8 to U9
