File: SALIDA 1.kicad_sch (KiCad schematic)
At the start: 205 parts, among them IC13 VNI4140K, IC17 VNI4140K, J5 1728840000, J5.bak 1728840000, J6 1728840000, Q10 MMBT3904, Q11 MMBT3904, Q12 MMBT3904, Q13 DMP3099L, Q14 DMP3099L, Q15 DMP3099L, Q4 MMBT3904, Q5 DMP3099L, Q6 MMBT3904, Q7 DMP3099L, Q8 MMBT3904, Q9 DMP3099L, U10 ULN2003, U12 LM7705, U13 ${SIM.PARAMS}, U14 MCP1799T-5002H/TT, U15 TSB582, U15.bak TSB582, U16 MCP23S17_SS, U17 MCP1799T-5002H/TT, U18 LM7705, U19 74LVC1G17, U20 74LVC1G17, U21 74LVC1G17, U22 74LVC1G17, U23 74LVC1G17, U24 74LVC1G17, U25 ULN2003A, U8.bak TSB582, U9 ULN2003

Commit message: 14-Mayo-26
se agregaron varias sheet de esquematico crecio al 80% la parte de esquematico
Parts:
- renumbered C76 to C36, C77 to C37, C36 to C38, C75 to C39, C37 to C40, C57 to C41, C31 to C42, C32 to C43, C62 to C44, C63 to C45, C64 to C46, C61 to C47, C60 to C48, C59 to C49, C55 to C50, C54 to C51, C49 to C52, C73 to C53, C74 to C54, C52 to C55, C53 to C56, C48 to C57, C72 to C58, C71 to C59, C70 to C60, C69 to C61, C50 to C62, C51 to C63, C47 to C64, C46 to C65, C68 to C66, C66 to C67, C67 to C68, C80 to C69, C30 to C70, C65 to C71, C45 to C72, C81 to C73, C58 to C74, C56 to C75, D17 to D18, D18 to D19, D19 to D20, D20 to D21, D23 to D22, D24 to D23, D25 to D24, D26 to D25, D21 to D26, D22 to D31, IC17 to IC14, J5.bak to J5.bak1, J5 to J7, J6 to J8, L9 to L7, L10 to L9, Q15 to Q10, Q9 to Q11, Q5 to Q12, Q7 to Q13, Q10 to Q2, Q11 to Q3, Q12 to Q4, Q8 to Q5, Q4 to Q6, Q6 to Q7, Q13 to Q8, Q14 to Q9, R72 to R100, R80 to R101, R137 to R102, R138 to R103, R139 to R104, R140 to R105, R82 to R106, R83 to R107, R84 to R108, R73 to R109, R74 to R110, R75 to R111, R85 to R112, R76 to R113, R90 to R114, R86 to R115, R77 to R116, R87 to R117, R67 to R118, R88 to R119, R70 to R120, R89 to R121, R69 to R122, R35 to R123, R36 to R124, R37 to R125, R38 to R126, R39 to R127, R40 to R128, R41 to R27, R42 to R28, R43 to R29, R44 to R30, R45 to R31, R46 to R32, R47 to R33, R48 to R34, R125 to R35, R126 to R36, R127 to R37, R128 to R38, R49 to R39, R50 to R40, R51 to R41, R52 to R42, R129 to R43, R130 to R44, R131 to R45, R132 to R46, R141 to R47, R68 to R48, R65 to R49, R29 to R50, R30 to R51, R31 to R52, R66 to R53, R28 to R54, R32 to R55, R133 to R56, R134 to R57, R135 to R58, R136 to R59, R34 to R60, R99 to R61, R100 to R62, R101 to R63, R97 to R64, R93 to R65, R95 to R66, R102 to R67, R104 to R68, R103 to R69, R98 to R70, R94 to R71, R96 to R72, R123 to R73, R121 to R74, R118 to R75, R124 to R76, R116 to R77, R122 to R78, R112 to R79, R120 to R80, R119 to R81, R110 to R82, R111 to R83, R109 to R84, R106 to R85, R91 to R86, R92 to R87, R117 to R88, R78 to R89, R113 to R90, R114 to R91, R115 to R92, R108 to R93, R105 to R94, R107 to R95, R79 to R96, R71 to R97, R81 to R98, R33 to R99, TH3 to TH2, U13 to U10, U22 to U11, U23 to U12, U24 to U13, U21 to U14, U20 to U15, U15.bak to U15.bak1, U19 to U16, U15 to U17, U14 to U18, U25 to U19, U12 to U20, U18 to U21, U17 to U22, U9 to U23, U10 to U8, U8.bak to U8.bak1, U16 to U9, V3 to V1, V1 to V2, V2 to V3

Commit message: 15-mayo-26
15 mayo 26
Parts:
- added R234, R235, R236, R237, R238: 0R, Resistor_SMD:R_0603_1608Metric, symbol Device:R_US
- renumbered J7 to J5, J8 to J6
Connections:
- net +3.3v: now also R234.2, R237.2, R238.1; no longer U9.16 (A1)
- net GND: now also R235.1, R236.1, R238.2; no longer U9.15 (A0), U9.17 (A2)
- net BIN:BIN-MONITOR_3V3_J7: no longer names the net of U9.28 (GPA7)
- new net: R235.2, U9.17 (A2)
- new net: R234.1, U9.16 (A1)
- new net: R236.2, R237.1, U9.15 (A0)
- no-connect marks 6 -> 7

Commit message: 22 mayo 26 actualizacion
se actualizo la PCB para la rama laptop Antigua
Parts:
- J5, J7: renamed from J6; footprint CONECTORES GRACIDA:1728840000_17-25 -> CONECTORES GRACIDA:16POS-2LINEAS-3.5PITCH
- J5.bak1: footprint CONECTORES GRACIDA:1728840000 -> CONECTORES GRACIDA:16POS-2LINEAS-3.5PITCH
- J6: renamed from J5; footprint CONECTORES GRACIDA:1728840000 -> CONECTORES GRACIDA:16POS-2LINEAS-3.5PITCH
- renumbered C33 to C37, C34 to C38, C35 to C39, C36 to C40, C37 to C41, C38 to C42, C39 to C43, C40 to C44, C41 to C45, C42 to C46, C43 to C47, C44 to C48, C45 to C49, C46 to C50, C47 to C51, C48 to C52, C49 to C53, C50 to C54, C51 to C55, C52 to C56, C53 to C57, C54 to C58, C55 to C59, C56 to C60, C57 to C61, C58 to C62, C59 to C63, C60 to C64, C61 to C65, C62 to C66, C63 to C67, C64 to C68, C65 to C69, C66 to C70, C67 to C71, C68 to C72, C69 to C73, C70 to C74, C71 to C75, C72 to C76, C73 to C77, C74 to C78, C75 to C79, F1 to F6, IC13 to IC3, IC14 to IC4, L9 to L10, L6 to L7, L7 to L8, L8 to L9, R93 to R100, R94 to R101, R95 to R102, R96 to R103, R97 to R104, R98 to R105, R99 to R106, R100 to R107, R101 to R108, R102 to R109, R103 to R110, R104 to R111, R105 to R112, R106 to R113, R107 to R114, R108 to R115, R109 to R116, R110 to R117, R111 to R118, R112 to R119, R113 to R120, R114 to R121, R115 to R122, R116 to R123, R117 to R124, R118 to R125, R119 to R126, R120 to R127, R121 to R128, R122 to R129, R123 to R130, R124 to R131, R125 to R132, R126 to R133, R127 to R134, R128 to R135, R27 to R29, R28 to R30, R29 to R31, R30 to R32, R31 to R33, R32 to R34, R33 to R35, R34 to R36, R35 to R37, R36 to R38, R37 to R39, R38 to R40, R39 to R41, R40 to R42, R41 to R43, R42 to R44, R43 to R45, R44 to R46, R45 to R47, R46 to R48, R47 to R49, R238 to R50, R237 to R51, R48 to R52, R235 to R53, R234 to R54, R236 to R55, R49 to R56, R50 to R57, R51 to R58, R52 to R59, R53 to R60, R54 to R61, R55 to R62, R56 to R63, R57 to R64, R58 to R65, R59 to R66, R60 to R67, R61 to R68, R62 to R69, R63 to R70, R64 to R71, R65 to R72, R66 to R73, R67 to R74, R68 to R75, R69 to R76, R70 to R77, R71 to R78, R72 to R79, R73 to R80, R74 to R81, R75 to R82, R76 to R83, R77 to R84, R78 to R85, R79 to R86, R80 to R87, R81 to R88, R82 to R89, R83 to R90, R84 to R91, R85 to R92, R86 to R93, R87 to R94, R88 to R95, R89 to R96, R90 to R97, R91 to R98, R92 to R99, U13 to U10, U14 to U11, U15 to U12, U16 to U13, U17 to U14, U18 to U15, U19 to U16, U20 to U17, U21 to U18, U22 to U19, U23 to U20, U8 to U5, U9 to U6, U10 to U7, U11 to U8, U12 to U9

Commit message: 26-05-26
Parts:
- removed C37, C39, C42, C44, C54, C55, C56, C61, C67, C74, C76: 0.1uF, Capacitor_SMD:C_0603_1608Metric_Pad1.08x0.95mm_HandSolder, symbol Device:C_Small
- removed C38: 47uF, Capacitor_Tantalum_SMD:CP_EIA-1608-10_AVX-L_HandSolder, symbol Device:C_Small_US
- removed C59: 10uF, Capacitor_SMD:C_0603_1608Metric, symbol Device:C_Small
- removed C60, C66: 4.7uF, Capacitor_SMD:C_0603_1608Metric, symbol Device:C_Small
- removed C68: 470nF, Capacitor_SMD:C_0603_1608Metric, symbol Device:C_Small
- removed C69: 22uF, symbol Device:C_Small
- removed D18, D19, D20, D21: LED, LED_SMD:LED_0603_1608Metric_Pad1.05x0.95mm_HandSolder, symbol Device:LED
- removed D26: LED, LED_SMD:LED_0402_1005Metric, symbol Device:LED
- removed IC3: VNI4140K, Package_SO:ST_PowerSSO-24_SlugDown_ThermalVias, symbol CI GRACIDA:VNI4140K
- removed J5: 1728840000, CONECTORES GRACIDA:16POS-2LINEAS-3.5PITCH, symbol CONECTORES GRACIDA:1728840000_17-25
- removed J5.bak1: 1728840000, CONECTORES GRACIDA:16POS-2LINEAS-3.5PITCH, symbol CONECTORES GRACIDA:1728840000
- removed L7: 10uH, Inductor_SMD:L_0603_1608Metric_Pad1.05x0.95mm_HandSolder, symbol Device:L_Small
- removed L9: 0603, Inductor_SMD:L_0603_1608Metric_Pad1.05x0.95mm_HandSolder, symbol Device:L_Iron_Small
- removed R103, R104: 0 ohms, Resistor_SMD:R_0603_1608Metric_Pad0.98x0.95mm_HandSolder, symbol Device:R_Small_US
- removed R105, R107, R114, R115, R117, R118: 10k, Resistor_SMD:R_0603_1608Metric_Pad0.98x0.95mm_HandSolder, symbol Device:R_Small_US
- removed R106, R108, R128, R129: 10k, Resistor_SMD:R_0603_1608Metric, symbol Device:R_US
- removed R113, R116: 2.2, Resistor_SMD:R_0603_1608Metric_Pad0.98x0.95mm_HandSolder, symbol Device:R_Small_US
- removed R119, R120, R93: 1k, Resistor_SMD:R_0603_1608Metric_Pad0.98x0.95mm_HandSolder, symbol Device:R_Small_US
- removed R122, R123, R96: 100, Resistor_SMD:R_0603_1608Metric_Pad0.98x0.95mm_HandSolder, symbol Device:R_Small_US
- removed R125: 0 ohms, Resistor_SMD:R_0603_1608Metric, symbol Device:R_US
- removed R126, R127: 10, Resistor_SMD:R_0603_1608Metric, symbol Device:R_US
- removed R130, R131, R132, R133, R134, R135: 4.7k, Resistor_SMD:R_0805_2012Metric_Pad1.20x1.40mm_HandSolder, symbol Device:R_Small_US
- removed R29, R30, R31, R32, R33, R34, R35, R36: 4.7k, Capacitor_SMD:C_0603_1608Metric_Pad1.08x0.95mm_HandSolder, symbol Device:R_Small_US
- removed R41, R42, R43, R44: 10k, Capacitor_SMD:C_0603_1608Metric_Pad1.08x0.95mm_HandSolder, symbol Device:R_Small_US
- removed TH1: B59985C120A70, TERMISTORES GRACIDA:B59985C0120A070, symbol Device:Thermistor_PTC
- removed U15: MCP1799T-5002H/TT, Package_TO_SOT_SMD:SOT-23, symbol Regulator_Linear:MCP1799x-500xxTT
- removed U15.bak1, U8.bak1: TSB582, Package_DFN_QFN:DFN-8-1EP_6x5mm_P1.27mm_EP4x4mm, symbol OPAMPS GRACIDA:TSB582IYQ2T
- removed U17: LM7705, Package_SO:VSSOP-8_3x3mm_P0.65mm, symbol Regulator_SwitchedCapacitor:LM7705
- removed U20, U5: ULN2003, Package_SO:SOIC-16_4.55x10.3mm_P1.27mm, symbol Transistor_Array:ULN2003
Connections:
- no-connect marks 7 -> 4
Other:
- note removed: "MICRO"

Commit message: 05/06/26
Parts:
- J6: renamed from J7; footprint CONECTORES GRACIDA:16POS-2LINEAS-3.5PITCH -> CONECTORES GRACIDA:1728840000_17-25
- U14: renamed from U16; footprint (none) -> Package_SO:SOIC-16W_5.3x10.2mm_P1.27mm
- renumbered C40 to C30, C41 to C31, C43 to C32, C45 to C33, C46 to C34, C47 to C35, C48 to C36, C49 to C37, C50 to C38, C51 to C39, C52 to C40, C53 to C41, C57 to C42, C58 to C43, C62 to C44, C63 to C45, C64 to C46, C65 to C47, C70 to C48, C71 to C49, C72 to C50, C73 to C51, C75 to C52, C77 to C53, C78 to C54, C79 to C55, D22 to D13, D23 to D14, D24 to D15, D25 to D16, D27 to D17, D28 to D18, D29 to D19, D30 to D20, D31 to D21, IC4 to IC1, J6 to J5, L8 to L6, L10 to L7, Q2 to Q1, Q11 to Q10, Q12 to Q11, Q13 to Q12, Q3 to Q2, Q4 to Q3, Q5 to Q4, Q6 to Q5, Q7 to Q6, Q8 to Q7, Q9 to Q8, Q10 to Q9, R37 to R21, R38 to R22, R39 to R23, R40 to R24, R45 to R25, R46 to R26, R47 to R27, R48 to R28, R49 to R29, R50 to R30, R51 to R31, R52 to R32, R53 to R33, R54 to R34, R55 to R35, R56 to R36, R57 to R37, R58 to R38, R59 to R39, R60 to R40, R61 to R41, R62 to R42, R63 to R43, R64 to R44, R65 to R45, R66 to R46, R67 to R47, R68 to R48, R69 to R49, R70 to R50, R71 to R51, R72 to R52, R73 to R53, R74 to R54, R75 to R55, R76 to R56, R77 to R57, R78 to R58, R79 to R59, R80 to R60, R81 to R61, R82 to R62, R83 to R63, R84 to R64, R85 to R65, R86 to R66, R87 to R67, R88 to R68, R89 to R69, R90 to R70, R91 to R71, R92 to R72, R94 to R73, R95 to R74, R97 to R75, R98 to R76, R99 to R77, R100 to R78, R101 to R79, R102 to R80, R109 to R81, R110 to R82, R111 to R83, R112 to R84, R121 to R85, R124 to R86, TH2 to TH1, U11 to U10, U12 to U11, U13 to U12, U14 to U13, U18 to U15, U19 to U16, U6 to U5, U7 to U6, U8 to U7, U9 to U8, U10 to U9

Commit message: 22-jun-24
Connections:
- net +5V: now also U9.5 (VCC)
Other:
- moved on the sheet: R56
Changed lines of the file:
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@@
 	)
 	(junction
-		(at 350.52 190.5)
+		(at 186.69 175.26)
 		(diameter 0)
 		(color 0 0 0 0)
 	)
 	(junction
-		(at 189.23 175.26)
+		(at 350.52 190.5)
 		(diameter 0)
 		(color 0 0 0 0)
@@
 	(wire
 		(pts
-			(xy 189.23 182.88) (xy 189.23 184.15)
-		)
-		(stroke
-			(width 0)
-			(type default)
-		)
-	)
-	(wire
-		(pts
 			(xy 346.71 175.26) (xy 350.52 175.26)
 		)
@@
 	(wire
 		(pts
+			(xy 186.69 185.42) (xy 186.69 184.15)
+		)
+		(stroke
+			(width 0)
+			(type default)
+		)
+	)
+	(wire
+		(pts
 			(xy 91.44 76.2) (xy 91.44 77.47)
 		)
@@
 	(wire
 		(pts
-			(xy 186.69 175.26) (xy 189.23 175.26)
+			(xy 186.69 175.26) (xy 232.41 175.26)
 		)
 		(stroke
@@
 	(wire
 		(pts
+			(xy 186.69 176.53) (xy 186.69 175.26)
+		)
+		(stroke
+			(width 0)
+			(type default)
+		)
+	)
+	(wire
+		(pts
 			(xy 306.07 121.92) (xy 311.15 121.92)
 		)
@@
 	(wire
 		(pts
-			(xy 189.23 175.26) (xy 232.41 175.26)
-		)
-		(stroke
-			(width 0)
-			(type default)
-		)
-	)
-	(wire
-		(pts
 			(xy 246.38 36.83) (xy 248.92 36.83)
 		)
@@
 	(wire
 		(pts
+			(xy 152.4 198.12) (xy 152.4 199.39)
+		)
+		(stroke
+			(width 0)
+			(type default)
+		)
+	)
+	(wire
+		(pts
 			(xy 44.45 194.31) (xy 41.91 194.31)
 		)
@@
 	(symbol
 		(lib_id "power:GNDREF")
-		(at 189.23 184.15 0)
+		(at 186.69 185.42 0)
 		(unit 1)
 		(exclude_from_sim no)
@@
 		(dnp no)
 		(property "Reference" "#PWR0114"
-			(at 189.23 190.5 0)
+			(at 186.69 191.77 0)
 			(effects
 				(font
@@
 		)
 		(property "Value" "GND"
-			(at 193.548 183.896 0)
+			(at 191.008 185.166 0)
 			(effects
 				(font
@@
 		)
 		(property "Footprint" ""
-			(at 189.23 184.15 0)
+			(at 186.69 185.42 0)
 			(effects
 				(font
@@
 		)
 		(property "Datasheet" ""
-			(at 189.23 184.15 0)
+			(at 186.69 185.42 0)
 			(effects
 				(font
@@
 		)
 		(property "Description" "Power symbol creates a global label with name \"GNDREF\" , reference supply ground"
-			(at 189.23 184.15 0)
+			(at 186.69 185.42 0)
 			(effects
 				(font
@@
 	(symbol
 		(lib_id "Device:R_US")
-		(at 189.23 179.07 180)
+		(at 186.69 180.34 180)
 		(unit 1)
 		(exclude_from_sim no)
@@
 		(dnp no)
 		(property "Reference" "R56"
-			(at 191.77 177.7999 0)
+			(at 189.23 179.0699 0)
 			(effects
 				(font
@@
 		)
 		(property "Value" "1k"
-			(at 190.754 180.34 0)
+			(at 188.214 181.61 0)
 			(effects
 				(font
@@
 		)
 		(property "Footprint" "Resistor_SMD:R_0603_1608Metric"
-			(at 188.214 178.816 90)
+			(at 185.674 180.086 90)
 			(effects
 				(font
@@
 		)
 		(property "Datasheet" "~"
-			(at 189.23 179.07 0)
+			(at 186.69 180.34 0)
 			(effects
 				(font
@@
 		)
 		(property "Description" "Resistor, US symbol"
-			(at 189.23 179.07 0)
+			(at 186.69 180.34 0)
 			(effects
 				(font
