File: SALIDA 1.kicad_sch (KiCad schematic)
At the start: 135 parts, among them IC1 VNI4140K, J5 1728840000, J6 1728840000, Q1 MMBT3904, Q10 DMP3099L, Q11 DMP3099L, Q12 DMP3099L, Q2 MMBT3904, Q3 MMBT3904, Q4 MMBT3904, Q5 MMBT3904, Q6 MMBT3904, Q7 DMP3099L, Q8 DMP3099L, Q9 DMP3099L, U10 74LVC1G17, U11 74LVC1G17, U12 74LVC1G17, U13 TSB582, U14 ULN2003A, U15 LM7705, U16 MCP1799T-5002H/TT, U5 MCP23S17_SS, U6 ${SIM.PARAMS}, U7 74LVC1G17, U8 74LVC1G17, U9 74LVC1G17

Commit message: 13-jul-26
Parts:
- removed R62, R68, R85: 100, Resistor_SMD:R_0603_1608Metric_Pad0.98x0.95mm_HandSolder, symbol Device:R_Small_US
- removed R64, R74, R86: 1k, Resistor_SMD:R_0603_1608Metric_Pad0.98x0.95mm_HandSolder, symbol Device:R_Small_US
- removed R66, R70, R72, R76, R77, R78: 10k, Resistor_SMD:R_0603_1608Metric_Pad0.98x0.95mm_HandSolder, symbol Device:R_Small_US
- removed R69, R75: 2.2, Resistor_SMD:R_0603_1608Metric_Pad0.98x0.95mm_HandSolder, symbol Device:R_Small_US
- removed R73, R79: 0 ohms, Resistor_SMD:R_0603_1608Metric_Pad0.98x0.95mm_HandSolder, symbol Device:R_Small_US
- added R62, R68, R85: 100, Resistor_SMD:R_0603_1608Metric, symbol Device:R_US
- added R64, R74, R86: 1k, Resistor_SMD:R_0603_1608Metric, symbol Device:R_US
- added R66, R70, R72, R76, R77, R78: 10k, Resistor_SMD:R_0603_1608Metric, symbol Device:R_US
- added R69, R75: 2.2k, Resistor_SMD:R_0603_1608Metric, symbol Device:R_US
- added R73, R79: 0 ohms, Resistor_SMD:R_0603_1608Metric, symbol Device:R_US
- C42, C43: footprint Capacitor_SMD:C_0603_1608Metric_Pad1.08x0.95mm_HandSolder -> Capacitor_SMD:C_0603_1608Metric; Mouser (none) -> 346-CM105X7T106M06AT; Price (none) -> 0.455; now in the parts list
- C44: footprint (none) -> Capacitor_SMD:C_0603_1608Metric
- C46, C52, C54, C55: footprint Capacitor_SMD:C_0603_1608Metric_Pad1.08x0.95mm_HandSolder -> Capacitor_SMD:C_0603_1608Metric; Mouser (none) -> 81-GCJ188M8EC475KE8D; Price (none) -> 0.416; now in the parts list
- D21: footprint LED_SMD:LED_0402_1005Metric -> LED_SMD:LED_0603_1608Metric
- U13: footprint Package_DFN_QFN:DFN-8-1EP_6x5mm_P1.27mm_EP4x4mm -> Package_SO:SO-8_3.9x4.9mm_P1.27mm
Connections:
- net +12V: now also C55.1; no longer C55.2
- net GND: now also C46.2, C54.2, C55.2, J5.6 (MZ), R73.2, R79.2, R85.1, R86.2; no longer C46.1, C54.1, C55.1, J5.10 (GND), J5.11 (GND), J5.12 (GND), J5.13 (GND), J5.14 (GND), J5.15 (GND), J5.16 (GND), J5.9 (GND)
- net at J5.1 (DA0), R63.2, R65.2: now also J5.10 (GND), J5.11 (GND), J5.12 (GND), J5.13 (GND), J5.9 (GND)
- net at R60.2, R61.2: no longer J5.2 (DA1)
- net at Q11.3 (D), R58.2: no longer J5.3 (FUR)
- net at Q12.3 (D), R59.2: no longer J5.4 (FUL)
- net at Q10.3 (D), R57.2: no longer J5.5 (FREI)
- net at Q8.3 (D), R56.2: no longer J5.6 (MZ)
- net at Q9.3 (D), R55.1: no longer J5.7 (ICM)
- net at Q7.3 (D), R54.2: no longer J5.8 (OUT2)
- net at R65.1, U13.1 (OUT1): now also J5.15 (GND), R68.2
- net at U13.2 (IN1-): now also R75.2
- net at C47.1, U15.7 (CRES): now also C46.1; no longer C46.2
- net at R61.1, U13.7 (OUT2): now also R62.1
- net at C50.2, U15.8 (CF-): now also C52.2; no longer C52.1
- net at C50.1, U15.1 (CF+): now also C52.1; no longer C52.2
- net at C48.2, C49.1, D21.2 (A)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: now also C54.1; no longer C54.2
- net at D21.1 (K): now also R86.1
- net at U13.6 (IN2-): now also R69.2
- net at U15.3 (SD): now also R85.2
- new net: R62.2, R64.1
- new net: R64.2, R66.1
- new net: R75.1, R76.1, R78.2
- new net: R76.2, R77.1
- new net: R72.1, R73.1
- new net: R69.1, R70.1, R72.2
- new net: R78.1, R79.1
- new net: R66.2, R70.2
- new net: R74.1, R77.2
- new net: R68.1, R74.2
Other:
- moved on the sheet: C48, C49, D21, J5, R80, U13A, U16

Commit message: 13-jul-26_6pm
Parts:
- renumbered R56 to R55, R55 to R56, R69 to R68, R70 to R69, R68 to R70, R74 to R73, R73 to R74, R80 to R79, R79 to R80
