File: SALIDA 1.kicad_sch (KiCad schematic)
At the start: 135 parts, among them IC1 VNI4140K, J5 1728840000, J6 1728840000, Q1 MMBT3904, Q10 DMP3099L, Q11 DMP3099L, Q12 DMP3099L, Q2 MMBT3904, Q3 MMBT3904, Q4 MMBT3904, Q5 MMBT3904, Q6 MMBT3904, Q7 DMP3099L, Q8 DMP3099L, Q9 DMP3099L, U10 74LVC1G17, U11 74LVC1G17, U12 74LVC1G17, U13 TSB582, U14 ULN2003A, U15 LM7705, U16 MCP1799T-5002H/TT, U5 MCP23S17_SS, U6 ${SIM.PARAMS}, U7 74LVC1G17, U8 74LVC1G17, U9 74LVC1G17

Commit message: 21-JUL-26
Connections:
- net at J5.15 (GND), R65.1, U13.1 (OUT1): no longer R70.2
- net at J5.7 (ICM): now also J5.8 (OUT2), R70.2
Other:
- moved on the sheet: J5
