File: _autosave-01_IO-ASD-PLUS.kicad_sch (KiCad schematic)
At the start: 2 parts

Commit message: 15-mayo-26
15 mayo 26
Other:
- sheet ENTRADAS ports: added Error_Conn_Entrada_+24v; removed none
- sheet ENTRADAS1 ports: added Error_Conn_Entrada_+24v; removed none
Changed lines of the file:
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@@
 	)
 	(sheet
-		(at 257.8354 41.91)
-		(size 15.621 19.685)
+		(at 257.8354 41.275)
+		(size 15.621 20.32)
 		(exclude_from_sim no)
 		(in_bom yes)
@@
 		)
 		(property "Sheetname" "ENTRADAS1"
-			(at 257.3274 40.894 0)
+			(at 257.3274 40.259 0)
 			(effects
 				(font
@@
 		)
 		(property "Sheetfile" "ENTRADAS.kicad_sch"
-			(at 258.0894 62.484 0)
+			(at 258.0894 61.849 0)
 			(effects
 				(font
@@
 				)
 				(justify left)
+			)
+		)
+		(pin "Error_Conn_Entrada_+24v" output
+			(at 273.4564 43.18 0)
+			(effects
+				(font
+					(size 0.6858 0.6858)
+					(color 255 0 0 1)
+				)
+				(justify right)
 			)
 		)
@@
 				(font
 					(size 1.27 1.27)
+					(color 255 0 0 1)
 				)
 				(justify right)
@@
 				(font
 					(size 1.27 1.27)
+					(color 255 0 0 1)
 				)
 				(justify right)
@@
 			)
 		)
+		(pin "Error_Conn_Entrada_+24v" output
+			(at 273.4564 68.58 0)
+			(effects
+				(font
+					(size 0.6858 0.6858)
+					(color 255 0 0 1)
+				)
+				(justify right)
+			)
+		)
 		(instances
 			(project "01_IO-ASD-PLUS"
@@
 			(effects
 				(font
-					(size 0.635 0.635)
+					(size 0.6858 0.6858)
 					(color 255 0 0 1)
 				)
