File: 01_IO-ASD-PLUS.kicad_sch (KiCad schematic)
At the start: 2 parts

Commit message: 15-may-26
Other:
- sheet ENTRADAS ports: added Error_Conn_Entrada_+24v; removed none
- sheet ENTRADAS1 ports: added Error_Conn_Entrada_+24v; removed none
- sheet Ent Especial ports: added AN0_POT, AN1_POT, Error_Conn_Entrada_ESP+24v, opto_out1, opto_out2, opto_out3, opto_out4; removed none
- sheet Processador ports: added !CS_Exp, !CS_J5_J6, ADC2, ADC3, BUSY_DISPLAY, DAC0, DAC1, INTA_J5_J6, INT_FT812, METAL_INTERRUPCION, MO1, MO2, MO3, MO4, Metal1, Metal2; removed none

Commit message: pcb 18 may 26
 falta poner la fuente de +12/ ya esta casi todo
Other:
- added sheet Error (error.kicad_sch)
- sheet FUENTES ports: added Error_3.3v_comm, Error_3.3v_proc; removed none

Commit message: 22 mayo 26 actualizacion
se actualizo la PCB para la rama laptop Antigua
Parts:
- renumbered R180 to R1, R181 to R2
Changed lines of the file:
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@@
 		(on_board yes)
 		(dnp no)
-		(property "Reference" "#PWR0294"
+		(property "Reference" "#PWR01"
 			(at 185.42 30.48 0)
 			(effects
@@
 			(project "01_IO-ASD-PLUS"
 				(path "/38a2da3c-ed29-422f-ab41-066ccf490e61"
-					(reference "#PWR0294")
+					(reference "#PWR01")
 					(unit 1)
 				)
@@
 		(on_board yes)
 		(dnp no)
-		(property "Reference" "R180"
+		(property "Reference" "R1"
 			(at 186.182 29.21 0)
 			(effects
@@
 			(project "01_IO-ASD-PLUS"
 				(path "/38a2da3c-ed29-422f-ab41-066ccf490e61"
-					(reference "R180")
+					(reference "R1")
 					(unit 1)
 				)
@@
 		(on_board yes)
 		(dnp no)
-		(property "Reference" "R181"
+		(property "Reference" "R2"
 			(at 197.612 30.48 0)
 			(effects
@@
 			(project "01_IO-ASD-PLUS"
 				(path "/38a2da3c-ed29-422f-ab41-066ccf490e61"
-					(reference "R181")
+					(reference "R2")
 					(unit 1)
 				)
