File: Comm_Serial.kicad_sch (KiCad schematic)
At the start: 15 parts, among them J10 1728810000, U25 MAX3232, U28 MAX3232

Commit message: 15-mayo-26
15 mayo 26
Parts:
- added C129, C130, C140: 0.1uF, Capacitor_SMD:C_0603_1608Metric_Pad1.08x0.95mm_HandSolder, symbol Device:C_Small
- added J9: 8P8C_LED_Shielded, symbol Connector:8P8C_LED_Shielded
- added L10: 200uH, Inductores_GSI:DLW43_MUR, symbol INDUCTORES_GSI:DLW43MH201XK2L
- added R136, R137, R138, R139, R140, R176, R177, R187, R229, R230: 0R, Resistor_SMD:R_0603_1608Metric, symbol Device:R_US
- added R178: 1.5K, Resistor_SMD:R_0603_1608Metric, symbol Device:R_US
- added R179: 620, Resistor_SMD:R_0603_1608Metric, symbol Device:R_US
- added R182: 120 1%, Resistor_SMD:R_0603_1608Metric, symbol Device:R_US
- added T3: Transformer_1P_1S, symbol Device:Transformer_1P_1S
- added TP10, TP11, TP12, TP13, TP14, TP15, TP16, TP17, TP18, TP19, TP20, TP21, TP22, TP23, TP24: ~, symbol Connector:TestPoint
- added TP8: INT TestPoint, symbol Connector:TestPoint
- added TP9: PD TestPoint, symbol Connector:TestPoint
- added U29: LTC6820, Package_SO:MSOP-16-1EP_3x4.039mm_P0.5mm_EP1.651x2.845mm_ThermalVias, symbol MICROS_DIGITAL_GSI_v2:LTC6820
Connections:
- net PD_N_LOGIC is gone; now on net INT_N_LOGIC: R134.2, U28.10 (T2IN)
- net +3.3v: now also C129.1, C130.2, C140.1, R136.2, R137.2, R139.2, R140.2, U29.1 (EN), U29.6 (VDDs), U29.9 (VDD)
- net Busy_Tx_Logic: now also TP21.1
- net GND: now also C129.2, C130.1, C140.2, J9.8, R138.1, R176.2, R177.2, R179.2, R187.2, U29.14 (GND)
- net INT_N_LOGIC: now also TP22.1, TP23.1
- net Metal_INT_Logic: now also TP24.1
- net Serial_Rx_from_Cons_Serv_Logic: now also TP20.1
- net Serial_Rx_from_uP_Logic: now also TP19.1
- net Serial_Tx_a_Consola_Serv_Logic: now also TP18.1
- net Serial_Tx_a_Proc_Logic: now also TP17.1
- net INT_N_RS232: no longer names the net of J10.10 (X9)
- net INT_N_RS232: now also R230.2; no longer U28.13 (R1IN)
- net PD_N_RS232: no longer names the net of U28.7 (T2OUT)
- net PD_N_RS232: now also J9.3, R229.1, TP9.1; no longer J10.8 (X8)
- new net: R140.1, R177.1, U29.7 (POL)
- new net: L10.1, U29.10 (IM)
- new net: L10.2, R182.2, T3.2 (AA)
- new net: L10.3, R182.1, T3.3 (AB)
- new net: L10.4, U29.11 (IP)
- new net: J9.1, T3.4 (SA), TP16.1
- new net: R178.2, R179.1, TP14.1, U29.15 (ICMP)
- new net: J10.8 (X8), R229.2
- new net: J9.2, T3.1 (SB), TP15.1
- new net: R136.1, U29.12 (MSTR)
- new net: R139.1, R176.1, U29.8 (PHA)
- new net: R178.1, U29.16 (IBIAS)
- new net: R137.1, R138.2, U29.13 (SLOW)
- new net: J9.SH, R187.1
- new net !CS_LTC6820: TP13.1, U29.5 (!CS)
- new net +24V: J9.7
- new net Led_ctrl/INT: J9.6, R230.1, TP8.1, U28.13 (R1IN)
- new net Led_ctrl/LED1_A: J9.10
- new net Led_ctrl/LED1_C: J9.9
- new net Led_ctrl/LED2_A: J9.12
- new net Led_ctrl/LED2_C: J9.11
- new net MISO: TP11.1, U29.3 (MISO)
- new net MOSI: TP10.1, U29.2 (MOSI)
- new net SCKL: TP12.1, U29.4 (SCKL)
- no-connect marks 0 -> 2
Other:
- added sheet Led_ctrl (Led_ctrl.kicad_sch)
- note added: "conector ethernet terminarlo y cto leds"
- note added: "poner aqui el voltaje a medir"
- note added: "resistencias de pullup de MISO Y MOSI esta en root sheet"

Commit message: pcb 18 may 26
 falta poner la fuente de +12/ ya esta casi todo
Parts:
- added F4: Fuse, symbol Device:Fuse
Connections:
- net +3.3v: no longer C129.1, C130.2, C140.1, C78.1, C79.1, R136.2, R137.2, R139.2, R140.2, U25.16 (VCC), U28.16 (VCC), U29.1 (EN), U29.6 (VDDs), U29.9 (VDD)
- net 600mA: now reaches R178.2, R179.1, TP14.1, U29.15 (ICMP)
- net +2.0v: now reaches R178.1, U29.16 (IBIAS)
- new net +3.3v_Fuse3: C129.1, C130.2, C140.1, F4.2, R136.2, R137.2, R139.2, R140.2, U29.1 (EN), U29.6 (VDDs), U29.9 (VDD)
- new net +3.3v_Fuse_comm: C78.1, C79.1, F4.1, U25.16 (VCC), U28.16 (VCC)
Other:
- note removed: "poner aqui el voltaje a medir"
- moved on the sheet: R178

Commit message: 22 mayo 26 actualizacion
se actualizo la PCB para la rama laptop Antigua
Parts:
- renumbered C80 to C162, C129 to C163, C78 to C164, C130 to C165, C82 to C166, C122 to C167, C81 to C168, C140 to C169, C127 to C170, C128 to C171, C125 to C172, C79 to C173, C126 to C174, F4 to F7, J10 to J18, J9 to J19, L10 to L23, R179 to R255, R178 to R256, R139 to R257, R140 to R258, R176 to R259, R177 to R260, R138 to R261, R136 to R262, R137 to R263, R182 to R264, R229 to R265, R230 to R266, R187 to R267, R134 to R268, R135 to R269, T3 to T1, TP18 to TP11, TP11 to TP12, TP19 to TP13, TP12 to TP14, TP20 to TP15, TP13 to TP16, TP16 to TP17, TP15 to TP18, TP9 to TP19, TP8 to TP20, TP14 to TP8, TP17 to TP9, U25 to U36, U29 to U37, U28 to U38
Connections:
- net at L23.2, R264.2: now also T1.1 (AA); no longer T1.2 (AA)
- net at L23.3, R264.1: now also T1.2 (AB); no longer T1.3 (AB)
- net at J19.1, TP17.1: now also T1.3 (SA); no longer T1.4 (SA)
- net at J19.2, TP18.1: now also T1.4 (SB); no longer T1.1 (SB)

Commit message: 05/06/26
Parts:
- renumbered C162 to C117, C163 to C118, C164 to C119, C165 to C120, C166 to C121, C167 to C122, C168 to C123, C169 to C124, C170 to C125, C171 to C126, C172 to C127, C173 to C128, C174 to C129, J18 to J14, J19 to J15, L23 to L17, R255 to R182, R256 to R183, R257 to R184, R258 to R185, R259 to R186, R260 to R187, R261 to R188, R262 to R189, R263 to R190, R264 to R191, R265 to R192, R266 to R193, R267 to R194, R268 to R195, R269 to R196, U36 to U38, U37 to U39, U38 to U40
