File: Comm_Serial.kicad_sch (KiCad schematic)
At the start: 53 parts, among them J14 1728810000, J15 8P8C_LED_Shielded, T1 Transformer_1P_1S, U38 MAX3232, U39 LTC6820, U40 MAX3232

Commit message: 13-jul-26_6pm
Parts:
- renumbered J14 to J13, J15 to J14, U38 to U35, U39 to U36, U40 to U37

Commit message: 24/07/2026
Parts:
- J14: footprint (none) -> CONECTORES GRACIDA:WE-RJ45LAN
- T1: footprint (none) -> TRANSFORMADORES GRACIDA:TRANFORMADOR_1001C
Connections:
- net at R187.1, U36.7 (POL): no longer R185.1
- net at L17.1: now also R191.1, T1.2 (AB); no longer U36.10 (IM)
- net at R191.2, T1.1 (AA): now also L17.4; no longer L17.2
- net at U36.11 (IP): now also L17.3; no longer L17.4
- new net: L17.2, U36.10 (IM)
Changed lines of the file:
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@@
 	)
 	(junction
-		(at 77.47 171.45)
-		(diameter 0)
-		(color 0 0 0 0)
-	)
-	(junction
 		(at 54.61 72.39)
 		(diameter 0)
@@
 	(wire
 		(pts
-			(xy 77.47 179.07) (xy 77.47 171.45)
+			(xy 77.47 166.37) (xy 77.47 179.07)
 		)
 		(stroke
@@
 	(wire
 		(pts
-			(xy 77.47 171.45) (xy 77.47 166.37)
-		)
-		(stroke
-			(width 0)
-			(type default)
-		)
-	)
-	(wire
-		(pts
 			(xy 182.88 148.59) (xy 179.07 148.59)
 		)
@@
 	(wire
 		(pts
-			(xy 63.5 171.45) (xy 77.47 171.45)
-		)
-		(stroke
-			(width 0)
-			(type default)
-		)
-	)
-	(wire
-		(pts
 			(xy 259.08 58.42) (xy 259.08 72.39)
 		)
@@
 	)
 	(symbol
-		(lib_id "INDUCTORES_GSI:DLW43MH201XK2L")
-		(at 123.19 134.62 0)
-		(unit 1)
-		(exclude_from_sim no)
-		(in_bom yes)
-		(on_board yes)
-		(dnp no)
-		(fields_autoplaced yes)
-		(property "Reference" "L17"
-			(at 129.54 132.08 0)
-			(effects
-				(font
-					(size 1.27 1.27)
-				)
-			)
-		)
-		(property "Value" "200uH"
-			(at 129.54 134.62 0)
-			(effects
-				(font
-					(size 1.27 1.27)
-				)
-			)
-		)
-		(property "Footprint" "Inductores_GSI:DLW43_MUR"
-			(at 123.19 134.62 0)
-			(effects
-				(font
-					(size 1.27 1.27)
-				)
-				(hide yes)
-			)
-		)
-		(property "Datasheet" "https://www.mouser.mx/datasheet/3/76/1/DLW43MH201XK2#.pdf"
-			(at 123.19 134.62 0)
-			(effects
-				(font
-					(size 1.27 1.27)
-				)
-				(hide yes)
-			)
-		)
-		(property "Description" "1812 4.5x3.2mm 110mA"
-			(at 123.19 134.62 0)
-			(effects
-				(font
-					(size 1.27 1.27)
-				)
-				(hide yes)
-			)
-		)
-		(pin "3"
-		)
-		(pin "4"
-		)
-		(pin "1"
-		)
-		(pin "2"
-		)
-		(instances
-			(project ""
-				(path "/38a2da3c-ed29-422f-ab41-066ccf490e61/b83e4991-9806-4c27-8269-31bebca0e905"
-					(reference "L17")
-					(unit 1)
-				)
-			)
-		)
-	)
-	(symbol
 		(lib_id "Device:C_Small")
 		(at 212.09 25.4 270)
@@
 			)
 		)
-		(property "Footprint" ""
+		(property "Footprint" "TRANSFORMADORES GRACIDA:TRANFORMADOR_1001C"
 			(at 162.56 143.51 0)
 			(effects
@@
 	)
 	(symbol
+		(lib_name "DLW43MH201XK2L_1")
+		(lib_id "INDUCTORES_GSI:DLW43MH201XK2L")
+		(at 135.89 152.4 180)
+		(unit 1)
+		(exclude_from_sim no)
+		(in_bom yes)
+		(on_board yes)
+		(dnp no)
+		(fields_autoplaced yes)
+		(property "Reference" "L17"
+			(at 129.54 132.08 0)
+			(effects
+				(font
+					(size 1.27 1.27)
+				)
+			)
+		)
+		(property "Value" "200uH"
+			(at 129.54 134.62 0)
+			(effects
+				(font
+					(size 1.27 1.27)
+				)
+			)
+		)
+		(property "Footprint" "Inductores_GSI:DLW43_MUR"
+			(at 135.89 152.4 0)
+			(effects
+				(font
+					(size 1.27 1.27)
+				)
+				(hide yes)
+			)
+		)
+		(property "Datasheet" "https://www.mouser.mx/datasheet/3/76/1/DLW43MH201XK2#.pdf"
+			(at 135.89 152.4 0)
+			(effects
+				(font
+					(size 1.27 1.27)
+				)
+				(hide yes)
+			)
+		)
+		(property "Description" "1812 4.5x3.2mm 110mA"
+			(at 135.89 152.4 0)
+			(effects
+				(font
+					(size 1.27 1.27)
+				)
+				(hide yes)
+			)
+		)
+		(pin "4"
+		)
+		(pin "1"
+		)
+		(pin "2"
+		)
+		(pin "3"
+		)
+		(instances
+			(project ""
+				(path "/38a2da3c-ed29-422f-ab41-066ccf490e61/b83e4991-9806-4c27-8269-31bebca0e905"
+					(reference "L17")
+					(unit 1)
+				)
+			)
+		)
+	)
+	(symbol
 		(lib_id "Connector:8P8C_LED_Shielded")
 		(at 207.01 142.24 0)
@@
 			)
 		)
-		(property "Footprint" ""
+		(property "Footprint" "CONECTORES GRACIDA:WE-RJ45LAN"
 			(at 207.01 141.605 90)
 			(effects
