File: ENTRADAS.kicad_sch (KiCad schematic)
At the start: 27 parts, among them IC14 ILD206T, IC15 ILD206T, IC16 ILD206T, J7 1728840000, J8 1728810000, U11 MAX3227

Commit message: 14-Mayo-26
se agregaron varias sheet de esquematico crecio al 80% la parte de esquematico
Parts:
- removed R56: 10k, Capacitor_SMD:C_0603_1608Metric_Pad1.08x0.95mm_HandSolder, symbol Device:R_Small_US
- added C120, C121: 0.1uF, Capacitor_SMD:C_0603_1608Metric_Pad1.08x0.95mm_HandSolder, symbol Device:C_Small
- added IC18, IC19: ILD206T, SOIC:SOIC 8, symbol OPTOACOPLADORES:ILD206T
- added J*1: 1728840000, CONECTORES GRACIDA:16POS-2LINEAS-3.5PITCH, symbol CONECTORES GRACIDA:Weidmüller 1728840000 16pos P3.5mm socket
- added L16: L_Iron_Small, symbol Device:L_Iron_Small
- added R132, R169, R172, R173: 2.2k, Capacitor_SMD:C_0603_1608Metric_Pad1.08x0.95mm_HandSolder, symbol Device:R_Small_US
- added R168, R170, R171, R174, R175: 4.7k, Capacitor_SMD:C_0603_1608Metric_Pad1.08x0.95mm_HandSolder, symbol Device:R_Small_US
- added TH4: B59985C120A70, TERMISTORES GRACIDA:B59985C0120A070, symbol Device:Thermistor_PTC
- R131: renamed from R55; value 10k -> 4.7k
- renumbered C38 to C131, C39 to C134, C40 to C135, C41 to C136, C42 to C137, C43 to C138, C44 to C139, IC14 to IC15, IC15 to IC25, IC16 to IC26, J7 to J16, J8 to J17, L7 to L19, R53 to R129, R54 to R130, R57 to R196, R58 to R197, R59 to R198, R60 to R199, R61 to R200, R62 to R201, R63 to R202, R64 to R207, TH2 to TH8, U11 to U27
Connections:
- net +24V: now also TH4.2
- net +3.3V: now also R131.1, R168.1, R170.1, R171.1, R174.1, R175.1; no longer IC15.6 (C_3), IC15.8 (C_4)
- net GND: now also IC15.5 (E_1), IC15.7 (E_2), C120.1, C121.1, IC18.2 (C_1), IC18.4 (C_2), IC18.5 (E_1), IC18.7 (E_2), IC19.2 (C_1), IC19.4 (C_2), IC19.5 (E_1), IC19.7 (E_2), J*1. (9); no longer R131.2
- net at R129.1: now also J*1. (9); no longer J16.34 (BIN)
- net at R130.1: now also J*1. (9); no longer J16.37 (FS)
- new net: J*1. (9), R169.1
- new net: J*1. (9), R172.1
- new net: C120.2, J*1. (9), L16.1
- new net: J*1. (9), R132.1
- new net: J*1. (9), R173.1
- new net: IC18.3 (A_2), R169.2
- new net: C121.2, L16.2, TH4.1
- new net: IC19.1 (A_1), R172.2
- new net: IC18.1 (A_1), R132.2
- new net: IC19.3 (A_2), R173.2
- new net opto_out1: IC15.8 (C_4), R131.2
- new net opto_out2: IC15.6 (C_3), R168.2
- new net opto_out3: IC18.8 (C_4), R170.2
- new net opto_out4: IC18.6 (C_3), R171.2
- new net opto_out5: IC19.8 (C_4), R174.2
- new net opto_out6: IC19.6 (C_3), R175.2
Other:
- moved on the sheet: C131, C134, C135, C136, C137, C138, C139, IC15, IC25, IC26, J16, J17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

Commit message: 15-mayo-26
15 mayo 26
Connections:
- net Error_Conn_Entrada_+24v: now reaches C120.2, J*1. (9), L16.1

Commit message: 22 mayo 26 actualizacion
se actualizo la PCB para la rama laptop Antigua
Parts:
- removed IC15, IC18, IC19, IC25: ILD206T, SOIC:SOIC 8, symbol OPTOACOPLADORES:ILD206T
- removed R196, R197: 2.2k, Capacitor_SMD:C_0603_1608Metric_Pad1.08x0.95mm_HandSolder, symbol Device:R_Small_US
- removed R200, R201: 10k, Capacitor_SMD:C_0603_1608Metric_Pad1.08x0.95mm_HandSolder, symbol Device:R_Small_US
- added U23, U26, U27: ILD206T, Package_SO:SOIC-8_3.9x4.9mm_P1.27mm, symbol OPTOACOPLADORES:ILD206T
- C82: renamed from C131; now not fitted; now left out of the parts list
- C83: renamed from C134; now not fitted; now left out of the parts list
- C84: renamed from C135; now not fitted; now left out of the parts list
- C85: renamed from C136; now not fitted; now left out of the parts list
- C86: renamed from C137; now not fitted; now left out of the parts list
- C87: renamed from C138; now not fitted; now left out of the parts list
- C88: renamed from C139; now not fitted; now left out of the parts list
- IC6: renamed from IC26; now not fitted; now left out of the parts list
- J13: renamed from J17; now not fitted; now left out of the parts list
- J8: renamed from J16; footprint CONECTORES GRACIDA:1728840000_33-48 -> CONECTORES GRACIDA:16POS-2LINEAS-3.5PITCH; now not fitted; now left out of the parts list
- L12: renamed from L19; now not fitted; now left out of the parts list
- R138: renamed from R198; now not fitted; now left out of the parts list
- R139: renamed from R199; now not fitted; now left out of the parts list
- R148: renamed from R202; now not fitted; now left out of the parts list
- R149: renamed from R207; now not fitted; now left out of the parts list
- TH4: renamed from TH8; now not fitted; now left out of the parts list
- U42: renamed from U27; now not fitted; now left out of the parts list
- renumbered C121 to C80, C120 to C81, J*1 to J9, L16 to L11, R130 to R140, R129 to R141, R132 to R142, R169 to R143, R172 to R144, R173 to R145, R131 to R150, R170 to R151, R168 to R152, R174 to R153, R171 to R154, R175 to R155, TH4 to TH3
Connections:
- net GND: now also J13.3 (X1), U23.2 (C_1), U23.4 (C_2), U23.5 (E_1), U23.7 (E_2), U26.2 (C_1), U26.4 (C_2), U26.5 (E_1), U26.7 (E_2), U27.2 (C_1), U27.4 (C_2), U27.5 (E_1), U27.7 (E_2); no longer J13.5 (X2)
- net opto_out1: now also U23.8 (C_4)
- net opto_out2: now also U23.6 (C_3)
- net opto_out3: now also U26.8 (C_4)
- net opto_out4: now also U26.6 (C_3)
- net opto_out5: now also U27.8 (C_4)
- net opto_out6: now also U27.6 (C_3)
- net at R143.2: now also U26.3 (A_2)
- net at R144.2: now also U27.1 (A_1)
- net at R141.2: now also U23.3 (A_2)
- net at R140.2: now also U23.1 (A_1)
- net at R142.2: now also U26.1 (A_1)
- net at R145.2: now also U27.3 (A_2)
- net at U42.11 (T1IN): no longer J13.4 (X6)
- net at U42.9 (R1OUT): now also J13.10 (X9); no longer J13.2 (X5)

Commit message: 26-05-26
Parts:
- removed C82, C83, C84, C85, C86, C87, C88: 0.1uF, Capacitor_SMD:C_0603_1608Metric_Pad1.08x0.95mm_HandSolder, symbol Device:C_Small
- removed IC6: ILD206T, SOIC:SOIC 8, symbol OPTOACOPLADORES:ILD206T
- removed J13: 1728810000, CONECTORES GRACIDA:1728810000, symbol CONECTORES GRACIDA:1728810000
- removed J8: 1728840000, CONECTORES GRACIDA:16POS-2LINEAS-3.5PITCH, symbol CONECTORES GRACIDA:1728840000_33-48
- removed L12: 10uH, Inductor_SMD:L_0603_1608Metric_Pad1.05x0.95mm_HandSolder, symbol Device:L_Small
- removed R138, R139: 2.2k, Capacitor_SMD:C_0603_1608Metric_Pad1.08x0.95mm_HandSolder, symbol Device:R_Small_US
- removed R148, R149: 10k, Capacitor_SMD:C_0603_1608Metric_Pad1.08x0.95mm_HandSolder, symbol Device:R_Small_US
- removed TH4: B59985C120A70, TERMISTORES GRACIDA:B59985C0120A070, symbol Device:Thermistor_PTC
- removed U42: MAX3227, Package_SO:SSOP-16_5.3x6.2mm_P0.65mm, symbol Interface_UART:MAX3227
Connections:
- no-connect marks 2 -> 0

Commit message: 05/06/26
Parts:
- removed J9: 1728840000, CONECTORES GRACIDA:16POS-2LINEAS-3.5PITCH, symbol CONECTORES GRACIDA:Weidmüller 1728840000 16pos P3.5mm socket
- added J7: 1728840000, CONECTORES GRACIDA:16POS-2LINEAS-3.5PITCH, symbol CONECTORES GRACIDA:1728840000_1
- renumbered C80 to C56, C81 to C57, L11 to L8, R140 to R87, R141 to R88, R142 to R89, R143 to R90, R144 to R91, R145 to R92, R150 to R93, R151 to R94, R152 to R95, R153 to R96, R154 to R97, R155 to R98, TH3 to TH2, U23 to U17, U26 to U18, U27 to U19
Connections:
- net Error_Conn_Entrada_+24v: now also J7.1, J7.3, J7.4, J7.6, J7.8
- net GND: now also J7.11, J7.12, J7.14, J7.16, J7.9
- net at R90.1: now also J7.13
- net at R91.1: now also J7.15
- net at R88.1: now also J7.2
- net at R87.1: now also J7.5
- net at R89.1: now also J7.10
- net at R92.1: now also J7.7
