File: ENTRADAS.kicad_sch (KiCad schematic)
At the start: 20 parts, among them J7 1728840000, U17 ILD206T, U18 ILD206T, U19 ILD206T

Commit message: 13-jul-26_6pm
Parts:
- L8: footprint (none) -> Inductor_SMD:L_0603_1608Metric_Pad1.05x0.95mm_HandSolder
