File: FUENTES.kicad_sch (KiCad schematic)
At the start: 76 parts, among them J4 1604470000, U2 LTC3646E, U21 LTC3646EMSEPBF, U3 KF33BDT, U4 TLV70212_SOT23-5

Commit message: 05/06/26
Parts:
- C11, C12: footprint Capacitor_THT:C_Rect_L26.5mm_W11.5mm_P22.50mm_MKS4 -> Capacitor_THT:C_Rect_L10.0mm_W3.0mm_P7.50mm_FKS3_FKP3
- F1, F2, F3, F4, F5: value Fuse -> SF-2410HI050T-2; footprint (none) -> Fuse:Fuse_Littelfuse-NANO2-451_453
- renumbered L25 to L2, U21 to U1
Other:
- note added: "REVISAR, AL ESTAR CONECTADO ASI, TODOS LOS GND SE VUELVEN -12VV"
- note added: "revisar que sean iguales en el datasheet"
Changed lines of the file:
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@@
 		)
 	)
+	(text "revisar que sean iguales en el datasheet"
+		(exclude_from_sim no)
+		(at 196.85 106.172 0)
+		(effects
+			(font
+				(size 1.27 1.27)
+			)
+		)
+	)
 	(text "power switch\n"
 		(exclude_from_sim no)
@@
 		)
 	)
+	(text "REVISAR, AL ESTAR CONECTADO ASI, TODOS LOS GND SE VUELVEN -12VV"
+		(exclude_from_sim no)
+		(at 241.554 86.106 0)
+		(effects
+			(font
+				(size 1.27 1.27)
+			)
+		)
+	)
 	(junction
 		(at 76.2 22.86)
@@
 		(on_board yes)
 		(dnp no)
-		(property "Reference" "#PWR07"
+		(property "Reference" "#PWR09"
 			(at 30.48 105.41 0)
 			(effects
@@
 			(project "01_IO-ASD-PLUS"
 				(path "/38a2da3c-ed29-422f-ab41-066ccf490e61/02316654-b7a5-4033-a293-af0194a6badf"
-					(reference "#PWR07")
+					(reference "#PWR09")
 					(unit 1)
 				)
@@
 			)
 		)
-		(property "Value" "Fuse"
+		(property "Value" "SF-2410HI050T-2"
 			(at 216.408 81.28 90)
 			(effects
@@
 			)
 		)
-		(property "Footprint" ""
+		(property "Footprint" "Fuse:Fuse_Littelfuse-NANO2-451_453"
 			(at 217.17 86.868 90)
 			(effects
@@
 		(dnp no)
 		(property "Reference" "F2"
-			(at 111.76 83.058 90)
+			(at 111.252 77.216 90)
 			(effects
 				(font
@@
 			)
 		)
-		(property "Value" "Fuse"
-			(at 112.014 80.772 90)
+		(property "Value" "SF-2410HI050T-2"
+			(at 112.522 80.772 90)
 			(effects
 				(font
@@
 			)
 		)
-		(property "Footprint" ""
+		(property "Footprint" "Fuse:Fuse_Littelfuse-NANO2-451_453"
 			(at 115.57 80.518 90)
 			(effects
@@
 		(on_board yes)
 		(dnp no)
-		(property "Reference" "#PWR015"
+		(property "Reference" "#PWR014"
 			(at 43.18 158.75 0)
 			(effects
@@
 			(project "01_IO-ASD-PLUS"
 				(path "/38a2da3c-ed29-422f-ab41-066ccf490e61/02316654-b7a5-4033-a293-af0194a6badf"
-					(reference "#PWR015")
+					(reference "#PWR014")
 					(unit 1)
 				)
@@
 		(on_board yes)
 		(dnp no)
-		(property "Reference" "#PWR014"
+		(property "Reference" "#PWR015"
 			(at 45.72 105.41 0)
 			(effects
@@
 			(project "01_IO-ASD-PLUS"
 				(path "/38a2da3c-ed29-422f-ab41-066ccf490e61/02316654-b7a5-4033-a293-af0194a6badf"
-					(reference "#PWR014")
+					(reference "#PWR015")
 					(unit 1)
 				)
@@
 		(on_board yes)
 		(dnp no)
-		(property "Reference" "#PWR06"
+		(property "Reference" "#PWR08"
 			(at 30.48 74.93 0)
 			(effects
@@
 			(project "01_IO-ASD-PLUS"
 				(path "/38a2da3c-ed29-422f-ab41-066ccf490e61/02316654-b7a5-4033-a293-af0194a6badf"
-					(reference "#PWR06")
+					(reference "#PWR08")
 					(unit 1)
 				)
@@
 		(on_board yes)
 		(dnp no)
-		(property "Reference" "#PWR09"
+		(property "Reference" "#PWR07"
 			(at 26.67 143.51 0)
 			(effects
@@
 			(project "01_IO-ASD-PLUS"
 				(path "/38a2da3c-ed29-422f-ab41-066ccf490e61/02316654-b7a5-4033-a293-af0194a6badf"
-					(reference "#PWR09")
+					(reference "#PWR07")
 					(unit 1)
 				)
@@
 	)
 	(symbol
+		(lib_id "Connector:TestPoint")
+		(at 50.8 46.99 0)
+		(unit 1)
+		(exclude_from_sim no)
+		(in_bom yes)
+		(on_board yes)
+		(dnp no)
+		(fields_autoplaced yes)
+		(property "Reference" "TP4"
+			(at 53.34 43.6879 0)
+			(effects
+				(font
+					(size 1.27 1.27)
+				)
+				(justify left)
+			)
+		)
+		(property "Value" "TestPoint"
+			(at 53.34 44.9579 0)
+			(effects
+				(font
+					(size 1.27 1.27)
+				)
+				(justify left)
+				(hide yes)
+			)
+		)
+		(property "Footprint" "TestPoint:TestPoint_Loop_D1.80mm_Drill1.0mm_Beaded"
+			(at 55.88 46.99 0)
+			(effects
+				(font
+					(size 1.27 1.27)
+				)
+				(hide yes)
+			)
+		)
+		(property "Datasheet" "~"
+			(at 55.88 46.99 0)
+			(effects
+				(font
+					(size 1.27 1.27)
+				)
+				(hide yes)
+			)
+		)
+		(property "Description" "test point"
+			(at 50.8 46.99 0)
+			(effects
+				(font
+					(size 1.27 1.27)
+				)
+				(hide yes)
+			)
+		)
+		(pin "1"
+		)
+		(instances
+			(project "01_IO-ASD-PLUS"
+				(path "/38a2da3c-ed29-422f-ab41-066ccf490e61/02316654-b7a5-4033-a293-af0194a6badf"
+					(reference "TP4")
+					(unit 1)
+				)
+			)
+		)
+	)
+	(symbol
 		(lib_id "power:GNDREF")
 		(at 194.31 40.64 0)
@@
 		(dnp no)
 		(fields_autoplaced yes)
-		(property "Reference" "U21"
+		(property "Reference" "U1"
 			(at 91.44 120.65 0)
 			(effects
@@
 			(project "01_IO-ASD-PLUS"
 				(path "/38a2da3c-ed29-422f-ab41-066ccf490e61/02316654-b7a5-4033-a293-af0194a6badf"
-					(reference "U21")
+					(reference "U1")
 					(unit 1)
 				)
@@
 		(dnp no)
 		(fields_autoplaced yes)
-		(property "Reference" "L25"
+		(property "Reference" "L2"
 			(at 58.42 33.655 0)
 			(effects
@@
 			(project ""
 				(path "/38a2da3c-ed29-422f-ab41-066ccf490e61/02316654-b7a5-4033-a293-af0194a6badf"
-					(reference "L25")
+					(reference "L2")
 					(unit 1)
 				)
@@
 			)
 		)
-		(property "Footprint" "Capacitor_THT:C_Rect_L26.5mm_W11.5mm_P22.50mm_MKS4"
+		(property "Footprint" "Capacitor_THT:C_Rect_L10.0mm_W3.0mm_P7.50mm_FKS3_FKP3"
 			(at 130.81 81.28 0)
 			(effects
@@
 			)
 		)
-		(property "Value" "Fuse"
-			(at 232.41 26.67 90)
+		(property "Value" "SF-2410HI050T-2"
+			(at 232.41 29.972 90)
 			(effects
 				(font
@@
 			)
 		)
-		(property "Footprint" ""
+		(property "Footprint" "Fuse:Fuse_Littelfuse-NANO2-451_453"
 			(at 227.33 27.178 90)
 			(effects
@@
 		(on_board yes)
 		(dnp no)
-		(property "Reference" "#PWR013"
+		(property "Reference" "#PWR012"
 			(at 38.1 153.67 0)
 			(effects
@@
 			(project "01_IO-ASD-PLUS"
 				(path "/38a2da3c-ed29-422f-ab41-066ccf490e61/02316654-b7a5-4033-a293-af0194a6badf"
-					(reference "#PWR013")
+					(reference "#PWR012")
 					(unit 1)
 				)
@@
 			)
 		)
-		(property "Value" "Fuse"
-			(at 225.298 23.368 90)
+		(property "Value" "SF-2410HI050T-2"
+			(at 225.298 16.002 90)
 			(effects
 				(font
@@
 			)
 		)
-		(property "Footprint" ""
+		(property "Footprint" "Fuse:Fuse_Littelfuse-NANO2-451_453"
 			(at 227.33 29.718 90)
 			(effects
@@
 		(dnp no)
 		(property "Reference" "F1"
-			(at 115.824 81.534 90)
+			(at 122.174 75.184 90)
 			(effects
 				(font
@@
 			)
 		)
-		(property "Value" "Fuse"
-			(at 116.586 84.328 90)
+		(property "Value" "SF-2410HI050T-2"
+			(at 116.84 73.152 90)
 			(effects
 				(font
 					(size 1.27 1.27)
 				)
+				(hide yes)
 			)
 		)
-		(property "Footprint" ""
+		(property "Footprint" "Fuse:Fuse_Littelfuse-NANO2-451_453"
 			(at 115.57 76.708 90)
 			(effects
@@
 		(dnp no)
 		(fields_autoplaced yes)
-		(property "Reference" "#PWR012"
+		(property "Reference" "#PWR013"
 			(at 39.37 81.28 0)
 			(effects
@@
 			(project "01_IO-ASD-PLUS"
 				(path "/38a2da3c-ed29-422f-ab41-066ccf490e61/02316654-b7a5-4033-a293-af0194a6badf"
-					(reference "#PWR012")
+					(reference "#PWR013")
 					(unit 1)
 				)
@@
 			)
 		)
-		(property "Footprint" "Capacitor_THT:C_Rect_L26.5mm_W11.5mm_P22.50mm_MKS4"
+		(property "Footprint" "Capacitor_THT:C_Rect_L10.0mm_W3.0mm_P7.50mm_FKS3_FKP3"
 			(at 127 81.28 0)
 			(effects
@@
 	)
 	(symbol
-		(lib_id "Connector:TestPoint")
-		(at 50.8 46.99 0)
-		(unit 1)
-		(exclude_from_sim no)
-		(in_bom yes)
-		(on_board yes)
-		(dnp no)
-		(property "Reference" "TP4"
-			(at 51.562 45.212 0)
-			(effects
-				(font
-					(size 1.27 1.27)
-				)
-				(justify left)
-			)
-		)
-		(property "Value" "TestPoint"
-			(at 53.34 44.9579 0)
-			(effects
-				(font
-					(size 1.27 1.27)
-				)
-				(justify left)
-				(hide yes)
-			)
-		)
-		(property "Footprint" "TestPoint:TestPoint_Loop_D1.80mm_Drill1.0mm_Beaded"
-			(at 55.88 46.99 0)
-			(effects
-				(font
-					(size 1.27 1.27)
-				)
-				(hide yes)
-			)
-		)
-		(property "Datasheet" "~"
-			(at 55.88 46.99 0)
-			(effects
-				(font
-					(size 1.27 1.27)
-				)
-				(hide yes)
-			)
-		)
-		(property "Description" "test point"
-			(at 50.8 46.99 0)
-			(effects
-				(font
-					(size 1.27 1.27)
-				)
-				(hide yes)
-			)
-		)
-		(pin "1"
-		)
-		(instances
-			(project "01_IO-ASD-PLUS"
-				(path "/38a2da3c-ed29-422f-ab41-066ccf490e61/02316654-b7a5-4033-a293-af0194a6badf"
-					(reference "TP4")
-					(unit 1)
-				)
-			)
-		)
-	)
-	(symbol
 		(lib_id "power:+24V")
 		(at 26.67 124.46 0)
@@
 		(dnp no)
 		(fields_autoplaced yes)
-		(property "Reference" "#PWR08"
+		(property "Reference" "#PWR06"
 			(at 26.67 128.27 0)
 			(effects
@@
 			(project "01_IO-ASD-PLUS"
 				(path "/38a2da3c-ed29-422f-ab41-066ccf490e61/02316654-b7a5-4033-a293-af0194a6badf"
-					(reference "#PWR08")
+					(reference "#PWR06")
 					(unit 1)
 				)
