File: FUENTES.kicad_sch (KiCad schematic)
At the start: 76 parts, among them J4 1604470000, U1 LTC3646EMSEPBF, U2 LTC3646E, U3 KF33BDT, U4 TLV70212_SOT23-5

Commit message: 21-JUL-26
Changed lines of the file:
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@@
 	(text "revisar que sean iguales en el datasheet"
 		(exclude_from_sim no)
-		(at 196.85 106.172 0)
+		(at 223.774 105.41 0)
 		(effects
 			(font
-				(size 1.27 1.27)
+				(size 3.048 3.048)
+				(thickness 0.6096)
+				(bold yes)
+				(color 255 0 0 1)
 			)
 		)
@@
 		(effects
 			(font
-				(size 1.27 1.27)
+				(size 2.54 2.54)
+				(thickness 0.508)
+				(bold yes)
+				(color 255 0 255 1)
 			)
 		)

Commit message: 24/07/2026
Other:
- note added: "REVISAR, si se va a usar o no"
Changed lines of the file:
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@@
 	(text "revisar que sean iguales en el datasheet"
 		(exclude_from_sim no)
-		(at 223.774 105.41 0)
+		(at 226.568 115.316 0)
 		(effects
 			(font
@@
 		(effects
 			(font
+				(size 2.54 2.54)
+				(thickness 0.508)
+				(bold yes)
+				(color 255 0 255 1)
+			)
+		)
+	)
+	(text "REVISAR, si se va a usar o no\n"
+		(exclude_from_sim no)
+		(at 279.654 41.148 0)
+		(effects
+			(font
