File: Led_ctrl.kicad_sch (KiCad schematic)
At the start: 15 parts, among them U30 TLV2371DBV

Commit message: 22 mayo 26 actualizacion
se actualizo la PCB para la rama laptop Antigua
Parts:
- renumbered D35 to D40, R218 to R270, R216 to R271, R217 to R272, R227 to R273, R228 to R274, R223 to R275, R220 to R276, R219 to R277, R225 to R278, R224 to R279, R221 to R280, R222 to R281, R226 to R282, U30 to U39
Changed lines of the file:
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@@
 		(on_board yes)
 		(dnp no)
-		(property "Reference" "R218"
+		(property "Reference" "R270"
 			(at 66.548 65.278 90)
 			(effects
@@
 			(project "01_IO-ASD-PLUS"
 				(path "/38a2da3c-ed29-422f-ab41-066ccf490e61/b83e4991-9806-4c27-8269-31bebca0e905/3e235441-da5f-4b2f-962b-b7e4c230eeed"
-					(reference "R218")
+					(reference "R270")
 					(unit 1)
 				)
@@
 		(on_board yes)
 		(dnp no)
-		(property "Reference" "R219"
+		(property "Reference" "R277"
 			(at 112.268 79.502 90)
 			(effects
@@
 			(project "01_IO-ASD-PLUS"
 				(path "/38a2da3c-ed29-422f-ab41-066ccf490e61/b83e4991-9806-4c27-8269-31bebca0e905/3e235441-da5f-4b2f-962b-b7e4c230eeed"
-					(reference "R219")
+					(reference "R277")
 					(unit 1)
 				)
@@
 		(on_board yes)
 		(dnp no)
-		(property "Reference" "#PWR0309"
+		(property "Reference" "#PWR0434"
 			(at 129.54 90.17 0)
 			(effects
@@
 			(project "01_IO-ASD-PLUS"
 				(path "/38a2da3c-ed29-422f-ab41-066ccf490e61/b83e4991-9806-4c27-8269-31bebca0e905/3e235441-da5f-4b2f-962b-b7e4c230eeed"
-					(reference "#PWR0309")
+					(reference "#PWR0434")
 					(unit 1)
 				)
@@
 		(on_board yes)
 		(dnp no)
-		(property "Reference" "R225"
+		(property "Reference" "R278"
 			(at 116.332 89.408 90)
 			(effects
@@
 			(project "01_IO-ASD-PLUS"
 				(path "/38a2da3c-ed29-422f-ab41-066ccf490e61/b83e4991-9806-4c27-8269-31bebca0e905/3e235441-da5f-4b2f-962b-b7e4c230eeed"
-					(reference "R225")
+					(reference "R278")
 					(unit 1)
 				)
@@
 		(on_board yes)
 		(dnp no)
-		(property "Reference" "R217"
+		(property "Reference" "R272"
 			(at 94.742 41.148 90)
 			(effects
@@
 			(project "01_IO-ASD-PLUS"
 				(path "/38a2da3c-ed29-422f-ab41-066ccf490e61/b83e4991-9806-4c27-8269-31bebca0e905/3e235441-da5f-4b2f-962b-b7e4c230eeed"
-					(reference "R217")
+					(reference "R272")
 					(unit 1)
 				)
@@
 		(on_board yes)
 		(dnp no)
-		(property "Reference" "#PWR0301"
+		(property "Reference" "#PWR0431"
 			(at 92.71 38.1 0)
 			(effects
@@
 			(project "01_IO-ASD-PLUS"
 				(path "/38a2da3c-ed29-422f-ab41-066ccf490e61/b83e4991-9806-4c27-8269-31bebca0e905/3e235441-da5f-4b2f-962b-b7e4c230eeed"
-					(reference "#PWR0301")
+					(reference "#PWR0431")
 					(unit 1)
 				)
@@
 		(on_board yes)
 		(dnp no)
-		(property "Reference" "R227"
+		(property "Reference" "R273"
 			(at 110.998 98.298 90)
 			(effects
@@
 			(project "01_IO-ASD-PLUS"
 				(path "/38a2da3c-ed29-422f-ab41-066ccf490e61/b83e4991-9806-4c27-8269-31bebca0e905/3e235441-da5f-4b2f-962b-b7e4c230eeed"
-					(reference "R227")
+					(reference "R273")
 					(unit 1)
 				)
@@
 		(on_board yes)
 		(dnp no)
-		(property "Reference" "R224"
+		(property "Reference" "R279"
 			(at 131.572 48.768 90)
 			(effects
@@
 			(project "01_IO-ASD-PLUS"
 				(path "/38a2da3c-ed29-422f-ab41-066ccf490e61/b83e4991-9806-4c27-8269-31bebca0e905/3e235441-da5f-4b2f-962b-b7e4c230eeed"
-					(reference "R224")
+					(reference "R279")
 					(unit 1)
 				)
@@
 		(on_board yes)
 		(dnp no)
-		(property "Reference" "R222"
+		(property "Reference" "R281"
 			(at 127.508 69.342 90)
 			(effects
@@
 			(project "01_IO-ASD-PLUS"
 				(path "/38a2da3c-ed29-422f-ab41-066ccf490e61/b83e4991-9806-4c27-8269-31bebca0e905/3e235441-da5f-4b2f-962b-b7e4c230eeed"
-					(reference "R222")
+					(reference "R281")
 					(unit 1)
 				)
@@
 		(on_board yes)
 		(dnp no)
-		(property "Reference" "#PWR0303"
+		(property "Reference" "#PWR0430"
 			(at 90.17 85.09 0)
 			(effects
@@
 			(project "01_IO-ASD-PLUS"
 				(path "/38a2da3c-ed29-422f-ab41-066ccf490e61/b83e4991-9806-4c27-8269-31bebca0e905/3e235441-da5f-4b2f-962b-b7e4c230eeed"
-					(reference "#PWR0303")
+					(reference "#PWR0430")
 					(unit 1)
 				)
@@
 		(on_board yes)
 		(dnp no)
-		(property "Reference" "R228"
+		(property "Reference" "R274"
 			(at 110.998 105.918 90)
 			(effects
@@
 			(project "01_IO-ASD-PLUS"
 				(path "/38a2da3c-ed29-422f-ab41-066ccf490e61/b83e4991-9806-4c27-8269-31bebca0e905/3e235441-da5f-4b2f-962b-b7e4c230eeed"
-					(reference "R228")
+					(reference "R274")
 					(unit 1)
 				)
@@
 		(on_board yes)
 		(dnp no)
-		(property "Reference" "R220"
+		(property "Reference" "R276"
 			(at 116.332 69.088 90)
 			(effects
@@
 			(project "01_IO-ASD-PLUS"
 				(path "/38a2da3c-ed29-422f-ab41-066ccf490e61/b83e4991-9806-4c27-8269-31bebca0e905/3e235441-da5f-4b2f-962b-b7e4c230eeed"
-					(reference "R220")
+					(reference "R276")
 					(unit 1)
 				)
@@
 		(on_board yes)
 		(dnp no)
-		(property "Reference" "R223"
+		(property "Reference" "R275"
 			(at 116.332 58.928 90)
 			(effects
@@
 			(project "01_IO-ASD-PLUS"
 				(path "/38a2da3c-ed29-422f-ab41-066ccf490e61/b83e4991-9806-4c27-8269-31bebca0e905/3e235441-da5f-4b2f-962b-b7e4c230eeed"
-					(reference "R223")
+					(reference "R275")
 					(unit 1)
 				)
@@
 		(on_board yes)
 		(dnp no)
-		(property "Reference" "#PWR0304"
+		(property "Reference" "#PWR0429"
 			(at 44.45 78.74 0)
 			(effects
@@
 			(project "01_IO-ASD-PLUS"
 				(path "/38a2da3c-ed29-422f-ab41-066ccf490e61/b83e4991-9806-4c27-8269-31bebca0e905/3e235441-da5f-4b2f-962b-b7e4c230eeed"
-					(reference "#PWR0304")
+					(reference "#PWR0429")
 					(unit 1)
 				)
@@
 		(on_board yes)
 		(dnp no)
-		(property "Reference" "D35"
+		(property "Reference" "D40"
 			(at 98.806 45.212 0)
 			(effects
@@
 			(project ""
 				(path "/38a2da3c-ed29-422f-ab41-066ccf490e61/b83e4991-9806-4c27-8269-31bebca0e905/3e235441-da5f-4b2f-962b-b7e4c230eeed"
-					(reference "D35")
+					(reference "D40")
 					(unit 1)
 				)
@@
 		(on_board yes)
 		(dnp no)
-		(property "Reference" "R226"
+		(property "Reference" "R282"
 			(at 131.572 79.248 90)
 			(effects
@@
 			(project "01_IO-ASD-PLUS"
 				(path "/38a2da3c-ed29-422f-ab41-066ccf490e61/b83e4991-9806-4c27-8269-31bebca0e905/3e235441-da5f-4b2f-962b-b7e4c230eeed"
-					(reference "R226")
+					(reference "R282")
 					(unit 1)
 				)
@@
 		(on_board yes)
 		(dnp no)
-		(property "Reference" "#PWR0302"
+		(property "Reference" "#PWR0432"
 			(at 105.41 57.15 0)
 			(effects
@@
 			(project "01_IO-ASD-PLUS"
 				(path "/38a2da3c-ed29-422f-ab41-066ccf490e61/b83e4991-9806-4c27-8269-31bebca0e905/3e235441-da5f-4b2f-962b-b7e4c230eeed"
-					(reference "#PWR0302")
+					(reference "#PWR0432")
 					(unit 1)
 				)
@@
 		(on_board yes)
 		(dnp no)
-		(property "Reference" "U30"
+		(property "Reference" "U39"
 			(at 74.93 60.8898 0)
 			(effects
@@
 			(project ""
 				(path "/38a2da3c-ed29-422f-ab41-066ccf490e61/b83e4991-9806-4c27-8269-31bebca0e905/3e235441-da5f-4b2f-962b-b7e4c230eeed"
-					(reference "U30")
+					(reference "U39")
 					(unit 1)
 				)
@@
 		(on_board yes)
 		(dnp no)
-		(property "Reference" "R216"
+		(property "Reference" "R271"
 			(at 88.392 85.852 90)
 			(effects
@@
 			(project "01_IO-ASD-PLUS"
 				(path "/38a2da3c-ed29-422f-ab41-066ccf490e61/b83e4991-9806-4c27-8269-31bebca0e905/3e235441-da5f-4b2f-962b-b7e4c230eeed"
-					(reference "R216")
+					(reference "R271")
 					(unit 1)
 				)
@@
 		(on_board yes)
 		(dnp no)
-		(property "Reference" "#PWR0305"
+		(property "Reference" "#PWR0433"
 			(at 114.3 100.33 0)
 			(effects
@@
 			(project "01_IO-ASD-PLUS"
 				(path "/38a2da3c-ed29-422f-ab41-066ccf490e61/b83e4991-9806-4c27-8269-31bebca0e905/3e235441-da5f-4b2f-962b-b7e4c230eeed"
-					(reference "#PWR0305")
+					(reference "#PWR0433")
 					(unit 1)
 				)
@@
 		(on_board yes)
 		(dnp no)
-		(property "Reference" "R221"
+		(property "Reference" "R280"
 			(at 131.572 58.928 90)
 			(effects
@@
 			(project "01_IO-ASD-PLUS"
 				(path "/38a2da3c-ed29-422f-ab41-066ccf490e61/b83e4991-9806-4c27-8269-31bebca0e905/3e235441-da5f-4b2f-962b-b7e4c230eeed"
-					(reference "R221")
-					(unit 1)
-				)
+					(reference "R280")
+					(unit 1)
+				)

Commit message: 05/06/26
Parts:
- renumbered D40 to D30, R270 to R197, R271 to R198, R272 to R199, R273 to R200, R274 to R201, R275 to R202, R276 to R203, R277 to R204, R278 to R205, R279 to R206, R280 to R207, R281 to R208, R282 to R209, U39 to U41
Changed lines of the file:
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@@
 		(on_board yes)
 		(dnp no)
-		(property "Reference" "R270"
+		(property "Reference" "R197"
 			(at 66.548 65.278 90)
 			(effects
@@
 			(project "01_IO-ASD-PLUS"
 				(path "/38a2da3c-ed29-422f-ab41-066ccf490e61/b83e4991-9806-4c27-8269-31bebca0e905/3e235441-da5f-4b2f-962b-b7e4c230eeed"
-					(reference "R270")
+					(reference "R197")
 					(unit 1)
 				)
@@
 		(on_board yes)
 		(dnp no)
-		(property "Reference" "R277"
+		(property "Reference" "R204"
 			(at 112.268 79.502 90)
 			(effects
@@
 			(project "01_IO-ASD-PLUS"
 				(path "/38a2da3c-ed29-422f-ab41-066ccf490e61/b83e4991-9806-4c27-8269-31bebca0e905/3e235441-da5f-4b2f-962b-b7e4c230eeed"
-					(reference "R277")
+					(reference "R204")
 					(unit 1)
 				)
@@
 		(on_board yes)
 		(dnp no)
-		(property "Reference" "#PWR0434"
+		(property "Reference" "#PWR0319"
 			(at 129.54 90.17 0)
 			(effects
@@
 			(project "01_IO-ASD-PLUS"
 				(path "/38a2da3c-ed29-422f-ab41-066ccf490e61/b83e4991-9806-4c27-8269-31bebca0e905/3e235441-da5f-4b2f-962b-b7e4c230eeed"
-					(reference "#PWR0434")
+					(reference "#PWR0319")
 					(unit 1)
 				)
@@
 		(on_board yes)
 		(dnp no)
-		(property "Reference" "R278"
+		(property "Reference" "R205"
 			(at 116.332 89.408 90)
 			(effects
@@
 			(project "01_IO-ASD-PLUS"
 				(path "/38a2da3c-ed29-422f-ab41-066ccf490e61/b83e4991-9806-4c27-8269-31bebca0e905/3e235441-da5f-4b2f-962b-b7e4c230eeed"
-					(reference "R278")
+					(reference "R205")
 					(unit 1)
 				)
@@
 		(on_board yes)
 		(dnp no)
-		(property "Reference" "R272"
+		(property "Reference" "R199"
 			(at 94.742 41.148 90)
 			(effects
@@
 			(project "01_IO-ASD-PLUS"
 				(path "/38a2da3c-ed29-422f-ab41-066ccf490e61/b83e4991-9806-4c27-8269-31bebca0e905/3e235441-da5f-4b2f-962b-b7e4c230eeed"
-					(reference "R272")
+					(reference "R199")
 					(unit 1)
 				)
@@
 		(on_board yes)
 		(dnp no)
-		(property "Reference" "#PWR0431"
+		(property "Reference" "#PWR0316"
 			(at 92.71 38.1 0)
 			(effects
@@
 			(project "01_IO-ASD-PLUS"
 				(path "/38a2da3c-ed29-422f-ab41-066ccf490e61/b83e4991-9806-4c27-8269-31bebca0e905/3e235441-da5f-4b2f-962b-b7e4c230eeed"
-					(reference "#PWR0431")
+					(reference "#PWR0316")
 					(unit 1)
 				)
@@
 		(on_board yes)
 		(dnp no)
-		(property "Reference" "R273"
+		(property "Reference" "R200"
 			(at 110.998 98.298 90)
 			(effects
@@
 			(project "01_IO-ASD-PLUS"
 				(path "/38a2da3c-ed29-422f-ab41-066ccf490e61/b83e4991-9806-4c27-8269-31bebca0e905/3e235441-da5f-4b2f-962b-b7e4c230eeed"
-					(reference "R273")
+					(reference "R200")
 					(unit 1)
 				)
@@
 		(on_board yes)
 		(dnp no)
-		(property "Reference" "R279"
+		(property "Reference" "R206"
 			(at 131.572 48.768 90)
 			(effects
@@
 			(project "01_IO-ASD-PLUS"
 				(path "/38a2da3c-ed29-422f-ab41-066ccf490e61/b83e4991-9806-4c27-8269-31bebca0e905/3e235441-da5f-4b2f-962b-b7e4c230eeed"
-					(reference "R279")
+					(reference "R206")
 					(unit 1)
 				)
@@
 		(on_board yes)
 		(dnp no)
-		(property "Reference" "R281"
+		(property "Reference" "R208"
 			(at 127.508 69.342 90)
 			(effects
@@
 			(project "01_IO-ASD-PLUS"
 				(path "/38a2da3c-ed29-422f-ab41-066ccf490e61/b83e4991-9806-4c27-8269-31bebca0e905/3e235441-da5f-4b2f-962b-b7e4c230eeed"
-					(reference "R281")
+					(reference "R208")
 					(unit 1)
 				)
@@
 		(on_board yes)
 		(dnp no)
-		(property "Reference" "#PWR0430"
+		(property "Reference" "#PWR0315"
 			(at 90.17 85.09 0)
 			(effects
@@
 			(project "01_IO-ASD-PLUS"
 				(path "/38a2da3c-ed29-422f-ab41-066ccf490e61/b83e4991-9806-4c27-8269-31bebca0e905/3e235441-da5f-4b2f-962b-b7e4c230eeed"
-					(reference "#PWR0430")
+					(reference "#PWR0315")
 					(unit 1)
 				)
@@
 		(on_board yes)
 		(dnp no)
-		(property "Reference" "R274"
+		(property "Reference" "R201"
 			(at 110.998 105.918 90)
 			(effects
@@
 			(project "01_IO-ASD-PLUS"
 				(path "/38a2da3c-ed29-422f-ab41-066ccf490e61/b83e4991-9806-4c27-8269-31bebca0e905/3e235441-da5f-4b2f-962b-b7e4c230eeed"
-					(reference "R274")
+					(reference "R201")
 					(unit 1)
 				)
@@
 		(on_board yes)
 		(dnp no)
-		(property "Reference" "R276"
+		(property "Reference" "R203"
 			(at 116.332 69.088 90)
 			(effects
@@
 			(project "01_IO-ASD-PLUS"
 				(path "/38a2da3c-ed29-422f-ab41-066ccf490e61/b83e4991-9806-4c27-8269-31bebca0e905/3e235441-da5f-4b2f-962b-b7e4c230eeed"
-					(reference "R276")
+					(reference "R203")
 					(unit 1)
 				)
@@
 		(on_board yes)
 		(dnp no)
-		(property "Reference" "R275"
+		(property "Reference" "R202"
 			(at 116.332 58.928 90)
 			(effects
@@
 			(project "01_IO-ASD-PLUS"
 				(path "/38a2da3c-ed29-422f-ab41-066ccf490e61/b83e4991-9806-4c27-8269-31bebca0e905/3e235441-da5f-4b2f-962b-b7e4c230eeed"
-					(reference "R275")
+					(reference "R202")
 					(unit 1)
 				)
@@
 		(on_board yes)
 		(dnp no)
-		(property "Reference" "#PWR0429"
+		(property "Reference" "#PWR0314"
 			(at 44.45 78.74 0)
 			(effects
@@
 			(project "01_IO-ASD-PLUS"
 				(path "/38a2da3c-ed29-422f-ab41-066ccf490e61/b83e4991-9806-4c27-8269-31bebca0e905/3e235441-da5f-4b2f-962b-b7e4c230eeed"
-					(reference "#PWR0429")
+					(reference "#PWR0314")
 					(unit 1)
 				)
@@
 		(on_board yes)
 		(dnp no)
-		(property "Reference" "D40"
+		(property "Reference" "D30"
 			(at 98.806 45.212 0)
 			(effects
@@
 			(project ""
 				(path "/38a2da3c-ed29-422f-ab41-066ccf490e61/b83e4991-9806-4c27-8269-31bebca0e905/3e235441-da5f-4b2f-962b-b7e4c230eeed"
-					(reference "D40")
+					(reference "D30")
 					(unit 1)
 				)
@@
 		(on_board yes)
 		(dnp no)
-		(property "Reference" "R282"
+		(property "Reference" "R209"
 			(at 131.572 79.248 90)
 			(effects
@@
 			(project "01_IO-ASD-PLUS"
 				(path "/38a2da3c-ed29-422f-ab41-066ccf490e61/b83e4991-9806-4c27-8269-31bebca0e905/3e235441-da5f-4b2f-962b-b7e4c230eeed"
-					(reference "R282")
+					(reference "R209")
 					(unit 1)
 				)
@@
 		(on_board yes)
 		(dnp no)
-		(property "Reference" "#PWR0432"
+		(property "Reference" "#PWR0317"
 			(at 105.41 57.15 0)
 			(effects
@@
 			(project "01_IO-ASD-PLUS"
 				(path "/38a2da3c-ed29-422f-ab41-066ccf490e61/b83e4991-9806-4c27-8269-31bebca0e905/3e235441-da5f-4b2f-962b-b7e4c230eeed"
-					(reference "#PWR0432")
+					(reference "#PWR0317")
 					(unit 1)
 				)
@@
 		(on_board yes)
 		(dnp no)
-		(property "Reference" "U39"
+		(property "Reference" "U41"
 			(at 74.93 60.8898 0)
 			(effects
@@
 			(project ""
 				(path "/38a2da3c-ed29-422f-ab41-066ccf490e61/b83e4991-9806-4c27-8269-31bebca0e905/3e235441-da5f-4b2f-962b-b7e4c230eeed"
-					(reference "U39")
+					(reference "U41")
 					(unit 1)
 				)
@@
 		(on_board yes)
 		(dnp no)
-		(property "Reference" "R271"
+		(property "Reference" "R198"
 			(at 88.392 85.852 90)
 			(effects
@@
 			(project "01_IO-ASD-PLUS"
 				(path "/38a2da3c-ed29-422f-ab41-066ccf490e61/b83e4991-9806-4c27-8269-31bebca0e905/3e235441-da5f-4b2f-962b-b7e4c230eeed"
-					(reference "R271")
+					(reference "R198")
 					(unit 1)
 				)
@@
 		(on_board yes)
 		(dnp no)
-		(property "Reference" "#PWR0433"
+		(property "Reference" "#PWR0318"
 			(at 114.3 100.33 0)
 			(effects
@@
 			(project "01_IO-ASD-PLUS"
 				(path "/38a2da3c-ed29-422f-ab41-066ccf490e61/b83e4991-9806-4c27-8269-31bebca0e905/3e235441-da5f-4b2f-962b-b7e4c230eeed"
-					(reference "#PWR0433")
+					(reference "#PWR0318")
 					(unit 1)
 				)
@@
 		(on_board yes)
 		(dnp no)
-		(property "Reference" "R280"
+		(property "Reference" "R207"
 			(at 131.572 58.928 90)
 			(effects
@@
 			(project "01_IO-ASD-PLUS"
 				(path "/38a2da3c-ed29-422f-ab41-066ccf490e61/b83e4991-9806-4c27-8269-31bebca0e905/3e235441-da5f-4b2f-962b-b7e4c230eeed"
-					(reference "R280")
-					(unit 1)
-				)
+					(reference "R207")
+					(unit 1)
+				)
