File: Led_ctrl.kicad_sch (KiCad schematic)
At the start: 15 parts, among them U41 TLV2371DBV

Commit message: 13-jul-26_6pm
Parts:
- renumbered U41 to U38
Changed lines of the file:
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@@
 		(on_board yes)
 		(dnp no)
-		(property "Reference" "#PWR0319"
+		(property "Reference" "#PWR0418"
 			(at 129.54 90.17 0)
 			(effects
@@
 			(project "01_IO-ASD-PLUS"
 				(path "/38a2da3c-ed29-422f-ab41-066ccf490e61/b83e4991-9806-4c27-8269-31bebca0e905/3e235441-da5f-4b2f-962b-b7e4c230eeed"
-					(reference "#PWR0319")
+					(reference "#PWR0418")
 					(unit 1)
 				)
@@
 		(on_board yes)
 		(dnp no)
-		(property "Reference" "#PWR0316"
+		(property "Reference" "#PWR0413"
 			(at 92.71 38.1 0)
 			(effects
@@
 			(project "01_IO-ASD-PLUS"
 				(path "/38a2da3c-ed29-422f-ab41-066ccf490e61/b83e4991-9806-4c27-8269-31bebca0e905/3e235441-da5f-4b2f-962b-b7e4c230eeed"
-					(reference "#PWR0316")
+					(reference "#PWR0413")
 					(unit 1)
 				)
@@
 		(on_board yes)
 		(dnp no)
-		(property "Reference" "#PWR0315"
+		(property "Reference" "#PWR0415"
 			(at 90.17 85.09 0)
 			(effects
@@
 			(project "01_IO-ASD-PLUS"
 				(path "/38a2da3c-ed29-422f-ab41-066ccf490e61/b83e4991-9806-4c27-8269-31bebca0e905/3e235441-da5f-4b2f-962b-b7e4c230eeed"
-					(reference "#PWR0315")
+					(reference "#PWR0415")
 					(unit 1)
 				)
@@
 		(on_board yes)
 		(dnp no)
-		(property "Reference" "#PWR0314"
+		(property "Reference" "#PWR0416"
 			(at 44.45 78.74 0)
 			(effects
@@
 			(project "01_IO-ASD-PLUS"
 				(path "/38a2da3c-ed29-422f-ab41-066ccf490e61/b83e4991-9806-4c27-8269-31bebca0e905/3e235441-da5f-4b2f-962b-b7e4c230eeed"
-					(reference "#PWR0314")
+					(reference "#PWR0416")
 					(unit 1)
 				)
@@
 		(on_board yes)
 		(dnp no)
-		(property "Reference" "#PWR0317"
+		(property "Reference" "#PWR0414"
 			(at 105.41 57.15 0)
 			(effects
@@
 			(project "01_IO-ASD-PLUS"
 				(path "/38a2da3c-ed29-422f-ab41-066ccf490e61/b83e4991-9806-4c27-8269-31bebca0e905/3e235441-da5f-4b2f-962b-b7e4c230eeed"
-					(reference "#PWR0317")
+					(reference "#PWR0414")
 					(unit 1)
 				)
@@
 		(on_board yes)
 		(dnp no)
-		(property "Reference" "U41"
+		(property "Reference" "U38"
 			(at 74.93 60.8898 0)
 			(effects
@@
 			(project ""
 				(path "/38a2da3c-ed29-422f-ab41-066ccf490e61/b83e4991-9806-4c27-8269-31bebca0e905/3e235441-da5f-4b2f-962b-b7e4c230eeed"
-					(reference "U41")
+					(reference "U38")
 					(unit 1)
 				)
@@
 		(on_board yes)
 		(dnp no)
-		(property "Reference" "#PWR0318"
+		(property "Reference" "#PWR0417"
 			(at 114.3 100.33 0)
 			(effects
@@
 			(project "01_IO-ASD-PLUS"
 				(path "/38a2da3c-ed29-422f-ab41-066ccf490e61/b83e4991-9806-4c27-8269-31bebca0e905/3e235441-da5f-4b2f-962b-b7e4c230eeed"
-					(reference "#PWR0318")
-					(unit 1)
-				)
+					(reference "#PWR0417")
+					(unit 1)
+				)
