File: Port_Expansor.kicad_sch (KiCad schematic)
At the start: 19 parts, among them IC1 ILD206T, IC10 ILD206T, IC2 ILD206T, IC3 ILD206T, IC4 ILD206T, IC5 ILD206T, IC6 ILD206T, IC7 ILD206T, IC8 ILD206T, IC9 ILD206T, J4 1147330000, U2 5-1415390-1, U24 MCP23S17_SS, U3 5-1415390-1

Commit message: 15-mayo-26
15 mayo 26
Parts:
- added R231, R232, R233: 0R, Resistor_SMD:R_0603_1608Metric, symbol Device:R_US
Connections:
- net +3.3v: now also R232.1, R233.1; no longer U24.15 (A0), U24.16 (A1)
- net GND: now also R231.2
- new net: R233.2, U24.16 (A1)
- new net: R231.1, R232.2, U24.15 (A0)
Other:
- note added: "VER SI LO PONERMOS AL RESET MAESTRO"

Commit message: 22 mayo 26 actualizacion
se actualizo la PCB para la rama laptop Antigua
Parts:
- renumbered C76 to C160, C77 to C161, IC1 to IC20, IC2 to IC21, IC3 to IC22, IC4 to IC23, IC5 to IC24, IC6 to IC25, IC7 to IC26, IC8 to IC27, IC9 to IC28, IC10 to IC29, J4 to J17, R133 to R251, R233 to R252, R232 to R253, R231 to R254, U2 to U32, U24 to U33, U2 to U34, U3 to U35
Changed lines of the file:
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@@
 		(on_board no)
 		(dnp yes)
-		(property "Reference" "IC7"
+		(property "Reference" "IC26"
 			(at 119.38 -95.25 0)
 			(effects
@@
 			(project "01_IO-ASD-PLUS"
 				(path "/38a2da3c-ed29-422f-ab41-066ccf490e61/92659552-e3e9-4659-b9ad-ce458c1d5072"
-					(reference "IC7")
+					(reference "IC26")
 					(unit 1)
 				)
@@
 		(on_board no)
 		(dnp yes)
-		(property "Reference" "#PWR03"
+		(property "Reference" "#PWR0396"
 			(at 102.87 -109.22 0)
 			(effects
@@
 			(project "01_IO-ASD-PLUS"
 				(path "/38a2da3c-ed29-422f-ab41-066ccf490e61/92659552-e3e9-4659-b9ad-ce458c1d5072"
-					(reference "#PWR03")
+					(reference "#PWR0396")
 					(unit 1)
 				)
@@
 		(dnp yes)
 		(fields_autoplaced yes)
-		(property "Reference" "J4"
+		(property "Reference" "J17"
 			(at 151.13 -97.7901 0)
 			(effects
@@
 			(project "01_IO-ASD-PLUS"
 				(path "/38a2da3c-ed29-422f-ab41-066ccf490e61/92659552-e3e9-4659-b9ad-ce458c1d5072"
-					(reference "J4")
+					(reference "J17")
 					(unit 1)
 				)
@@
 		(dnp yes)
 		(fields_autoplaced yes)
-		(property "Reference" "IC10"
+		(property "Reference" "IC29"
 			(at 173.99 -29.21 0)
 			(effects
@@
 			(project "01_IO-ASD-PLUS"
 				(path "/38a2da3c-ed29-422f-ab41-066ccf490e61/92659552-e3e9-4659-b9ad-ce458c1d5072"
-					(reference "IC10")
+					(reference "IC29")
 					(unit 1)
 				)
@@
 		(on_board yes)
 		(dnp no)
-		(property "Reference" "#PWR0201"
+		(property "Reference" "#PWR0401"
 			(at 144.78 62.23 0)
 			(effects
@@
 			(project "01_IO-ASD-PLUS"
 				(path "/38a2da3c-ed29-422f-ab41-066ccf490e61/92659552-e3e9-4659-b9ad-ce458c1d5072"
-					(reference "#PWR0201")
+					(reference "#PWR0401")
 					(unit 1)
 				)
@@
 		(on_board no)
 		(dnp yes)
-		(property "Reference" "IC6"
+		(property "Reference" "IC25"
 			(at 119.38 -118.11 0)
 			(effects
@@
 			(project "01_IO-ASD-PLUS"
 				(path "/38a2da3c-ed29-422f-ab41-066ccf490e61/92659552-e3e9-4659-b9ad-ce458c1d5072"
-					(reference "IC6")
+					(reference "IC25")
 					(unit 1)
 				)
@@
 		(dnp yes)
 		(fields_autoplaced yes)
-		(property "Reference" "IC2"
+		(property "Reference" "IC21"
 			(at 106.68 -26.67 0)
 			(effects
@@
 			(project "01_IO-ASD-PLUS"
 				(path "/38a2da3c-ed29-422f-ab41-066ccf490e61/92659552-e3e9-4659-b9ad-ce458c1d5072"
-					(reference "IC2")
+					(reference "IC21")
 					(unit 1)
 				)
@@
 		(on_board yes)
 		(dnp no)
-		(property "Reference" "#PWR0316"
+		(property "Reference" "#PWR0399"
 			(at 125.73 128.27 0)
 			(effects
@@
 			(project "01_IO-ASD-PLUS"
 				(path "/38a2da3c-ed29-422f-ab41-066ccf490e61/92659552-e3e9-4659-b9ad-ce458c1d5072"
-					(reference "#PWR0316")
+					(reference "#PWR0399")
 					(unit 1)
 				)
@@
 		(on_board yes)
 		(dnp no)
-		(property "Reference" "R233"
+		(property "Reference" "R252"
 			(at 115.57 113.538 0)
 			(effects
@@
 			(project "01_IO-ASD-PLUS"
 				(path "/38a2da3c-ed29-422f-ab41-066ccf490e61/92659552-e3e9-4659-b9ad-ce458c1d5072"
-					(reference "R233")
+					(reference "R252")
 					(unit 1)
 				)
@@
 		(dnp yes)
 		(fields_autoplaced yes)
-		(property "Reference" "U2"
+		(property "Reference" "U34"
 			(at 165.1 -137.16 0)
 			(effects
@@
 			(project "01_IO-ASD-PLUS"
 				(path "/38a2da3c-ed29-422f-ab41-066ccf490e61/92659552-e3e9-4659-b9ad-ce458c1d5072"
-					(reference "U2")
+					(reference "U34")
 					(unit 1)
 				)
@@
 		(on_board yes)
 		(dnp yes)
-		(property "Reference" "R231"
+		(property "Reference" "R254"
 			(at 121.666 118.364 0)
 			(effects
@@
 			(project "01_IO-ASD-PLUS"
 				(path "/38a2da3c-ed29-422f-ab41-066ccf490e61/92659552-e3e9-4659-b9ad-ce458c1d5072"
-					(reference "R231")
+					(reference "R254")
 					(unit 1)
 				)
@@
 		(dnp yes)
 		(fields_autoplaced yes)
-		(property "Reference" "IC9"
+		(property "Reference" "IC28"
 			(at 154.94 -54.61 0)
 			(effects
@@
 			(project "01_IO-ASD-PLUS"
 				(path "/38a2da3c-ed29-422f-ab41-066ccf490e61/92659552-e3e9-4659-b9ad-ce458c1d5072"
-					(reference "IC9")
+					(reference "IC28")
 					(unit 1)
 				)
@@
 		(on_board yes)
 		(dnp no)
-		(property "Reference" "R133"
+		(property "Reference" "R251"
 			(at 112.522 96.012 90)
 			(effects
@@
 			(project "01_IO-ASD-PLUS"
 				(path "/38a2da3c-ed29-422f-ab41-066ccf490e61/92659552-e3e9-4659-b9ad-ce458c1d5072"
-					(reference "R133")
+					(reference "R251")
 					(unit 1)
 				)
@@
 		(dnp yes)
 		(fields_autoplaced yes)
-		(property "Reference" "IC8"
+		(property "Reference" "IC27"
 			(at 144.78 -78.74 0)
 			(effects
@@
 			(project "01_IO-ASD-PLUS"
 				(path "/38a2da3c-ed29-422f-ab41-066ccf490e61/92659552-e3e9-4659-b9ad-ce458c1d5072"
-					(reference "IC8")
+					(reference "IC27")
 					(unit 1)
 				)
@@
 		(dnp yes)
 		(fields_autoplaced yes)
-		(property "Reference" "U3"
+		(property "Reference" "U35"
 			(at 168.91 -113.03 0)
 			(effects
@@
 			(project "01_IO-ASD-PLUS"
 				(path "/38a2da3c-ed29-422f-ab41-066ccf490e61/92659552-e3e9-4659-b9ad-ce458c1d5072"
-					(reference "U3")
+					(reference "U35")
 					(unit 1)
 				)
@@
 		(on_board no)
 		(dnp yes)
-		(property "Reference" "U2"
+		(property "Reference" "U32"
 			(at 143.51 -143.51 0)
 			(effects
@@
 			(project "01_IO-ASD-PLUS"
 				(path "/38a2da3c-ed29-422f-ab41-066ccf490e61/92659552-e3e9-4659-b9ad-ce458c1d5072"
-					(reference "U2")
+					(reference "U32")
 					(unit 1)
 				)
@@
 		(on_board yes)
 		(dnp no)
-		(property "Reference" "C77"
+		(property "Reference" "C161"
 			(at 138.176 61.214 90)
 			(effects
@@
 			)
 		)
-		(property "Description" "COG NP0"
+		(property "Description" "Unpolarized capacitor, small symbol"
 			(at 140.208 59.436 90)
 			(effects
@@
 			(project "01_IO-ASD-PLUS"
 				(path "/38a2da3c-ed29-422f-ab41-066ccf490e61/92659552-e3e9-4659-b9ad-ce458c1d5072"
-					(reference "C77")
+					(reference "C161")
 					(unit 1)
 				)
@@
 		(dnp yes)
 		(fields_autoplaced yes)
-		(property "Reference" "IC3"
+		(property "Reference" "IC22"
 			(at 109.22 -77.47 0)
 			(effects
@@
 			(project "01_IO-ASD-PLUS"
 				(path "/38a2da3c-ed29-422f-ab41-066ccf490e61/92659552-e3e9-4659-b9ad-ce458c1d5072"
-					(reference "IC3")
+					(reference "IC22")
 					(unit 1)
 				)
@@
 		(on_board yes)
 		(dnp no)
-		(property "Reference" "#PWR0200"
+		(property "Reference" "#PWR0400"
 			(at 137.16 69.85 0)
 			(effects
@@
 			(project "01_IO-ASD-PLUS"
 				(path "/38a2da3c-ed29-422f-ab41-066ccf490e61/92659552-e3e9-4659-b9ad-ce458c1d5072"
-					(reference "#PWR0200")
+					(reference "#PWR0400")
 					(unit 1)
 				)
@@
 		(dnp no)
 		(fields_autoplaced yes)
-		(property "Reference" "U24"
+		(property "Reference" "U33"
 			(at 146.9233 63.5 0)
 			(effects
@@
 			(project "01_IO-ASD-PLUS"
 				(path "/38a2da3c-ed29-422f-ab41-066ccf490e61/92659552-e3e9-4659-b9ad-ce458c1d5072"
-					(reference "U24")
+					(reference "U33")
 					(unit 1)
 				)
@@
 		(dnp yes)
 		(fields_autoplaced yes)
-		(property "Reference" "IC5"
+		(property "Reference" "IC24"
 			(at 132.08 -29.21 0)
 			(effects
@@
 			(project "01_IO-ASD-PLUS"
 				(path "/38a2da3c-ed29-422f-ab41-066ccf490e61/92659552-e3e9-4659-b9ad-ce458c1d5072"
-					(reference "IC5")
+					(reference "IC24")
 					(unit 1)
 				)
@@
 		(dnp yes)
 		(fields_autoplaced yes)
-		(property "Reference" "IC4"
+		(property "Reference" "IC23"
 			(at 110.49 -52.07 0)
 			(effects
@@
 			(project "01_IO-ASD-PLUS"
 				(path "/38a2da3c-ed29-422f-ab41-066ccf490e61/92659552-e3e9-4659-b9ad-ce458c1d5072"
-					(reference "IC4")
+					(reference "IC23")
 					(unit 1)
 				)
@@
 		(on_board yes)
 		(dnp no)
-		(property "Reference" "C76"
+		(property "Reference" "C160"
 			(at 117.602 97.028 0)
 			(effects
@@
 			)
 		)
-		(property "Description" "COG NP0"
+		(property "Description" "Unpolarized capacitor, small symbol"
 			(at 120.396 98.552 90)
 			(effects
@@
 			(project "01_IO-ASD-PLUS"
 				(path "/38a2da3c-ed29-422f-ab41-066ccf490e61/92659552-e3e9-4659-b9ad-ce458c1d5072"
-					(reference "C76")
+					(reference "C160")
 					(unit 1)
 				)
@@
 		(on_board yes)
 		(dnp no)
-		(property "Reference" "#PWR0193"
+		(property "Reference" "#PWR0397"
 			(at 104.14 96.52 0)
 			(effects
@@
 			(project "01_IO-ASD-PLUS"
 				(path "/38a2da3c-ed29-422f-ab41-066ccf490e61/92659552-e3e9-4659-b9ad-ce458c1d5072"
-					(reference "#PWR0193")
+					(reference "#PWR0397")
 					(unit 1)
 				)
@@
 		(on_board yes)
 		(dnp no)
-		(property "Reference" "#PWR0196"
+		(property "Reference" "#PWR0398"
 			(at 123.19 110.49 0)
 			(effects
@@
 			(project "01_IO-ASD-PLUS"
 				(path "/38a2da3c-ed29-422f-ab41-066ccf490e61/92659552-e3e9-4659-b9ad-ce458c1d5072"
-					(reference "#PWR0196")
+					(reference "#PWR0398")
 					(unit 1)
 				)
@@
 		(dnp yes)
 		(fields_autoplaced yes)
-		(property "Reference" "IC1"
+		(property "Reference" "IC20"
 			(at 102.87 -143.51 0)
 			(effects
@@
 			(project "01_IO-ASD-PLUS"
 				(path "/38a2da3c-ed29-422f-ab41-066ccf490e61/92659552-e3e9-4659-b9ad-ce458c1d5072"
-					(reference "IC1")
+					(reference "IC20")
 					(unit 1)
 				)
@@
 		(on_board yes)
 		(dnp no)
-		(property "Reference" "R232"
+		(property "Reference" "R253"
 			(at 113.538 113.792 0)
 			(effects
@@
 			(project "01_IO-ASD-PLUS"
 				(path "/38a2da3c-ed29-422f-ab41-066ccf490e61/92659552-e3e9-4659-b9ad-ce458c1d5072"
-					(reference "R232")
+					(reference "R253")
 					(unit 1)
 				)
@@
 		(on_board yes)
 		(dnp no)
-		(property "Reference" "#PWR0202"
+		(property "Reference" "#PWR0402"
 			(at 144.78 127 0)
 			(effects
@@
 			(project "01_IO-ASD-PLUS"
 				(path "/38a2da3c-ed29-422f-ab41-066ccf490e61/92659552-e3e9-4659-b9ad-ce458c1d5072"
-					(reference "#PWR0202")
+					(reference "#PWR0402")
 					(unit 1)
 				)

Commit message: 05/06/26
Parts:
- removed IC20, IC21, IC22, IC23, IC24, IC25, IC26, IC27, IC28, IC29: ILD206T, SOIC:SOIC 8, symbol OPTOACOPLADORES:ILD206T
- removed J17: 1147330000, CONECTORES GRACIDA:3POS-5.08PITCH, symbol CONECTORES GRACIDA:1147330000
- removed RV5: Varistor, Varistor:RV_Disc_D12mm_W3.9mm_P7.5mm, symbol Device:Varistor
- removed U32, U34, U35: 5-1415390-1, RELAYS GRACIDA:5-1415390-1, symbol RELAYS_GRACIDA:5-1415390-1
- renumbered C160 to C115, C161 to C116, R251 to R178, R252 to R179, R253 to R180, R254 to R181, U33 to U35
