File: Port_Expansor.kicad_sch (KiCad schematic)
At the start: 7 parts, among them U35 MCP23S17_SS

Commit message: 13-jul-26_6pm
Parts:
- renumbered U35 to U34
Changed lines of the file:
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@@
 		(on_board yes)
 		(dnp no)
-		(property "Reference" "#PWR0286"
+		(property "Reference" "#PWR0383"
 			(at 144.78 62.23 0)
 			(effects
@@
 			(project "01_IO-ASD-PLUS"
 				(path "/38a2da3c-ed29-422f-ab41-066ccf490e61/92659552-e3e9-4659-b9ad-ce458c1d5072"
-					(reference "#PWR0286")
+					(reference "#PWR0383")
 					(unit 1)
 				)
@@
 		(on_board yes)
 		(dnp no)
-		(property "Reference" "#PWR0284"
+		(property "Reference" "#PWR0384"
 			(at 125.73 128.27 0)
 			(effects
@@
 			(project "01_IO-ASD-PLUS"
 				(path "/38a2da3c-ed29-422f-ab41-066ccf490e61/92659552-e3e9-4659-b9ad-ce458c1d5072"
-					(reference "#PWR0284")
+					(reference "#PWR0384")
 					(unit 1)
 				)
@@
 		(on_board yes)
 		(dnp no)
-		(property "Reference" "#PWR0285"
+		(property "Reference" "#PWR0386"
 			(at 137.16 69.85 0)
 			(effects
@@
 			(project "01_IO-ASD-PLUS"
 				(path "/38a2da3c-ed29-422f-ab41-066ccf490e61/92659552-e3e9-4659-b9ad-ce458c1d5072"
-					(reference "#PWR0285")
+					(reference "#PWR0386")
 					(unit 1)
 				)
@@
 		(dnp no)
 		(fields_autoplaced yes)
-		(property "Reference" "U35"
+		(property "Reference" "U34"
 			(at 146.9233 63.5 0)
 			(effects
@@
 			(project "01_IO-ASD-PLUS"
 				(path "/38a2da3c-ed29-422f-ab41-066ccf490e61/92659552-e3e9-4659-b9ad-ce458c1d5072"
-					(reference "U35")
+					(reference "U34")
 					(unit 1)
 				)
@@
 		(on_board yes)
 		(dnp no)
-		(property "Reference" "#PWR0282"
+		(property "Reference" "#PWR0381"
 			(at 104.14 96.52 0)
 			(effects
@@
 			(project "01_IO-ASD-PLUS"
 				(path "/38a2da3c-ed29-422f-ab41-066ccf490e61/92659552-e3e9-4659-b9ad-ce458c1d5072"
-					(reference "#PWR0282")
+					(reference "#PWR0381")
 					(unit 1)
 				)
@@
 		(on_board yes)
 		(dnp no)
-		(property "Reference" "#PWR0283"
+		(property "Reference" "#PWR0382"
 			(at 123.19 110.49 0)
 			(effects
@@
 			(project "01_IO-ASD-PLUS"
 				(path "/38a2da3c-ed29-422f-ab41-066ccf490e61/92659552-e3e9-4659-b9ad-ce458c1d5072"
-					(reference "#PWR0283")
+					(reference "#PWR0382")
 					(unit 1)
 				)
@@
 		(on_board yes)
 		(dnp no)
-		(property "Reference" "#PWR0287"
+		(property "Reference" "#PWR0385"
 			(at 144.78 127 0)
 			(effects
@@
 			(project "01_IO-ASD-PLUS"
 				(path "/38a2da3c-ed29-422f-ab41-066ccf490e61/92659552-e3e9-4659-b9ad-ce458c1d5072"
-					(reference "#PWR0287")
-					(unit 1)
-				)
+					(reference "#PWR0385")
+					(unit 1)
+				)

Commit message: 24/07/2026
Parts:
- R181: now left out of the parts list
Changed lines of the file:
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@@
 		(unit 1)
 		(exclude_from_sim no)
-		(in_bom yes)
+		(in_bom no)
 		(on_board yes)
 		(dnp yes)
