File: USB.kicad_sch (KiCad schematic)
At the start: 22 parts, among them J11 USB_Type A_ Receptacle, P1 USB_C_Plug_USB2.0, U26 TPS2024

Commit message: 14-Mayo-26
se agregaron varias sheet de esquematico crecio al 80% la parte de esquematico
Parts:
- renumbered C108 to C110, C113 to C111, C114 to C112, C112 to C113, C111 to C114, C110 to C115, D32 to D33, D33 to D34, J11 to J12, L13 to L12, L12 to L13, R151 to R152, R150 to R153, R158 to R154, R159 to R155, R157 to R156, R154 to R157, R152 to R158, R153 to R159

Commit message: 22 mayo 26 actualizacion
se actualizo la PCB para la rama laptop Antigua
Parts:
- renumbered C109 to C119, C110 to C120, C111 to C121, C112 to C122, C113 to C123, C114 to C124, C115 to C125, L12 to L15, L13 to L16, R152 to R175, R153 to R176, R154 to R177, R155 to R178, R156 to R179, R157 to R180, R158 to R181, R159 to R182, U26 to U25

Commit message: 05/06/26
Parts:
- renumbered C119 to C88, C120 to C89, C121 to C90, C122 to C91, C123 to C92, C124 to C93, C125 to C94, D33 to D23, D34 to D24, J12 to J10, L15 to L11, L16 to L12, R175 to R118, R176 to R119, R177 to R120, R178 to R121, R179 to R122, R180 to R123, R181 to R124, R182 to R125, U25 to U23
