File: USB.kicad_sch (KiCad schematic)
At the start: 22 parts, among them J10 USB_Type A_ Receptacle, P1 USB_C_Plug_USB2.0, U23 TPS2024

Commit message: 17-07-26
Parts:
- U23: footprint (none) -> SOIC:SOIC 8
Changed lines of the file:
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@@
 			)
 		)
-		(property "Footprint" ""
+		(property "Footprint" "SOIC:SOIC 8"
 			(at 59.69 40.64 0)
 			(effects

Commit message: 21-JUL-26
Parts:
- removed U23: TPS2024, SOIC:SOIC 8, symbol MICROS_DIGITAL_GSI:TPS2024
- added U23: TPS2024, Package_SO:SOIC-8_3.9x4.9mm_P1.27mm, symbol MICROS_DIGITAL_GSI_v2:TPS2024
- J10: footprint (none) -> Connector_USB:USB_A_Molex_105057_Vertical
- L11: footprint (none) -> Inductor_SMD:L_0603_1608Metric_Pad1.05x0.95mm_HandSolder
- P1: footprint (none) -> CONECTORES GRACIDA:USB4145030070C
Connections:
- net +5V: now also U23.2 (IN)
- net +VBUS_OUT: now also U23.6 (OUT)
- net GND: now also U23.1 (GND)
- net USB_Current_Status: now also U23.5 (!OC)
- net USB_Power_Switcher: now also U23.4 (!_ENABLE)
Changed lines of the file:
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@@
 	(wire
 		(pts
-			(xy 57.15 45.72) (xy 52.07 45.72)
+			(xy 52.07 45.72) (xy 57.15 45.72)
 		)
 		(stroke
@@
 			)
 		)
-		(property "Footprint" ""
+		(property "Footprint" "Inductor_SMD:L_0603_1608Metric_Pad1.05x0.95mm_HandSolder"
 			(at 163.83 102.87 0)
 			(effects
@@
 			)
 		)
-		(property "Footprint" ""
+		(property "Footprint" "CONECTORES GRACIDA:USB4145030070C"
 			(at 198.12 118.11 0)
 			(effects
@@
 			)
 		)
-		(property "Footprint" ""
+		(property "Footprint" "Connector_USB:USB_A_Molex_105057_Vertical"
 			(at 198.12 59.69 0)
 			(effects
@@
 	)
 	(symbol
-		(lib_id "MICROS_DIGITAL_GSI:TPS2024")
-		(at 59.69 40.64 0)
-		(unit 1)
-		(exclude_from_sim no)
-		(in_bom yes)
-		(on_board yes)
-		(dnp no)
-		(fields_autoplaced yes)
-		(property "Reference" "U23"
-			(at 83.82 35.56 0)
-			(effects
-				(font
-					(size 1.27 1.27)
-				)
-			)
-		)
-		(property "Value" "TPS2024"
-			(at 83.82 38.1 0)
-			(effects
-				(font
-					(size 1.27 1.27)
-				)
-			)
-		)
-		(property "Footprint" "SOIC:SOIC 8"
-			(at 59.69 40.64 0)
-			(effects
-				(font
-					(size 1.27 1.27)
-				)
-				(hide yes)
-			)
-		)
-		(property "Datasheet" ""
-			(at 59.69 40.64 0)
-			(effects
-				(font
-					(size 1.27 1.27)
-				)
-				(hide yes)
-			)
-		)
-		(property "Description" ""
-			(at 59.69 40.64 0)
-			(effects
-				(font
-					(size 1.27 1.27)
-				)
-				(hide yes)
-			)
-		)
-		(pin ""
-		)
-		(pin ""
-		)
-		(pin ""
-		)
-		(pin ""
-		)
-		(pin ""
-		)
-		(instances
-			(project ""
-				(path "/38a2da3c-ed29-422f-ab41-066ccf490e61/8d296a6f-d65d-491e-bf56-0b9d64795b89"
-					(reference "U23")
-					(unit 1)
-				)
-			)
-		)
-	)
-	(symbol
 		(lib_id "power:GNDREF")
 		(at 121.92 53.34 0)
@@
 					(unit 1)
 				)
+			)
+		)
+	)
+	(symbol
+		(lib_id "MICROS_DIGITAL_GSI_v2:TPS2024")
+		(at 59.69 40.64 0)
+		(unit 1)
+		(exclude_from_sim no)
+		(in_bom yes)
+		(on_board yes)
+		(dnp no)
+		(fields_autoplaced yes)
+		(property "Reference" "U23"
+			(at 83.82 35.56 0)
+			(effects
+				(font
+					(size 1.27 1.27)
+				)
+			)
+		)
+		(property "Value" "TPS2024"
+			(at 83.82 38.1 0)
+			(effects
+				(font
+					(size 1.27 1.27)
+				)
+			)
+		)
+		(property "Footprint" "Package_SO:SOIC-8_3.9x4.9mm_P1.27mm"
+			(at 59.69 40.64 0)
+			(effects
+				(font
+					(size 1.27 1.27)
+				)
+				(hide yes)
+			)
+		)
+		(property "Datasheet" ""
+			(at 59.69 40.64 0)
+			(effects
+				(font
+					(size 1.27 1.27)
+				)
+				(hide yes)
+			)
+		)
+		(property "Description" ""
+			(at 59.69 40.64 0)
+			(effects
+				(font
+					(size 1.27 1.27)
+				)
+				(hide yes)
+			)
+		)
+		(pin "2"
+		)
+		(pin "5"
+		)
+		(pin "1"
+		)
+		(pin "4"
+		)
+		(pin "6"
+		)
+		(instances
+			(project ""
+				(path "/38a2da3c-ed29-422f-ab41-066ccf490e61/8d296a6f-d65d-491e-bf56-0b9d64795b89"
+					(reference "U23")
+					(unit 1)
+				)
