File: error.kicad_sch (KiCad schematic)
At the start: 2 parts, among them U36 74LS30, U37 TLV702475_SOT23-5

Commit message: 22 mayo 26 actualizacion
se actualizo la PCB para la rama laptop Antigua
Parts:
- renumbered U37 to U40, U36 to U41
Changed lines of the file:
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@@
 		(on_board yes)
 		(dnp no)
-		(property "Reference" "#PWR0207"
+		(property "Reference" "#PWR0435"
 			(at 116.84 44.45 0)
 			(effects
@@
 			(project "01_IO-ASD-PLUS"
 				(path "/38a2da3c-ed29-422f-ab41-066ccf490e61/4c77ec8b-a074-45ff-aaf3-88eedcbac288"
-					(reference "#PWR0207")
+					(reference "#PWR0435")
 					(unit 1)
 				)
@@
 		(dnp no)
 		(fields_autoplaced yes)
-		(property "Reference" "U36"
+		(property "Reference" "U41"
 			(at 172.7117 73.66 0)
 			(effects
@@
 			(project ""
 				(path "/38a2da3c-ed29-422f-ab41-066ccf490e61/4c77ec8b-a074-45ff-aaf3-88eedcbac288"
-					(reference "U36")
+					(reference "U41")
 					(unit 1)
 				)
@@
 		(dnp no)
 		(fields_autoplaced yes)
-		(property "Reference" "U37"
+		(property "Reference" "U40"
 			(at 91.44 53.34 0)
 			(effects
@@
 			(project ""
 				(path "/38a2da3c-ed29-422f-ab41-066ccf490e61/4c77ec8b-a074-45ff-aaf3-88eedcbac288"
-					(reference "U37")
+					(reference "U40")
 					(unit 1)
 				)

Commit message: 05/06/26
Parts:
- renumbered U40 to U42, U41 to U43
Changed lines of the file:
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@@
 		(on_board yes)
 		(dnp no)
-		(property "Reference" "#PWR0435"
+		(property "Reference" "#PWR0320"
 			(at 116.84 44.45 0)
 			(effects
@@
 			(project "01_IO-ASD-PLUS"
 				(path "/38a2da3c-ed29-422f-ab41-066ccf490e61/4c77ec8b-a074-45ff-aaf3-88eedcbac288"
-					(reference "#PWR0435")
+					(reference "#PWR0320")
 					(unit 1)
 				)
@@
 		(dnp no)
 		(fields_autoplaced yes)
-		(property "Reference" "U41"
+		(property "Reference" "U43"
 			(at 172.7117 73.66 0)
 			(effects
@@
 			(project ""
 				(path "/38a2da3c-ed29-422f-ab41-066ccf490e61/4c77ec8b-a074-45ff-aaf3-88eedcbac288"
-					(reference "U41")
+					(reference "U43")
 					(unit 1)
 				)
@@
 		(dnp no)
 		(fields_autoplaced yes)
-		(property "Reference" "U40"
+		(property "Reference" "U42"
 			(at 91.44 53.34 0)
 			(effects
@@
 			(project ""
 				(path "/38a2da3c-ed29-422f-ab41-066ccf490e61/4c77ec8b-a074-45ff-aaf3-88eedcbac288"
-					(reference "U40")
+					(reference "U42")
 					(unit 1)
 				)
