File: error.kicad_sch (KiCad schematic)
At the start: 2 parts, among them U42 TLV702475_SOT23-5, U43 74LS30

Commit message: 13-jul-26_6pm
Parts:
- renumbered U42 to U39, U43 to U40
Changed lines of the file:
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@@
 		(on_board yes)
 		(dnp no)
-		(property "Reference" "#PWR0320"
+		(property "Reference" "#PWR0419"
 			(at 116.84 44.45 0)
 			(effects
@@
 			(project "01_IO-ASD-PLUS"
 				(path "/38a2da3c-ed29-422f-ab41-066ccf490e61/4c77ec8b-a074-45ff-aaf3-88eedcbac288"
-					(reference "#PWR0320")
+					(reference "#PWR0419")
 					(unit 1)
 				)
@@
 		(dnp no)
 		(fields_autoplaced yes)
-		(property "Reference" "U43"
+		(property "Reference" "U40"
 			(at 172.7117 73.66 0)
 			(effects
@@
 			(project ""
 				(path "/38a2da3c-ed29-422f-ab41-066ccf490e61/4c77ec8b-a074-45ff-aaf3-88eedcbac288"
-					(reference "U43")
+					(reference "U40")
 					(unit 1)
 				)
@@
 		(dnp no)
 		(fields_autoplaced yes)
-		(property "Reference" "U42"
+		(property "Reference" "U39"
 			(at 91.44 53.34 0)
 			(effects
@@
 			(project ""
 				(path "/38a2da3c-ed29-422f-ab41-066ccf490e61/4c77ec8b-a074-45ff-aaf3-88eedcbac288"
-					(reference "U42")
+					(reference "U39")
 					(unit 1)
 				)
