File: 01_IO-ASD-PLUS.kicad_pcb (KiCad board)
At the start: 2 copper layers, 180 x 158 mm, 187 parts, among them IC1 LDK320AM120R, IC10 ILD206T, IC11 TLV61048DBVT, IC12 ILD206T, IC13 VNI4140K, IC14 ILD206T, IC15 ILD206T, IC16 ILD206T, IC2 ILD206T, IC3 ILD206T, IC4 ILD206T, IC5 ILD206T, IC6 ILD206T, IC7 ILD206T, IC8 ILD206T, IC9 ILD206T, J1 1604470000, J12 1728810000, J2 1147330000, J3 1147330000, J4 1147330000, J5 1728840000, J6 1728840000, J7 1728840000, K1 G2RL-1-H, K1 G5Q-1A, K3 G2RL-1-E, Q1 FMMT491TC, U1 KF33BDT, U10 MAX3227, U2 5-1415390-1, U3 5-1415390-1, U4 5-1415390-1, U5 LTC3646EMSEPBF, U6 LTC3646EMSEPBF, U7 TSB582IYQ2T, U8 ULN2003, U9 ULN2003

Commit message: 7-may-26 346
se esta trabajando en los reles esquematico y pcb
Parts:
- added D1: LED, LED_SMD:LED_0603_1608Metric, F.Cu at (228.4, 99.2)
- added D2: LED, LED_SMD:LED_0603_1608Metric, F.Cu at (228.4, 101.8)
- added D3: LED, LED_SMD:LED_0603_1608Metric, F.Cu at (228.4, 104.4)
- added K2: G2RL-1-H, Relay_THT:Relay_SPDT_Omron_G2RL-1, F.Cu at (201.4, 101.1)
- added K3: G2RL-1-H, Relay_THT:Relay_SPDT_Omron_G2RL-1, F.Cu at (215.5, 101.1)
- added R3: 1.2k, Resistor_SMD:R_0603_1608Metric, F.Cu at (228.3, 106.9)
- added R4: 1.2k, Resistor_SMD:R_0603_1608Metric, F.Cu at (228.3, 109.4)
- added R5: 1.2k, Resistor_SMD:R_0603_1608Metric, F.Cu at (228.3, 111.9)
- renumbered C14 to C1, C19 to C10, C12 to C11, C20 to C12, C21 to C14, C1 to C15, C2 to C16, C3 to C17, C4 to C18, C28 to C19, C15 to C2, C27 to C20, C26 to C21, C6 to C22, C29 to C23, C32 to C24, C5 to C25, C30 to C26, C7 to C27, C8 to C28, C31 to C29, C16 to C3, C25 to C30, C24 to C31, C23 to C32, C35 to C33, C33 to C35, C17 to C4, C44 to C41, C41 to C42, C42 to C43, C43 to C44, C22 to C5, C9 to C6, C10 to C7, C18 to C8, C11 to C9, D13 to D10, D6 to D11, D8 to D12, D7 to D13, D9 to D14, D10 to D15, D11 to D16, D14 to D17, D15 to D18, D16 to D19, D17 to D20, D3 to D4, D4 to D5, D2 to D6, D1 to D7, D5 to D8, D12 to D9, IC7 to IC1, IC1 to IC12, IC16 to IC15, IC15 to IC16, IC8 to IC2, IC12 to IC3, IC3 to IC5, IC4 to IC6, IC9 to IC7, IC5 to IC8, IC6 to IC9, J3 to J1, J4 to J2, J2 to J3, J1 to J4, J12 to J8, L3 to L1, L4 to L2, L2 to L3, L5 to L4, L1 to L5, R11 to R10, R34 to R11, R35 to R12, R12 to R13, R7 to R14, R8 to R15, R2 to R16, R1 to R17, R26 to R18, R27 to R19, R30 to R20, R28 to R21, R29 to R22, R3 to R23, R4 to R24, R32 to R25, R33 to R26, R31 to R27, R14 to R28, R13 to R29, R15 to R30, R16 to R31, R18 to R32, R19 to R33, R17 to R34, R20 to R35, R21 to R36, R22 to R37, R23 to R38, R24 to R39, R25 to R40, R40 to R41, R41 to R42, R42 to R43, R43 to R44, R36 to R45, R37 to R46, R38 to R47, R39 to R48, R44 to R49, R45 to R50, R46 to R51, R47 to R52, R49 to R53, R48 to R54, R50 to R55, R51 to R56, R56 to R57, R57 to R58, R52 to R59, R9 to R6, R53 to R60, R58 to R61, R59 to R62, R54 to R63, R55 to R64, R5 to R7, R10 to R8, R6 to R9, RV2 to RV1, RV6 to RV2, TP5 to TP3, TP3 to TP4, TP6 to TP5, TP7 to TP6, TP4 to TP7, U9 to U10, U10 to U11, U3 to U2, U2 to U3, U6 to U5, U1 to U6, U5 to U7, U7 to U8, U8 to U9
Connections:
- IC2 pad 1: unconnected-(IC8-A_1-Pad1) (its old number) -> unconnected-(IC2-A_1-Pad1)
- IC2 pad 2: unconnected-(IC8-C_1-Pad2) (its old number) -> unconnected-(IC2-C_1-Pad2)
- IC2 pad 3: unconnected-(IC8-A_2-Pad3) (its old number) -> unconnected-(IC2-A_2-Pad3)
- IC2 pad 4: unconnected-(IC8-C_2-Pad4) (its old number) -> unconnected-(IC2-C_2-Pad4)
- IC2 pad 5: unconnected-(IC8-E_1-Pad5) (its old number) -> unconnected-(IC2-E_1-Pad5)
- IC2 pad 6: unconnected-(IC8-C_3-Pad6) (its old number) -> unconnected-(IC2-C_3-Pad6)
- IC2 pad 7: unconnected-(IC8-E_2-Pad7) (its old number) -> unconnected-(IC2-E_2-Pad7)
- IC2 pad 8: unconnected-(IC8-C_4-Pad8) (its old number) -> unconnected-(IC2-C_4-Pad8)
- IC3 pad 5: unconnected-(IC12-E_1-Pad5) -> Net-(IC3-E_1)
- IC3 pad 6: unconnected-(IC12-C_3-Pad6) -> +5v
- IC3 pad 7: unconnected-(IC12-E_2-Pad7) -> Net-(IC3-E_2)
- IC3 pad 8: unconnected-(IC12-C_4-Pad8) -> +5v
- K1 pad A1: unconnected-(K1-PadA1) -> Net-(U1-COM)
- K1 pad A2: unconnected-(K1-PadA2) -> Net-(D1-K)
- RV1 pad 1: unconnected-(RV2-Pad1) (its old number) -> unconnected-(RV1-Pad1)
- RV1 pad 2: unconnected-(RV2-Pad2) (its old number) -> unconnected-(RV1-Pad2)

Commit message: 13-Mayo26 se agrego hoja de procesador y USB
hoja de USB AL 95% HOJA DEL procesador al 75%
Parts:
- removed ? (x7): , 
- removed the IC2 at (342.4, 40.3)
- removed J3: 1147330000, CONECTORES GRACIDA:3POS-5.08PITCH
- removed the K1 at (209.1, 150.8)
- removed the K3 at (178.4, 140.8)
- removed REF**: TestPoint_THTPad_D4.0mm_Drill2.0mm, TestPoint:TestPoint_THTPad_D4.0mm_Drill2.0mm
- removed the RV1 at (191.6, 183.8)
- added J9: 1147330000, CONECTORES GRACIDA:3POS-5.08PITCH, F.Cu at (251.2, 199.9)
- added RV5: Varistor, Varistor:RV_Disc_D12mm_W3.9mm_P7.5mm, F.Cu at (234.3, 186.3)
- moved RV2 150.8 mm to (266.2, 187.1)
- moved U2 78.5 mm to (243.2, 251.6)
- moved U3 78.5 mm to (221.4, 249.3)
- moved U4 78.5 mm to (193.8, 250.3)
- moved RV1 74.0 mm to (285.5, 187.6)
- moved K2 73.4 mm to (241.5, 162.6)
- moved K3 61.1 mm to (210.2, 161.9)
- moved J1 57.1 mm to (209.1, 200.3), turned to 0 degrees
- moved J6 48.2 mm to (131.9, 138.7)
- moved J7 47.5 mm to (131.9, 114.4)
- moved J8 45.6 mm to (132.3, 157.6)
- moved RV4 40.5 mm to (245.0, 143.1)
- moved K1 40.0 mm to (272.7, 164.1)
- moved J5 38.8 mm to (160.1, 176.8)
- moved RV3 34.5 mm to (254.9, 187.0)
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Connections:
- J1 pad 1: unconnected-(J1-Pad1) -> Net-(J1-Pad1)
- J1 pad 2: unconnected-(J1-Pad2) -> Net-(J1-Pad2)
- J1 pad 3: unconnected-(J1-Pad3) -> Net-(J1-Pad3)
- J2 pad 1: unconnected-(J2-Pad1) -> Net-(J2-Pad1)
- J2 pad 2: unconnected-(J2-Pad2) -> Net-(J2-Pad2)
- J2 pad 3: unconnected-(J2-Pad3) -> Net-(J2-Pad3)
- K1 pad 11: unconnected-(K1-Pad11) -> Net-(J2-Pad2)
- K1 pad 12: unconnected-(K1-Pad12) -> Net-(J2-Pad1)
- K1 pad 14: unconnected-(K1-Pad14) -> Net-(J2-Pad3)
- K2 pad 11: unconnected-(K2-Pad11) -> Net-(J9-Pad2)
- K2 pad 12: unconnected-(K2-Pad12) -> Net-(J9-Pad1)
- K2 pad 14: unconnected-(K2-Pad14) -> Net-(J9-Pad3)
- K3 pad 11: unconnected-(K3-Pad11) -> Net-(J1-Pad2)
- K3 pad 12: unconnected-(K3-Pad12) -> Net-(J1-Pad1)
- K3 pad 14: unconnected-(K3-Pad14) -> Net-(J1-Pad3)
- RV1 pad 1: unconnected-(RV1-Pad1) -> Net-(J2-Pad3)
- RV1 pad 2: unconnected-(RV1-Pad2) -> Net-(J2-Pad2)
- RV2 pad 1: unconnected-(RV2-Pad1) -> Net-(J2-Pad1)
- RV2 pad 2: unconnected-(RV2-Pad2) -> Net-(J2-Pad2)
- RV3 pad 1: unconnected-(RV3-Pad1) -> Net-(J9-Pad1)
- RV3 pad 2: unconnected-(RV3-Pad2) -> Net-(J9-Pad2)

Commit message: 14-Mayo-26
se agregaron varias sheet de esquematico crecio al 80% la parte de esquematico
Parts:
- removed the C30 at (46.5, 164.7)
- removed the C32 at (41.5, 164.7)
- removed C33, C35: 0.1uF, Capacitor_SMD:C_0603_1608Metric_Pad1.08x0.95mm_HandSolder
- removed C34: 47uF, Capacitor_Tantalum_SMD:CP_EIA-1608-10_AVX-L_HandSolder
- removed the D17 at (48.1, 184.1)
- removed D18, D19, D20: LED, LED_SMD:LED_0603_1608Metric_Pad1.05x0.95mm_HandSolder
- removed IC13: VNI4140K, Package_SO:ST_PowerSSO-24_SlugDown_ThermalVias
- removed the J5 at (160.1, 176.8)
- removed J6: 1728840000, CONECTORES GRACIDA:1728840000_17-25
- removed L6: 10uH, Inductor_SMD:L_0603_1608Metric_Pad1.05x0.95mm_HandSolder
- removed R28, R31, R34: 10ohms, Resistor_SMD:R_0603_1608Metric_Pad0.98x0.95mm_HandSolder
- removed R29, R30: 1k, Resistor_SMD:R_0603_1608Metric_Pad0.98x0.95mm_HandSolder
- removed R32: 10k, Resistor_SMD:R_0603_1608Metric_Pad0.98x0.95mm_HandSolder
- removed R33: 30ohms, Resistor_SMD:R_0603_1608Metric_Pad0.98x0.95mm_HandSolder
- removed R39, R40: 4.7k, Resistor_SMD:R_0805_2012Metric_Pad1.20x1.40mm_HandSolder
- removed R41, R42, R48: 4.7k, Capacitor_SMD:C_0603_1608Metric_Pad1.08x0.95mm_HandSolder
- removed R49, R50, R51, R52: 10k, Capacitor_SMD:C_0603_1608Metric_Pad1.08x0.95mm_HandSolder
- removed TH1: B59985C120A70, TERMISTORES GRACIDA:B59985C0120A070
- removed U10: ULN2003, Package_SO:SOIC-16_4.55x10.3mm_P1.27mm
- removed U8: TSB582IYQ2T, Package_DFN_QFN:DFN-8-1EP_6x5mm_P1.27mm_EP4x4mm
- added C100: 0.1uF, Capacitor_SMD:C_0603_1608Metric_Pad1.08x0.95mm_HandSolder, F.Cu at (28.7, 86.5)
- added C101: 0.1uF, Capacitor_SMD:C_0603_1608Metric_Pad1.08x0.95mm_HandSolder, F.Cu at (28.7, 89.0)
- added C102: 0.1uF, Capacitor_SMD:C_0603_1608Metric_Pad1.08x0.95mm_HandSolder, F.Cu at (33.0, 71.4)
- added C103: 0.1uF, Capacitor_SMD:C_0603_1608Metric_Pad1.08x0.95mm_HandSolder, F.Cu at (33.0, 74.0)
- added C104: 0.1uF, Capacitor_SMD:C_0603_1608Metric_Pad1.08x0.95mm_HandSolder, F.Cu at (33.0, 76.5)
- added C105: 0.1uF, Capacitor_SMD:C_0603_1608Metric_Pad1.08x0.95mm_HandSolder, F.Cu at (33.0, 79.0)
- added C106: 0.1uF, Capacitor_SMD:C_0603_1608Metric_Pad1.08x0.95mm_HandSolder, F.Cu at (33.0, 81.5)
- added C107: 18pF, Capacitor_SMD:C_0603_1608Metric_Pad1.08x0.95mm_HandSolder, F.Cu at (33.0, 84.0)
- added C108: 18pF, Capacitor_SMD:C_0603_1608Metric_Pad1.08x0.95mm_HandSolder, F.Cu at (33.0, 86.5)
- added C109: 0.1uF, Capacitor_SMD:C_0603_1608Metric_Pad1.08x0.95mm_HandSolder, F.Cu at (62.1, 83.5)
- added C110: 0.1uF, Capacitor_SMD:C_0603_1608Metric_Pad1.08x0.95mm_HandSolder, F.Cu at (62.1, 86.0)
- added C111: 0.1uF, Capacitor_SMD:C_0603_1608Metric_Pad1.08x0.95mm_HandSolder, F.Cu at (62.1, 88.5)
- added C113: 0.1uF, Capacitor_SMD:C_0603_1608Metric_Pad1.08x0.95mm_HandSolder, F.Cu at (62.1, 91.0)
- added C115: 0.1uF, Capacitor_SMD:C_0603_1608Metric_Pad1.08x0.95mm_HandSolder, F.Cu at (62.1, 93.5)
- added C18: 0.1uF, Capacitor_SMD:C_0603_1608Metric_Pad1.08x0.95mm_HandSolder, F.Cu at (68.5, 83.5)
- added C27: 0.01uF, Capacitor_SMD:C_0603_1608Metric_Pad1.08x0.95mm_HandSolder, F.Cu at (68.5, 86.0)
- added C39: 0.1uF, Capacitor_SMD:C_0603_1608Metric_Pad1.08x0.95mm_HandSolder, F.Cu at (33.8, 47.6)
- added C41: 0.1uF, Capacitor_SMD:C_0603_1608Metric_Pad1.08x0.95mm_HandSolder, F.Cu at (33.8, 50.1)
- added C44: 0.1uF, Capacitor_SMD:C_0603_1608Metric_Pad1.08x0.95mm_HandSolder, F.Cu at (33.8, 52.7)
- added C45: 0.1uF, Capacitor_SMD:C_0603_1608Metric_Pad1.08x0.95mm_HandSolder, F.Cu at (33.8, 55.2)
- added C46: 0.1uF, Capacitor_SMD:C_0603_1608Metric_Pad1.08x0.95mm_HandSolder, F.Cu at (33.8, 57.7)
- added C47: 0.1uF, Capacitor_SMD:C_0603_1608Metric_Pad1.08x0.95mm_HandSolder, F.Cu at (33.8, 60.2)
- added C48: 0.1uF, Capacitor_SMD:C_0603_1608Metric_Pad1.08x0.95mm_HandSolder, F.Cu at (33.8, 62.7)
- added C49: 0.1uF, Capacitor_SMD:C_0603_1608Metric_Pad1.08x0.95mm_HandSolder, F.Cu at (38.2, 45.1)
- added C59: 470nF, Capacitor_SMD:C_0603_1608Metric, F.Cu at (51.1, 45.1)
- added C61: 4.7uF, Capacitor_SMD:C_0603_1608Metric, F.Cu at (51.1, 47.6)
- added C67: 10uF, Capacitor_SMD:C_0603_1608Metric, F.Cu at (51.1, 50.1)
- added C68: 4.7uF, Capacitor_SMD:C_0603_1608Metric, F.Cu at (51.1, 52.7)
- added C69: 0.1uF, Capacitor_SMD:C_0603_1608Metric_Pad1.08x0.95mm_HandSolder, F.Cu at (38.2, 47.6)
- added C73: 0.1uF, Capacitor_SMD:C_0603_1608Metric_Pad1.08x0.95mm_HandSolder, F.Cu at (38.2, 50.1)
- added C83: 1nF, Capacitor_SMD:C_0603_1608Metric_Pad1.08x0.95mm_HandSolder, F.Cu at (24.3, 71.4)
- added C84: 0.1uF, Capacitor_SMD:C_0603_1608Metric_Pad1.08x0.95mm_HandSolder, F.Cu at (24.3, 74.0)
- added C85: 0.1uF, Capacitor_SMD:C_0603_1608Metric_Pad1.08x0.95mm_HandSolder, F.Cu at (24.3, 76.5)
- added C86: 0.1uF, Capacitor_SMD:C_0603_1608Metric_Pad1.08x0.95mm_HandSolder, F.Cu at (24.3, 79.0)
- added C87: 0.1uF, Capacitor_SMD:C_0603_1608Metric_Pad1.08x0.95mm_HandSolder, F.Cu at (24.3, 81.5)
- added C88: 0.01uF, Capacitor_SMD:C_0603_1608Metric_Pad1.08x0.95mm_HandSolder, F.Cu at (24.3, 84.0)
- added C91: 0.01uF, Capacitor_SMD:C_0603_1608Metric_Pad1.08x0.95mm_HandSolder, F.Cu at (24.3, 86.5)
- added C92: 0.1uF, Capacitor_SMD:C_0603_1608Metric_Pad1.08x0.95mm_HandSolder, F.Cu at (24.3, 89.0)
- added C94: 10pF, Capacitor_SMD:C_0603_1608Metric_Pad1.08x0.95mm_HandSolder, F.Cu at (28.7, 71.4)
- added C95: 10pF, Capacitor_SMD:C_0603_1608Metric_Pad1.08x0.95mm_HandSolder, F.Cu at (28.7, 74.0)
- added C96: 0.01uF, Capacitor_SMD:C_0603_1608Metric_Pad1.08x0.95mm_HandSolder, F.Cu at (28.7, 76.5)
- added C97: 0.1uF, Capacitor_SMD:C_0603_1608Metric_Pad1.08x0.95mm_HandSolder, F.Cu at (28.7, 79.0)
- added C98: 1uF, Capacitor_SMD:C_0603_1608Metric_Pad1.08x0.95mm_HandSolder, F.Cu at (28.7, 81.5)
- added C99: 0.1uF, Capacitor_SMD:C_0603_1608Metric_Pad1.08x0.95mm_HandSolder, F.Cu at (28.7, 84.0)
- added CN1: 10way 1.27mm, CONECTORES GRACIDA:MicroMatch_10way_P1.75mm, F.Cu at (185.7, 175.5)
- added D12: SP0502BAHT, Package_TO_SOT_SMD:SOT-23, F.Cu at (73.1, 89.1)
- added D22: LED, LED_SMD:LED_0603_1608Metric_Pad1.05x0.95mm_HandSolder, F.Cu at (29.5, 45.2)
- added D23: LED, LED_SMD:LED_0603_1608Metric_Pad1.05x0.95mm_HandSolder, F.Cu at (29.5, 47.8)
- added D24: LED, LED_SMD:LED_0603_1608Metric_Pad1.05x0.95mm_HandSolder, F.Cu at (29.5, 50.3)
- added D25: LED, LED_SMD:LED_0603_1608Metric_Pad1.05x0.95mm_HandSolder, F.Cu at (29.5, 52.9)
- added D27: LED, LED_SMD:LED_0603_1608Metric_Pad1.05x0.95mm_HandSolder, F.Cu at (29.5, 55.5)
- added D28: LED, LED_SMD:LED_0603_1608Metric_Pad1.05x0.95mm_HandSolder, F.Cu at (29.5, 58.1)
- added D29: LED, LED_SMD:LED_0603_1608Metric_Pad1.05x0.95mm_HandSolder, F.Cu at (29.5, 60.7)
- added D30: LED, LED_SMD:LED_0603_1608Metric_Pad1.05x0.95mm_HandSolder, F.Cu at (29.5, 63.3)
- added D31: LED, LED_SMD:LED_0402_1005Metric, F.Cu at (68.9, 42.7)
- added D32: PMEG2010BER, Diode_SMD:Nexperia_CFP3_SOD-123W, F.Cu at (38.0, 97.9)
- added D33: LED, LED_SMD:LED_0603_1608Metric_Pad1.05x0.95mm_HandSolder, F.Cu at (62.1, 96.1)
- added D34: LED, LED_SMD:LED_0603_1608Metric_Pad1.05x0.95mm_HandSolder, F.Cu at (62.1, 98.7)
- added F1: Fuse_Small, Capacitor_SMD:C_0603_1608Metric, F.Cu at (51.1, 55.2)
- added IC14: VNI4140K, Package_SO:ST_PowerSSO-24_SlugDown_ThermalVias, F.Cu at (71.7, 49.8)
- added J4: 1147330000, CONECTORES GRACIDA:3POS-5.08PITCH, F.Cu at (60.1, 75.7)
- added J7: 1728840000, CONECTORES GRACIDA:1728840000, F.Cu at (31.3, 24.9)
- added J8: 1728840000, CONECTORES GRACIDA:1728840000_17-25, F.Cu at (31.3, 38.5)
- added L7: 0603, Inductor_SMD:L_0603_1608Metric_Pad1.05x0.95mm_HandSolder, F.Cu at (38.2, 52.7)
- added L9: 10uH, Inductor_SMD:L_0603_1608Metric_Pad1.05x0.95mm_HandSolder, F.Cu at (38.2, 55.2)
- added Q10: DMP3099L, Package_TO_SOT_SMD:SOT-23, F.Cu at (67.1, 32.2)
- added Q11: DMP3099L, Package_TO_SOT_SMD:SOT-23, F.Cu at (67.1, 36.7)
- added Q12: DMP3099L, Package_TO_SOT_SMD:SOT-23, F.Cu at (72.1, 18.9)
- added Q13: DMP3099L, Package_TO_SOT_SMD:SOT-23, F.Cu at (72.1, 23.3)
- added Q2: MMBT3904, Package_TO_SOT_SMD:SOT-23, F.Cu at (62.2, 18.9)
- added Q3: MMBT3904, Package_TO_SOT_SMD:SOT-23, F.Cu at (62.2, 23.3)
- added Q4: MMBT3904, Package_TO_SOT_SMD:SOT-23, F.Cu at (62.2, 27.8)
- added Q5: MMBT3904, Package_TO_SOT_SMD:SOT-23, F.Cu at (62.2, 32.2)
- added Q6: MMBT3904, Package_TO_SOT_SMD:SOT-23, F.Cu at (62.2, 36.7)
- added Q7: MMBT3904, Package_TO_SOT_SMD:SOT-23, F.Cu at (67.1, 18.9)
- added Q8: DMP3099L, Package_TO_SOT_SMD:SOT-23, F.Cu at (67.1, 23.3)
- added Q9: DMP3099L, Package_TO_SOT_SMD:SOT-23, F.Cu at (67.1, 27.8)
- added R102: 10k, Capacitor_SMD:C_0603_1608Metric_Pad1.08x0.95mm_HandSolder, F.Cu at (46.9, 47.6)
- added R103: 10k, Capacitor_SMD:C_0603_1608Metric_Pad1.08x0.95mm_HandSolder, F.Cu at (46.9, 50.1)
- added R104: 10k, Capacitor_SMD:C_0603_1608Metric_Pad1.08x0.95mm_HandSolder, F.Cu at (46.9, 52.7)
- added R105: 10k, Capacitor_SMD:C_0603_1608Metric_Pad1.08x0.95mm_HandSolder, F.Cu at (46.9, 55.2)
- added R141: 2.2k, Resistor_SMD:R_0603_1608Metric, F.Cu at (24.1, 91.5)
- added R142: 10k, Resistor_SMD:R_0603_1608Metric, F.Cu at (24.1, 94.0)
- added R143: 10k, Resistor_SMD:R_0603_1608Metric, F.Cu at (24.1, 96.5)
- added R144: 0, Resistor_SMD:R_0603_1608Metric, F.Cu at (24.1, 99.1)
- added R145: 0, Resistor_SMD:R_0603_1608Metric, F.Cu at (24.1, 101.6)
- added R146: 1K, Resistor_SMD:R_0603_1608Metric, F.Cu at (24.1, 104.1)
- added R147: 12k 1%, Resistor_SMD:R_0603_1608Metric, F.Cu at (28.1, 91.5)
- added R148: 1K, Resistor_SMD:R_0603_1608Metric, F.Cu at (28.1, 94.0)
- added R149: 12k 1%, Resistor_SMD:R_0603_1608Metric, F.Cu at (28.1, 96.5)
- added R150: 12.3k 1%, Resistor_SMD:R_0603_1608Metric, F.Cu at (28.1, 99.1)
- added R151: 10k, Resistor_SMD:R_0603_1608Metric, F.Cu at (28.1, 101.6)
- added R152: 10k, Resistor_SMD:R_0603_1608Metric, F.Cu at (57.9, 83.5)
- added R153: 10k, Resistor_SMD:R_0603_1608Metric, F.Cu at (57.9, 86.0)
- added R154: 470, Resistor_SMD:R_0603_1608Metric, F.Cu at (57.9, 88.5)
- added R155: 470, Resistor_SMD:R_0603_1608Metric, F.Cu at (57.9, 91.0)
- added R156: 5.1k 1%, Resistor_SMD:R_0603_1608Metric, F.Cu at (57.9, 93.5)
- added R157: 0, Resistor_SMD:R_0603_1608Metric, F.Cu at (57.9, 96.0)
- added R158: 0, Resistor_SMD:R_0603_1608Metric, F.Cu at (57.9, 98.6)
- added R159: 0, Resistor_SMD:R_0603_1608Metric, F.Cu at (57.9, 101.1)
- added R56: 10k, Capacitor_SMD:C_0603_1608Metric_Pad1.08x0.95mm_HandSolder, F.Cu at (42.5, 57.7)
- added R57: 10k, Capacitor_SMD:C_0603_1608Metric_Pad1.08x0.95mm_HandSolder, F.Cu at (42.5, 60.2)
- added R58: 10k, Capacitor_SMD:C_0603_1608Metric_Pad1.08x0.95mm_HandSolder, F.Cu at (42.5, 62.7)
- added R59: 10k, Capacitor_SMD:C_0603_1608Metric_Pad1.08x0.95mm_HandSolder, F.Cu at (46.9, 45.1)
- added R61: 2.2k, Resistor_SMD:R_0603_1608Metric, F.Cu at (51.1, 60.2)
- added R62: 2.2k, Resistor_SMD:R_0603_1608Metric, F.Cu at (55.1, 45.1)
- added R63: 2.2k, Resistor_SMD:R_0603_1608Metric, F.Cu at (55.1, 47.6)
- added R64: 2.2k, Resistor_SMD:R_0603_1608Metric, F.Cu at (55.1, 50.1)
- added R65: 2.2k, Resistor_SMD:R_0603_1608Metric, F.Cu at (55.1, 52.7)
- added R66: 2.2k, Resistor_SMD:R_0603_1608Metric, F.Cu at (55.1, 55.2)
- added R67: 1k, Resistor_SMD:R_0603_1608Metric, F.Cu at (55.1, 57.7)
- added R68: 1k, Resistor_SMD:R_0603_1608Metric, F.Cu at (55.1, 60.2)
- added R69: 1k, Resistor_SMD:R_0603_1608Metric, F.Cu at (59.1, 45.1)
- added R70: 1k, Resistor_SMD:R_0603_1608Metric, F.Cu at (59.1, 47.6)
- added R71: 1k, Resistor_SMD:R_0603_1608Metric, F.Cu at (59.1, 50.1)
- added R72: 1k, Resistor_SMD:R_0603_1608Metric, F.Cu at (59.1, 52.7)
- added R73: 10k, Resistor_SMD:R_0603_1608Metric, F.Cu at (59.1, 55.2)
- added R74: 10, Resistor_SMD:R_0603_1608Metric, F.Cu at (59.1, 57.7)
- added R76: 10k, Resistor_SMD:R_0603_1608Metric, F.Cu at (59.1, 60.2)
- added R78: 10, Resistor_SMD:R_0603_1608Metric, F.Cu at (63.1, 45.1)
- added R80: 0 ohms, Resistor_SMD:R_0603_1608Metric, F.Cu at (63.1, 47.6)
- added R84: 10k, Resistor_SMD:R_0603_1608Metric, F.Cu at (63.1, 50.1)
- added R95: 10k, Resistor_SMD:R_0603_1608Metric, F.Cu at (63.1, 52.7)
- added U11: 74LVC1G17, Package_TO_SOT_SMD:SOT-23-5, F.Cu at (24.7, 19.1)
- added U12: 74LVC1G17, Package_TO_SOT_SMD:SOT-23-5, F.Cu at (24.7, 23.7)
- added U13: 74LVC1G17, Package_TO_SOT_SMD:SOT-23-5, F.Cu at (24.7, 28.3)
- added U14: 74LVC1G17, Package_TO_SOT_SMD:SOT-23-5, F.Cu at (24.7, 32.9)
- added U15: 74LVC1G17, Package_TO_SOT_SMD:SOT-23-5, F.Cu at (24.7, 37.6)
- added U16: 74LVC1G17, Package_TO_SOT_SMD:SOT-23-5, F.Cu at (24.7, 42.2)
- added U17: TSB582, Package_DFN_QFN:DFN-8-1EP_6x5mm_P1.27mm_EP4x4mm, F.Cu at (53.8, 64.9)
- added U21: LM7705, Package_SO:VSSOP-8_3x3mm_P0.65mm, F.Cu at (63.5, 41.3)
- added U22: MCP1799T-5002H/TT, Package_TO_SOT_SMD:SOT-23, F.Cu at (72.1, 27.8)
- added U25: FT900L-C-T, footprints:LQFP_100_14X14X1P4_BRI, F.Cu at (44.5, 79.6)
- added U7: TLV70212_SOT23-5, Package_TO_SOT_SMD:SOT-23-5, F.Cu at (73.2, 84.6)
- C36: value 0.1uF -> 47uF; footprint Capacitor_SMD:C_0603_1608Metric_Pad1.08x0.95mm_HandSolder -> Capacitor_Tantalum_SMD:CP_EIA-1608-10_AVX-L_HandSolder
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- renumbered C8 to C10, C10 to C11, C14 to C13, C22 to C14, C25 to C15, C27 to C16, C28 to C17, C6 to C19, C7 to C20, C19 to C21, C20 to C22, C21 to C23, C9 to C24, C11 to C25, C13 to C26, C23 to C28, C24 to C29, C5 to C3, C26 to C30, C29 to C32, C3 to C4, C4 to C5, C15 to C6, C16 to C7, C38 to C76, C39 to C77, C40 to C78, C41 to C79, C17 to C8, C42 to C80, C43 to C81, C44 to C82, C18 to C9, D12 to D13, D13 to D14, D14 to D15, D15 to D16, D16 to D17, D6 to D5, D5 to D6, IC2 to IC1, IC14 to IC15, IC15 to IC16, IC16 to IC17, IC1 to IC2, IC5 to IC3, IC6 to IC4, IC7 to IC5, IC3 to IC6, J2 to J1, J8 to J10, J9 to J2, J1 to J3, J4 to J5, J7 to J9, L7 to L10, L5 to L4, L4 to L5, R11 to R10, R16 to R11, R17 to R12, R53 to R129, R12 to R13, R54 to R130, R55 to R131, R56 to R132, R57 to R133, R58 to R134, R59 to R135, R60 to R136, R61 to R137, R62 to R138, R63 to R139, R13 to R14, R64 to R140, R14 to R15, R15 to R16, R23 to R17, R24 to R18, R18 to R19, R3 to R2, R19 to R20, R20 to R21, R21 to R22, R22 to R23, R25 to R24, R26 to R25, R27 to R26, R4 to R3, R5 to R4, R6 to R5, R7 to R6, R8 to R7, R9 to R8, R10 to R9, RV2 to RV1, RV1 to RV2, RV5 to RV4, RV4 to RV5, TH2 to TH3, U2 to U1, U3 to U2, U11 to U24, U4 to U3, U5 to U4, U7 to U5
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Connections:
- net Net-(D1-K) renamed /Reles/METAL1_RELE
- net Net-(D2-K) renamed /Reles/METAL2_RELE
- net Net-(D3-K) renamed /Reles/FAULT_RELE
- C31 pad 1: Net-(U8A-VCC-) -> +1.2V
- C36 pad 1: GND -> +24V
- C36 pad 2: Net-(C36-Pad2) -> GND
- C37 pad 2: Net-(C37-Pad2) -> +24V
- IC2 pad 6: unconnected-(IC1-C_3-Pad6) (its old number) -> Net-(IC2-C_3)
- IC2 pad 7: unconnected-(IC1-E_2-Pad7) (its old number) -> Net-(IC2-E_2)
- IC2 pad 8: unconnected-(IC1-C_4-Pad8) (its old number) -> Net-(IC2-C_4)
- IC5 pad 2: unconnected-(IC7-C_1-Pad2) -> Net-(IC2-C_4)
- IC5 pad 3: unconnected-(IC7-A_2-Pad3) -> Net-(IC2-E_2)
- IC5 pad 4: unconnected-(IC7-C_2-Pad4) -> Net-(IC2-C_3)
- IC6 pad 5: Net-(IC3-E_1) -> unconnected-(IC6-E_1-Pad5)
- IC6 pad 7: Net-(IC3-E_2) -> unconnected-(IC6-E_2-Pad7)
- R35 pad 1: +24V -> Net-(IC14-STAT4)
- R35 pad 2: Net-(J5-FUR) -> +3.3V
- R36 pad 1: +24V -> Net-(IC14-STAT3)
- R36 pad 2: Net-(J5-FUL) -> +3.3V
- R37 pad 1: +24V -> Net-(IC14-STAT2)
- R37 pad 2: Net-(J5-FREI) -> +3.3V
- R38 pad 1: +24V -> Net-(IC14-STAT1)
- R38 pad 2: Net-(J5-MZ) -> +3.3V
- R43 pad 1: Net-(IC13-STAT2) -> GND
- R43 pad 2: +3.3V -> /SALIDA J5 y J6/IN1_MO1
- R44 pad 1: Net-(IC13-STAT1) -> GND
- R44 pad 2: +3.3V -> /SALIDA J5 y J6/IN2_MO2
- R45 pad 2: Net-(IC13-IN1) -> /SALIDA J5 y J6/IN3_MO3
- R46 pad 2: Net-(IC13-IN2) -> /SALIDA J5 y J6/IN4_MO4
- R47 pad 1: GND -> Net-(U9-~{RESET})
- R47 pad 2: Net-(IC13-IN3) -> +3.3v
- U9 pad 1: unconnected-(U9-I1-Pad1) -> Net-(U9-GPB0)
- U9 pad 10: unconnected-(U9-O7-Pad10) -> GND
- U9 pad 11: Net-(J5-OUT2) -> /SALIDA J5 y J6/!CS_MCP23S7_SS_1_J5
- U9 pad 12: Net-(J5-ICM) -> /SALIDA J5 y J6/SCK_MCP23S7-SS_1_J5
- U9 pad 13: Net-(J5-MZ) -> /SALIDA J5 y J6/MOSI_MCP23S7_SS_1_J5
- U9 pad 14: Net-(J5-FREI) -> /SALIDA J5 y J6/MISO_MCP23S7_SS_1_J5
- U9 pad 15: Net-(J5-FUL) -> GND
- U9 pad 16: Net-(J5-FUR) -> +3.3v
- U9 pad 2: unconnected-(U9-I2-Pad2) -> Net-(U9-GPB1)
- U9 pad 3: unconnected-(U9-I3-Pad3) -> Net-(U9-GPB2)
- U9 pad 4: unconnected-(U9-I4-Pad4) -> Net-(U9-GPB3)
- U9 pad 5: unconnected-(U9-I5-Pad5) -> Net-(U9-GPB4)
- U9 pad 6: unconnected-(U9-I6-Pad6) -> Net-(U9-GPB5)
- U9 pad 7: unconnected-(U9-I7-Pad7) -> Net-(IC14-STAT1)
- U9 pad 8: GND -> Net-(IC14-STAT2)
- U9 pad 9: GND -> +3.3v

Commit message: 22 mayo 26 actualizacion
se actualizo la PCB para la rama laptop Antigua
Parts:
- removed the C22 at (344.1, 112.6)
- removed the C23 at (341.6, 112.6)
- removed the C28 at (349.1, 112.6)
- removed the C29 at (341.6, 108.2)
- removed C30: 2.2uF, Capacitor_SMD:C_0603_1608Metric_Pad1.08x0.95mm_HandSolder
- removed C32: 0.1uF, Capacitor_SMD:C_0603_1608Metric_Pad1.08x0.95mm_HandSolder
- removed D13, D14: BZT52BC18, Diode_SMD:D_SOD-123F
- removed D15, D16, D17: B120AF-13, Diode_SMD:D_SMA
- removed IC1, IC10, IC2, IC3, IC8, IC9: ILD206T, SOIC:SOIC 8
- removed IC11: TLV61048DBVT, Package_TO_SOT_SMD:TSOT-23-6_HandSoldering
- removed IC12: LDK320AM120R, Package_TO_SOT_SMD:SOT-23-5
- removed the IC4 at (318.7, 183.6)
- removed the IC5 at (313.0, 80.0)
- removed the IC6 at (134.0, 241.2)
- removed the J4 at (60.1, 75.7)
- removed the L5 at (346.2, 96.0)
- removed Q1: FMMT491TC, Package_TO_SOT_SMD:TSOT-23_HandSoldering
- removed R132: 10k, Capacitor_SMD:C_0603_1608Metric_Pad1.08x0.95mm_HandSolder
- removed the R19 at (344.1, 108.2)
- removed the R20 at (346.6, 108.2)
- removed R21: 1ohm, Resistor_SMD:R_0603_1608Metric_Pad0.98x0.95mm_HandSolder
- removed R22: 1M, Resistor_SMD:R_0603_1608Metric_Pad0.98x0.95mm_HandSolder
- removed R23: 70.5k, Resistor_SMD:R_0603_1608Metric_Pad0.98x0.95mm_HandSolder
- removed R24, R25: 0ohms, Resistor_SMD:R_0603_1608Metric_Pad0.98x0.95mm_HandSolder
- removed R26: 10ohm, Resistor_SMD:R_0603_1608Metric_Pad0.98x0.95mm_HandSolder
- removed RV5: Varistor, Varistor:RV_Disc_D12mm_W3.9mm_P7.5mm
- removed the U1 at (243.2, 251.6)
- removed the U2 at (221.4, 249.3)
- removed U25: FT900L-C-T, footprints:LQFP_100_14X14X1P4_BRI
- removed the U3 at (193.8, 250.3)
- removed U7: TLV70212_SOT23-5, Package_TO_SOT_SMD:SOT-23-5
- added C108: 0.1uF, Capacitor_SMD:C_0603_1608Metric_Pad1.08x0.95mm_HandSolder, F.Cu at (273.3, -14.8)
- added C11: 2.2uF, Capacitor_THT:C_Rect_L26.5mm_W11.5mm_P22.50mm_MKS4, F.Cu at (219.9, -12.1)
- added C111: 0.1uF, Capacitor_SMD:C_0603_1608Metric_Pad1.08x0.95mm_HandSolder, F.Cu at (273.3, -12.3)
- added C114: 0.1uF, Capacitor_SMD:C_0603_1608Metric_Pad1.08x0.95mm_HandSolder, F.Cu at (273.3, -9.79)
- added C12: 2.2uF, Capacitor_THT:C_Rect_L26.5mm_W11.5mm_P22.50mm_MKS4, F.Cu at (219.9, 1.00)
- added C126: 0.1uF, Capacitor_SMD:C_0603_1608Metric_Pad1.08x0.95mm_HandSolder, F.Cu at (249.3, 12.6)
- added C127: 0.1uF, Capacitor_SMD:C_0603_1608Metric_Pad1.08x0.95mm_HandSolder, F.Cu at (249.3, 15.1)
- added C128: 0.1uF, Capacitor_SMD:C_0603_1608Metric_Pad1.08x0.95mm_HandSolder, F.Cu at (249.3, 17.6)
- added C129: 0.1uF, Capacitor_SMD:C_0603_1608Metric_Pad1.08x0.95mm_HandSolder, F.Cu at (249.3, 20.1)
- added C130: 0.1uF, Capacitor_SMD:C_0603_1608Metric_Pad1.08x0.95mm_HandSolder, F.Cu at (249.3, 22.6)
- added C131: 0.1uF, Capacitor_SMD:C_0603_1608Metric_Pad1.08x0.95mm_HandSolder, F.Cu at (249.3, 25.1)
- added C132: 0.1uF, Capacitor_SMD:C_0603_1608Metric_Pad1.08x0.95mm_HandSolder, F.Cu at (249.3, 27.7)
- added C133: 0.1uF, Capacitor_SMD:C_0603_1608Metric_Pad1.08x0.95mm_HandSolder, F.Cu at (249.3, 30.2)
- added C134: 0.1uF, Capacitor_SMD:C_0603_1608Metric_Pad1.08x0.95mm_HandSolder, F.Cu at (253.7, 12.6)
- added C135: 0.1uF, Capacitor_SMD:C_0603_1608Metric_Pad1.08x0.95mm_HandSolder, F.Cu at (249.3, 34.7)
- added C136: 0.1uF, Capacitor_SMD:C_0603_1608Metric_Pad1.08x0.95mm_HandSolder, F.Cu at (249.3, 37.2)
- added C137: 0.1uF, Capacitor_SMD:C_0603_1608Metric_Pad1.08x0.95mm_HandSolder, F.Cu at (249.3, 39.7)
- added C138: 0.1uF, Capacitor_SMD:C_0603_1608Metric_Pad1.08x0.95mm_HandSolder, F.Cu at (249.3, 42.2)
- added C139: 0.1uF, Capacitor_SMD:C_0603_1608Metric_Pad1.08x0.95mm_HandSolder, F.Cu at (249.3, 44.7)
- added C140: 0.1uF, Capacitor_SMD:C_0603_1608Metric_Pad1.08x0.95mm_HandSolder, F.Cu at (249.3, 47.2)
- added C141: 0.1uF, Capacitor_SMD:C_0603_1608Metric_Pad1.08x0.95mm_HandSolder, F.Cu at (249.3, 49.7)
- added C142: 0.1uF, Capacitor_SMD:C_0603_1608Metric_Pad1.08x0.95mm_HandSolder, F.Cu at (249.3, 52.2)
- added C143: 0.1uF, Capacitor_SMD:C_0603_1608Metric_Pad1.08x0.95mm_HandSolder, F.Cu at (253.7, 34.7)
- added C149: 470nF, Capacitor_SMD:C_0603_1608Metric, F.Cu at (219.1, 23.9)
- added C151: 4.7uF, Capacitor_SMD:C_0603_1608Metric, F.Cu at (219.1, 26.4)
- added C152: 0.1uF, Capacitor_SMD:C_0603_1608Metric_Pad1.08x0.95mm_HandSolder, F.Cu at (224.4, 38.9)
- added C153: 0.1uF, Capacitor_SMD:C_0603_1608Metric_Pad1.08x0.95mm_HandSolder, F.Cu at (224.4, 41.5)
- added C155: 10uF, Capacitor_SMD:C_0603_1608Metric, F.Cu at (219.1, 28.9)
- added C156: 4.7uF, Capacitor_SMD:C_0603_1608Metric, F.Cu at (219.1, 31.4)
- added C160: 0.1uF, Capacitor_SMD:C_0603_1608Metric_Pad1.08x0.95mm_HandSolder, F.Cu at (290.2, -7.28)
- added C161: 0.1uF, Capacitor_SMD:C_0603_1608Metric_Pad1.08x0.95mm_HandSolder, F.Cu at (290.2, -4.77)
- added C162: 0.1uF, Capacitor_SMD:C_0603_1608Metric_Pad1.08x0.95mm_HandSolder, F.Cu at (308.3, 72.7)
- added C163: 0.1uF, Capacitor_SMD:C_0603_1608Metric_Pad1.08x0.95mm_HandSolder, F.Cu at (308.3, 75.2)
- added C164: 0.1uF, Capacitor_SMD:C_0603_1608Metric_Pad1.08x0.95mm_HandSolder, F.Cu at (308.3, 77.7)
- added C165: 0.1uF, Capacitor_SMD:C_0603_1608Metric_Pad1.08x0.95mm_HandSolder, F.Cu at (308.3, 80.2)
- added C166: 0.1uF, Capacitor_SMD:C_0603_1608Metric_Pad1.08x0.95mm_HandSolder, F.Cu at (308.3, 82.7)
- added C167: 0.1uF, Capacitor_SMD:C_0603_1608Metric_Pad1.08x0.95mm_HandSolder, F.Cu at (312.6, 72.7)
- added C168: 0.1uF, Capacitor_SMD:C_0603_1608Metric_Pad1.08x0.95mm_HandSolder, F.Cu at (312.6, 75.2)
- added C169: 0.1uF, Capacitor_SMD:C_0603_1608Metric_Pad1.08x0.95mm_HandSolder, F.Cu at (312.6, 77.7)
- added C170: 0.1uF, Capacitor_SMD:C_0603_1608Metric_Pad1.08x0.95mm_HandSolder, F.Cu at (312.6, 80.2)
- added C171: 0.1uF, Capacitor_SMD:C_0603_1608Metric_Pad1.08x0.95mm_HandSolder, F.Cu at (312.6, 82.7)
- added C172: 0.1uF, Capacitor_SMD:C_0603_1608Metric_Pad1.08x0.95mm_HandSolder, F.Cu at (317.0, 72.7)
- added C173: 0.1uF, Capacitor_SMD:C_0603_1608Metric_Pad1.08x0.95mm_HandSolder, F.Cu at (317.0, 75.2)
- added C174: 0.1uF, Capacitor_SMD:C_0603_1608Metric_Pad1.08x0.95mm_HandSolder, F.Cu at (317.0, 77.7)
- added C24: 1500pF, Capacitor_THT:C_Disc_D9.0mm_W5.0mm_P10.00mm, F.Cu at (218.9, 17.4)
- added C80: 0.1uF, Capacitor_SMD:C_0603_1608Metric_Pad1.08x0.95mm_HandSolder, F.Cu at (310.3, 92.8)
- added C81: 0.1uF, Capacitor_SMD:C_0603_1608Metric_Pad1.08x0.95mm_HandSolder, F.Cu at (310.3, 95.3)
- added C97: 0.1uF, Capacitor_SMD:C_0603_1608Metric_Pad1.08x0.95mm_HandSolder, F.Cu at (273.3, -17.3)
- added D35: BZV55B3V3, Diode_SMD:D_MiniMELF, F.Cu at (240.4, 24.3)
- added D36: BZV55B3V3, Diode_SMD:D_MiniMELF, F.Cu at (240.4, 27.6)
- added D37: BZV55B11, Diode_SMD:D_MiniMELF, F.Cu at (240.4, 31.0)
- added D38: BZV55B11, Diode_SMD:D_MiniMELF, F.Cu at (240.4, 34.3)
- added D39: LED, LED_SMD:LED_0402_1005Metric, F.Cu at (240.6, 38.7)
- added D40: BZV55C15, Diode_SMD:D_MiniMELF, F.Cu at (297.3, 105.8)
- added J*1: 1728840000, CONECTORES GRACIDA:16POS-2LINEAS-3.5PITCH, F.Cu at (333.5, 225.1)
- added J*2: 1728840000, CONECTORES GRACIDA:16POS-2LINEAS-3.5PITCH, F.Cu at (299.0, 180.3)
- added J*3: 1728840000, CONECTORES GRACIDA:16POS-2LINEAS-3.5PITCH, F.Cu at (333.5, 180.3)
- added J*4: 1728840000, CONECTORES GRACIDA:16POS-2LINEAS-3.5PITCH, F.Cu at (333.5, 209.5)
- added J11: RJ45_Wuerth_7499010211A, Connector_RJ:RJ45_Wuerth_7499010211A_Horizontal, F.Cu at (252.7, -13.5)
- added J13: 1728840000, CONECTORES GRACIDA:1728840000_33-48, F.Cu at (299.0, 166.7)
- added J14: 1728810000, CONECTORES GRACIDA:1728810000, F.Cu at (299.0, 193.9)
- added J15: 1728840000, CONECTORES GRACIDA:16POS-2LINEAS-3.5PITCH, F.Cu at (333.5, 166.7)
- added J16: 1728810000, CONECTORES GRACIDA:1728810000, F.Cu at (333.5, 193.9)
- added J18: 1728810000, CONECTORES GRACIDA:1728810000, F.Cu at (299.0, 209.5)
- added J21: 1728840000, CONECTORES GRACIDA:16POS-2LINEAS-3.5PITCH, F.Cu at (53.0, 35.0)
- added L18: 10uH, Inductor_SMD:L_0603_1608Metric_Pad1.05x0.95mm_HandSolder, F.Cu at (253.7, 15.1)
- added L20: 10uH, Inductor_SMD:L_0603_1608Metric_Pad1.05x0.95mm_HandSolder, F.Cu at (253.7, 37.2)
- added L21: 0603, Inductor_SMD:L_0603_1608Metric_Pad1.05x0.95mm_HandSolder, F.Cu at (224.4, 44.0)
- added L23: 200uH, Inductores_GSI:DLW43_MUR, F.Cu at (300.0, 217.4)
- added L25: SDR0906-3R9ML, Inductores_GSI:SDR0906-3R9ML, F.Cu at (167.0, 31.5)
- added L4: 4.7uH, Inductor_SMD:L_0805_2012Metric_Pad1.15x1.40mm_HandSolder, F.Cu at (233.0, 9.00)
- added PS1: REC15E-2412DZ, Fuentes_GSI:REC15E-2412DZ, F.Cu at (265.5, 126.1)
- added PS2: MGFW402412, Fuentes_GSI:MGFW400512, F.Cu at (234.3, 120.3)
- added R1: 2.7K, Resistor_SMD:R_0603_1608Metric, F.Cu at (286.6, -0.26)
- added R142: 2.2k, Capacitor_SMD:C_0603_1608Metric_Pad1.08x0.95mm_HandSolder, F.Cu at (310.3, 97.8)
- added R143: 2.2k, Capacitor_SMD:C_0603_1608Metric_Pad1.08x0.95mm_HandSolder, F.Cu at (310.3, 100.3)
- added R144: 2.2k, Capacitor_SMD:C_0603_1608Metric_Pad1.08x0.95mm_HandSolder, F.Cu at (310.3, 102.8)
- added R145: 2.2k, Capacitor_SMD:C_0603_1608Metric_Pad1.08x0.95mm_HandSolder, F.Cu at (310.3, 105.3)
- added R151: 4.7k, Capacitor_SMD:C_0603_1608Metric_Pad1.08x0.95mm_HandSolder, F.Cu at (314.6, 92.8)
- added R152: 4.7k, Capacitor_SMD:C_0603_1608Metric_Pad1.08x0.95mm_HandSolder, F.Cu at (314.6, 95.3)
- added R153: 4.7k, Capacitor_SMD:C_0603_1608Metric_Pad1.08x0.95mm_HandSolder, F.Cu at (314.6, 97.8)
- added R154: 4.7k, Capacitor_SMD:C_0603_1608Metric_Pad1.08x0.95mm_HandSolder, F.Cu at (314.6, 100.3)
- added R155: 4.7k, Capacitor_SMD:C_0603_1608Metric_Pad1.08x0.95mm_HandSolder, F.Cu at (314.6, 102.8)
- added R159: 1K, Resistor_SMD:R_0603_1608Metric, F.Cu at (269.1, -17.3)
- added R160: 1K, Resistor_SMD:R_0603_1608Metric, F.Cu at (269.1, -14.8)
- added R166: 160, Resistor_SMD:R_0603_1608Metric, F.Cu at (269.1, -12.3)
- added R167: 160, Resistor_SMD:R_0603_1608Metric, F.Cu at (269.1, -9.79)
- added R171: 49.9R, Resistor_SMD:R_0603_1608Metric, F.Cu at (269.1, -7.28)
- added R172: 49.9R, Resistor_SMD:R_0603_1608Metric, F.Cu at (269.1, -4.77)
- added R173: 49.9R, Resistor_SMD:R_0603_1608Metric, F.Cu at (269.1, -2.26)
- added R174: 49.9R, Resistor_SMD:R_0603_1608Metric, F.Cu at (269.1, 0.25)
- added R183: 2.2k, Capacitor_SMD:C_0603_1608Metric_Pad1.08x0.95mm_HandSolder, F.Cu at (253.7, 17.6)
- added R184: 2.2k, Capacitor_SMD:C_0603_1608Metric_Pad1.08x0.95mm_HandSolder, F.Cu at (253.7, 20.1)
- added R185: 2.2k, Capacitor_SMD:C_0603_1608Metric_Pad1.08x0.95mm_HandSolder, F.Cu at (253.7, 22.6)
- added R186: 2.2k, Capacitor_SMD:C_0603_1608Metric_Pad1.08x0.95mm_HandSolder, F.Cu at (253.7, 25.1)
- added R187: 2.2k, Capacitor_SMD:C_0603_1608Metric_Pad1.08x0.95mm_HandSolder, F.Cu at (253.7, 27.7)
- added R188: 2.2k, Capacitor_SMD:C_0603_1608Metric_Pad1.08x0.95mm_HandSolder, F.Cu at (253.7, 30.2)
- added R189: 2.2k, Capacitor_SMD:C_0603_1608Metric_Pad1.08x0.95mm_HandSolder, F.Cu at (258.0, 12.6)
- added R190: 2.2k, Capacitor_SMD:C_0603_1608Metric_Pad1.08x0.95mm_HandSolder, F.Cu at (258.0, 15.1)
- added R191: 2.2k, Capacitor_SMD:C_0603_1608Metric_Pad1.08x0.95mm_HandSolder, F.Cu at (258.0, 17.6)
- added R192: 2.2k, Capacitor_SMD:C_0603_1608Metric_Pad1.08x0.95mm_HandSolder, F.Cu at (258.0, 20.1)
- added R193: 10k, Capacitor_SMD:C_0603_1608Metric_Pad1.08x0.95mm_HandSolder, F.Cu at (258.0, 22.6)
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- renumbered C86 to C100, C103 to C101, C106 to C102, C94 to C103, C95 to C104, C102 to C105, C96 to C106, C97 to C107, C98 to C109, C99 to C110, C100 to C112, C101 to C113, C104 to C115, C105 to C116, C107 to C117, C108 to C118, C109 to C119, C110 to C120, C111 to C121, C113 to C123, C115 to C125, C11 to C13, C12 to C14, C14 to C15, C15 to C16, C13 to C17, C16 to C18, C17 to C19, C18 to C20, C19 to C22, C20 to C23, C24 to C25, C25 to C26, C26 to C27, C27 to C28, C31 to C29, C36 to C40, C37 to C41, C39 to C43, C41 to C45, C44 to C48, C45 to C49, C46 to C50, C47 to C51, C48 to C52, C49 to C53, C59 to C63, C61 to C65, C67 to C71, C68 to C72, C69 to C73, C73 to C77, C76 to C82, C77 to C83, C78 to C84, C79 to C85, C80 to C86, C81 to C87, C82 to C88, C83 to C89, C84 to C90, C85 to C91, C87 to C92, C88 to C93, C91 to C96, C92 to C98, D6 to D5, D5 to D6, D8 to D7, D7 to D8, F1 to F6, IC14 to IC4, IC16 to IC5, IC17 to IC6, IC15 to IC7, J5 to J4, J9 to J8, L9 to L10, L10 to L12, L4 to L5, L7 to L8, R6 to R10, R95 to R102, R102 to R109, R8 to R11, R103 to R110, R104 to R111, R105 to R112, R10 to R12, R133 to R136, R134 to R137, R135 to R138, R136 to R139, R11 to R14, R130 to R140, R129 to R141, R137 to R146, R138 to R147, R139 to R148, R140 to R149, R12 to R15, R141 to R156, R142 to R157, R143 to R158, R14 to R16, R146 to R161, R144 to R162, R145 to R163, R151 to R164, R148 to R165, R147 to R168, R149 to R169, R15 to R17, R150 to R170, R152 to R175, R153 to R176, R154 to R177, R155 to R178, R156 to R179, R16 to R18, R157 to R180, R158 to R181, R159 to R182, R17 to R19, R18 to R20, R35 to R37, R36 to R38, R37 to R39, R2 to R4, R38 to R40, R43 to R45, R44 to R46, R45 to R47, R46 to R48, R47 to R49, R3 to R5, R4 to R6, R56 to R63, R57 to R64, R58 to R65, R59 to R66, R61 to R68, R62 to R69, R5 to R7, R63 to R70, R64 to R71, R65 to R72, R66 to R73, R67 to R74, R68 to R75, R69 to R76, R70 to R77, R71 to R78, R72 to R79, R7 to R8, R73 to R80, R74 to R81, R76 to R83, R78 to R85, R80 to R87, R84 to R91, TH3 to TH4, TP4 to TP3, TP3 to TP4, U13 to U10, U14 to U11, U15 to U12, U16 to U13, U17 to U14, U21 to U18, U22 to U19, U6 to U3, U9 to U6, U11 to U8, U12 to U9
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Connections:
- net /SALIDA J5 y J6/!CS_MCP23S7_SS_1_J5 renamed /Processador/!CS_J5_J6
- net /SALIDA J5 y J6/DA0_Analog renamed /Processador/DAC1
- net /SALIDA J5 y J6/DA1_Analog renamed /Processador/DAC0
- net /SALIDA J5 y J6/Error_ULN_Fault_+24v renamed /Error/24v_in2
- net /SALIDA J5 y J6/IN1_MO1 renamed /Processador/MO4
- net /SALIDA J5 y J6/IN4_MO4 renamed /Processador/MO1
- net /SALIDA J5 y J6/INTA_MCP23S17_SS renamed /Processador/INTA_J5_J6
- C1 pad 2: GND -> -12V_Analog
- C10 pad 1: Net-(U4-BOOST) -> Net-(U21-BOOST)
- C10 pad 2: Net-(U4-SW) -> Net-(U21-SW)
- C100 pad 1: +3.3V -> +3.3v_Fuse
- C100 pad 2: GND -> -12V_Analog
- C101 pad 1: +3.3V -> +3.3v_Fuse
- C101 pad 2: GND -> -12V_Analog
- C102 pad 2: GND -> -12V_Analog
- C103 pad 2: GND -> -12V_Analog
- C104 pad 2: GND -> -12V_Analog
- C105 pad 2: GND -> -12V_Analog
- C106 pad 1: +1.2Vreg -> +3.3v_Fuse
- C106 pad 2: GND -> -12V_Analog
- C107 pad 2: GND -> -12V_Analog
- C109 pad 2: GND -> -12V_Analog
- C110 pad 2: GND -> -12V_Analog
- C112 pad 1: +3.3V -> +3.3v_Fuse
- C112 pad 2: GND -> -12V_Analog
- C113 pad 1: +3.3V -> +3.3v_Fuse
- C113 pad 2: GND -> -12V_Analog
- C115 pad 1: +3.3V -> +3.3v_Fuse
- C115 pad 2: GND -> -12V_Analog
- C116 pad 1: +3.3V -> +3.3v_Fuse
- C116 pad 2: GND -> -12V_Analog
- C117 pad 1: GND -> -12V_Analog
- C118 pad 2: GND -> -12V_Analog
- C119 pad 1: GND -> -12V_Analog
- C120 pad 2: GND -> -12V_Analog
- C121 pad 1: GND -> -12V_Analog
- C123 pad 1: GND -> -12V_Analog
- C125 pad 1: GND -> -12V_Analog
- C13 pad 2: Net-(U4-VFB) -> Net-(U21-VFB)
- C14 pad 2: GND -> -12V_Analog
- C17 pad 2: GND -> -12V_Analog
- C18 pad 2: GND -> -12V_Analog
- C19 pad 2: GND -> -12V_Analog
- C2 pad 2: GND -> -12V_Analog
- C20 pad 2: GND -> -12V_Analog
- C21 pad 1: +3.3V -> -12V_Analog
- C21 pad 2: GND -> Net-(PS1--Vo)
- C22 pad 2: GND -> -12V_Analog
- C23 pad 2: GND -> -12V_Analog
- C25 pad 2: GND -> -12V_Analog
- C26 pad 2: GND -> -12V_Analog
- C27 pad 2: GND -> -12V_Analog
- C28 pad 2: GND -> -12V_Analog
- C29 pad 2: GND -> -12V_Analog
- C4 pad 2: GND -> -12V_Analog
- C40 pad 2: GND -> -12V_Analog
- C41 pad 1: GND -> -12V_Analog
- C43 pad 2: GND -> -12V_Analog
- C45 pad 2: GND -> -12V_Analog
- C48 pad 1: GND -> -12V_Analog
- C49 pad 1: GND -> -12V_Analog
- C5 pad 1: Net-(U4-INTVCC) -> Net-(U21-INTVCC)
- C5 pad 2: GND -> -12V_Analog
- C50 pad 1: GND -> -12V_Analog
- C51 pad 1: GND -> -12V_Analog
- C52 pad 1: GND -> -12V_Analog
- C53 pad 1: GND -> -12V_Analog
- C6 pad 2: GND -> -12V_Analog
- C63 pad 2: GND -> -12V_Analog
- C65 pad 2: GND -> -12V_Analog
- C7 pad 2: GND -> -12V_Analog
- C71 pad 2: GND -> -12V_Analog
- C73 pad 1: /SALIDA J5 y J6/Error_LAMP_Fault_+24v -> /Error/24v_in1
- C73 pad 2: GND -> -12V_Analog
- C77 pad 2: GND -> -12V_Analog
- C8 pad 2: GND -> -12V_Analog
- C82 pad 1: GND -> -12V_Analog
- C83 pad 1: GND -> -12V_Analog
- C84 pad 1: Net-(U24-C1-) -> Net-(U21-C1-)
- C84 pad 2: Net-(U24-C1+) -> Net-(U21-C1+)
- C85 pad 1: GND -> -12V_Analog
- C86 pad 1: Net-(U24-C2-) -> Net-(U21-C2-)
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
Commit message: 26-05-26
Parts:
- removed J*1, J*2, J*3: 1728840000, CONECTORES GRACIDA:16POS-2LINEAS-3.5PITCH
- removed J13, J8: 1728840000, CONECTORES GRACIDA:1728840000_33-48
- removed J14, J16: 1728810000, CONECTORES GRACIDA:1728810000
- added TH2: B59985C120A70, TERMISTORES GRACIDA:B59985C0120A070, F.Cu at (328.8, 113.1)
- added TH3: B59985C120A70, TERMISTORES GRACIDA:B59985C0120A070, F.Cu at (328.8, 121.7)
- added TH5: B59985C120A70, TERMISTORES GRACIDA:B59985C0120A070, F.Cu at (340.4, 104.5)
- added TH7: B59985C120A70, TERMISTORES GRACIDA:B59985C0120A070, F.Cu at (340.4, 113.1)
- added TH9: B59985C120A70, TERMISTORES GRACIDA:B59985C0120A070, F.Cu at (328.8, 104.5)
- moved J15 185.0 mm to (150.1, 142.4)
- moved J18 171.6 mm to (160.8, 107.7)
- moved J21 156.7 mm to (150.1, 158.0)
- moved J6 155.1 mm to (158.5, 191.1)
- moved CN1 146.3 mm to (40.3, 191.7)
- moved J7 122.7 mm to (123.5, 191.1)
- moved J*4 87.9 mm to (355.1, 124.3)
- moved D1 86.4 mm to (284.5, 164.9), turned to -90 degrees
- moved R4 82.1 mm to (286.5, 164.9), turned to 90 degrees
- moved D2 68.1 mm to (254.0, 164.9), turned to -90 degrees
- moved R5 62.0 mm to (256.0, 164.9), turned to 90 degrees
- moved D3 60.8 mm to (223.0, 164.9), turned to -90 degrees
- moved R6 53.1 mm to (225.0, 164.9), turned to 90 degrees
- moved J9 21.4 mm to (123.5, 177.1)
- moved J3 10.8 mm to (219.8, 201.1), turned to 180 degrees
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