File: 01_IO-ASD-PLUS.kicad_pcb (KiCad board)
At the start: 2 copper layers, 180 x 158 mm, 458 parts, among them CN1 10way 1.27mm, IC4 VNI4140K, IC5 ILD206T, IC6 ILD206T, IC7 ILD206T, J1 1147330000, J11 RJ45_Wuerth_7499010211A, J15 1728840000, J18 1728810000, J2 1147330000, J21 1728840000, J3 1147330000, J4 1604470000, J6 1728840000, J7 1728840000, J9 1728840000, K1 G2RL-1-H, K2 G2RL-1-H, K3 G2RL-1-H, Q10 DMP3099L, Q11 DMP3099L, Q12 DMP3099L, Q13 DMP3099L, Q2 MMBT3904, Q3 MMBT3904, Q4 MMBT3904, Q5 MMBT3904, Q6 MMBT3904, Q7 MMBT3904, Q8 DMP3099L, Q9 DMP3099L, U1 FT900Q, U10 74LVC1G17, U11 74LVC1G17, U12 74LVC1G17, U13 74LVC1G17, U14 TSB582, U18 LM7705, U19 MCP1799T-5002H/TT, U2 LTC3646E, U21 LTC3646EMSEPBF, U22 24AA02E-OT, U23 ILD206T, U24 MCP9700Ax-ETT, U26 ILD206T, U27 ILD206T, U28 TLV9301xDBV, U29 TLV9301xDBV, U3 KF33BDT, U30 LM7705, U31 MCP1799T-5002H/TT, U33 MCP23S17_SS, U37 LTC6820, U39 TLV2371DBV, U40 TLV702475_SOT23-5, U43 ILD206T, U44 ILD206T, U45 ILD206T, U48 ILD206T, U49 ILD206T, U50 ILD206T, U6 MCP23S17_SS, U8 74LVC1G17, U9 74LVC1G17

Commit message: 05/06/26
Parts:
- removed J*4, J21: 1728840000, CONECTORES GRACIDA:16POS-2LINEAS-3.5PITCH
- added ?: , , F.Cu at (277.5, 58.3)
- added ?: , , F.Cu at (181.3, 58.3)
- added ?: , , F.Cu at (263.5, 58.3)
- added ?: , , F.Cu at (263.5, 178.3)
- added ?: , , F.Cu at (277.5, 178.3)
- added ?: , , F.Cu at (130.5, 144.1)
- added ?: , , F.Cu at (207.5, 203.3)
- added ?: , , F.Cu at (130.5, 58.3)
- added C122: 0.1uF, Capacitor_SMD:C_0603_1608Metric_Pad1.08x0.95mm_HandSolder, F.Cu at (169.5, -53.4)
- added C124: 0.1uF, Capacitor_SMD:C_0603_1608Metric_Pad1.08x0.95mm_HandSolder, F.Cu at (169.5, -50.9)
- added C30: 47uF, Capacitor_Tantalum_SMD:CP_EIA-1608-10_AVX-L_HandSolder, F.Cu at (145.0, -57.6)
- added C31: 0.1uF, Capacitor_SMD:C_0603_1608Metric_Pad1.08x0.95mm_HandSolder, F.Cu at (116.8, -53.4)
- added C32: 0.1uF, Capacitor_SMD:C_0603_1608Metric_Pad1.08x0.95mm_HandSolder, F.Cu at (116.8, -50.9)
- added C33: 0.1uF, Capacitor_SMD:C_0603_1608Metric_Pad1.08x0.95mm_HandSolder, F.Cu at (116.8, -48.4)
- added C36: 0.1uF, Capacitor_SMD:C_0603_1608Metric_Pad1.08x0.95mm_HandSolder, F.Cu at (116.8, -45.9)
- added C37: 0.1uF, Capacitor_SMD:C_0603_1608Metric_Pad1.08x0.95mm_HandSolder, F.Cu at (116.8, -43.4)
- added C38: 0.1uF, Capacitor_SMD:C_0603_1608Metric_Pad1.08x0.95mm_HandSolder, F.Cu at (116.8, -40.9)
- added C39: 0.1uF, Capacitor_SMD:C_0603_1608Metric_Pad1.08x0.95mm_HandSolder, F.Cu at (116.8, -38.4)
- added C47: 4.7uF, Capacitor_SMD:C_0603_1608Metric, F.Cu at (154.4, 214.7)
- added C56: 0.1uF, Capacitor_SMD:C_0603_1608Metric_Pad1.08x0.95mm_HandSolder, F.Cu at (112.5, -8.94)
- added C57: 0.1uF, Capacitor_SMD:C_0603_1608Metric_Pad1.08x0.95mm_HandSolder, F.Cu at (112.5, -6.43)
- added C58: 1nF, Capacitor_SMD:C_0603_1608Metric_Pad1.08x0.95mm_HandSolder, F.Cu at (147.0, -24.5)
- added C59: 0.1uF, Capacitor_SMD:C_0603_1608Metric_Pad1.08x0.95mm_HandSolder, F.Cu at (147.0, -22.0)
- added C60: 0.1uF, Capacitor_SMD:C_0603_1608Metric_Pad1.08x0.95mm_HandSolder, F.Cu at (147.0, -19.5)
- added C61: 0.1uF, Capacitor_SMD:C_0603_1608Metric_Pad1.08x0.95mm_HandSolder, F.Cu at (147.0, -17.0)
- added C62: 0.01uF, Capacitor_SMD:C_0603_1608Metric_Pad1.08x0.95mm_HandSolder, F.Cu at (147.0, -14.5)
- added C66: 0.1uF, Capacitor_SMD:C_0603_1608Metric_Pad1.08x0.95mm_HandSolder, F.Cu at (151.3, -24.5)
- added C67: 0.1uF, Capacitor_SMD:C_0603_1608Metric_Pad1.08x0.95mm_HandSolder, F.Cu at (151.3, -22.0)
- added C69: 0.1uF, Capacitor_SMD:C_0603_1608Metric_Pad1.08x0.95mm_HandSolder, F.Cu at (151.3, -19.5)
- added C70: 0.1uF, Capacitor_SMD:C_0603_1608Metric_Pad1.08x0.95mm_HandSolder, F.Cu at (151.3, -17.0)
- added C74: 0.1uF, Capacitor_SMD:C_0603_1608Metric_Pad1.08x0.95mm_HandSolder, F.Cu at (151.3, -14.5)
- added C75: 0.01uF, Capacitor_SMD:C_0603_1608Metric_Pad1.08x0.95mm_HandSolder, F.Cu at (155.7, -24.5)
- added C76: 0.1uF, Capacitor_SMD:C_0603_1608Metric_Pad1.08x0.95mm_HandSolder, F.Cu at (155.7, -22.0)
- added C78: 1uF, Capacitor_SMD:C_0603_1608Metric_Pad1.08x0.95mm_HandSolder, F.Cu at (155.7, -19.5)
- added C79: 0.1uF, Capacitor_SMD:C_0603_1608Metric_Pad1.08x0.95mm_HandSolder, F.Cu at (155.7, -17.0)
- added C94: 0.1uF, Capacitor_SMD:C_0603_1608Metric_Pad1.08x0.95mm_HandSolder, F.Cu at (154.4, -67.0)
- added C95: 0.1uF, Capacitor_SMD:C_0603_1608Metric_Pad1.08x0.95mm_HandSolder, F.Cu at (160.7, -46.4)
- added D13: LED, LED_SMD:LED_0603_1608Metric_Pad1.05x0.95mm_HandSolder, F.Cu at (79.6, 222.8)
- added D14: LED, LED_SMD:LED_0603_1608Metric_Pad1.05x0.95mm_HandSolder, F.Cu at (79.6, 220.8)
- added D15: LED, LED_SMD:LED_0603_1608Metric_Pad1.05x0.95mm_HandSolder, F.Cu at (79.6, 218.3)
- added D16: LED, LED_SMD:LED_0603_1608Metric_Pad1.05x0.95mm_HandSolder, F.Cu at (79.6, 215.6)
- added D17: LED, LED_SMD:LED_0603_1608Metric_Pad1.05x0.95mm_HandSolder, F.Cu at (143.0, 236.3)
- added D18: LED, LED_SMD:LED_0603_1608Metric_Pad1.05x0.95mm_HandSolder, F.Cu at (143.0, 238.9)
- added D19: LED, LED_SMD:LED_0603_1608Metric_Pad1.05x0.95mm_HandSolder, F.Cu at (143.0, 241.5)
- added D20: LED, LED_SMD:LED_0603_1608Metric_Pad1.05x0.95mm_HandSolder, F.Cu at (143.0, 244.1)
- added D21: LED, LED_SMD:LED_0402_1005Metric, F.Cu at (168.1, 215.5)
- added D26: BZV55B3V3, Diode_SMD:D_MiniMELF, F.Cu at (148.0, -0.30)
- added F1: SF-2410HI050T-2, Fuse:Fuse_Littelfuse-NANO2-451_453, F.Cu at (121.0, 104.4)
- added F2: SF-2410HI050T-2, Fuse:Fuse_Littelfuse-NANO2-451_453, F.Cu at (129.3, 104.4)
- added F3: SF-2410HI050T-2, Fuse:Fuse_Littelfuse-NANO2-451_453, F.Cu at (137.6, 104.4)
- added F4: SF-2410HI050T-2, Fuse:Fuse_Littelfuse-NANO2-451_453, F.Cu at (214.8, 68.6)
- added F5: SF-2410HI050T-2, Fuse:Fuse_Littelfuse-NANO2-451_453, F.Cu at (222.7, 68.6)
- added IC1: VNI4140K, Package_SO:ST_PowerSSO-24_SlugDown_ThermalVias, F.Cu at (88.9, 218.7)
- added J*1: 1728840000, CONECTORES GRACIDA:16POS-2LINEAS-3.5PITCH, F.Cu at (321.0, 184.6)
- added J12: 1728840000, CONECTORES GRACIDA:16POS-2LINEAS-3.5PITCH, F.Cu at (153.0, 160.1)
- added J14: 1728810000, CONECTORES GRACIDA:1728810000, F.Cu at (125.3, 117.6)
- added J5: 1728840000, CONECTORES GRACIDA:16POS-2LINEAS-3.5PITCH, F.Cu at (120.0, 179.6)
- added J8: Micro_SD_Card_Det1, CONECTORES GRACIDA:16POS-2LINEAS-3.5PITCH, F.Cu at (333.0, 166.6)
- added L15: 0603, Inductor_SMD:L_0603_1608Metric_Pad1.05x0.95mm_HandSolder, F.Cu at (147.0, 2.62)
- added L17: 200uH, Inductores_GSI:DLW43_MUR, F.Cu at (163.6, -52.2)
- added L6: 0603, Inductor_SMD:L_0603_1608Metric_Pad1.05x0.95mm_HandSolder, F.Cu at (116.8, -35.9)
- added L7: 10uH, Inductor_SMD:L_0603_1608Metric_Pad1.05x0.95mm_HandSolder, F.Cu at (122.0, 214.4)
- added Q1: MMBT3904, Package_TO_SOT_SMD:SOT-23, F.Cu at (143.3, -37.4)
- added R100: 10k, Resistor_SMD:R_0603_1608Metric, F.Cu at (159.8, -22.0)
- added R101: 10k, Resistor_SMD:R_0603_1608Metric, F.Cu at (159.8, -19.5)
- added R103: 1K, Resistor_SMD:R_0603_1608Metric, F.Cu at (159.8, -17.0)
- added R104: 1K, Resistor_SMD:R_0603_1608Metric, F.Cu at (159.8, -14.5)
- added R105: 0, Resistor_SMD:R_0603_1608Metric, F.Cu at (163.8, -24.5)
- added R106: 0, Resistor_SMD:R_0603_1608Metric, F.Cu at (163.8, -22.0)
- added R107: 10k, Resistor_SMD:R_0603_1608Metric, F.Cu at (163.8, -19.5)
- added R108: 1K, Resistor_SMD:R_0603_1608Metric, F.Cu at (163.8, -17.0)
- added R113: 12.3k 1%, Resistor_SMD:R_0603_1608Metric, F.Cu at (163.8, -14.5)
- added R114: 49.9R, Resistor_SMD:R_0603_1608Metric, F.Cu at (167.9, -24.5)
- added R115: 49.9R, Resistor_SMD:R_0603_1608Metric, F.Cu at (167.9, -22.0)
- added R116: 49.9R, Resistor_SMD:R_0603_1608Metric, F.Cu at (167.9, -19.5)
- added R117: 49.9R, Resistor_SMD:R_0603_1608Metric, F.Cu at (167.9, -17.0)
- added R118: 10k, Resistor_SMD:R_0603_1608Metric, F.Cu at (154.2, -64.5)
- added R119: 10k, Resistor_SMD:R_0603_1608Metric, F.Cu at (154.2, -62.0)
- added R120: 470, Resistor_SMD:R_0603_1608Metric, F.Cu at (154.2, -59.5)
- added R121: 470, Resistor_SMD:R_0603_1608Metric, F.Cu at (154.2, -57.0)
- added R122: 5.1k 1%, Resistor_SMD:R_0603_1608Metric, F.Cu at (154.2, -54.5)
- added R123: 0, Resistor_SMD:R_0603_1608Metric, F.Cu at (154.2, -52.0)
- added R124: 0, Resistor_SMD:R_0603_1608Metric, F.Cu at (154.2, -49.5)
- added R125: 0, Resistor_SMD:R_0603_1608Metric, F.Cu at (154.2, -47.0)
- added R126: 2.2k, Capacitor_SMD:C_0603_1608Metric_Pad1.08x0.95mm_HandSolder, F.Cu at (160.7, -43.9)
- added R127: 2.2k, Capacitor_SMD:C_0603_1608Metric_Pad1.08x0.95mm_HandSolder, F.Cu at (160.7, -41.4)
- added R128: 2.2k, Capacitor_SMD:C_0603_1608Metric_Pad1.08x0.95mm_HandSolder, F.Cu at (160.7, -38.9)
- added R129: 2.2k, Capacitor_SMD:C_0603_1608Metric_Pad1.08x0.95mm_HandSolder, F.Cu at (160.7, -36.3)
- added R130: 2.2k, Capacitor_SMD:C_0603_1608Metric_Pad1.08x0.95mm_HandSolder, F.Cu at (160.7, -33.8)
- added R131: 2.2k, Capacitor_SMD:C_0603_1608Metric_Pad1.08x0.95mm_HandSolder, F.Cu at (165.1, -46.4)
- added R132: 4.7k, Capacitor_SMD:C_0603_1608Metric_Pad1.08x0.95mm_HandSolder, F.Cu at (165.1, -43.9)
- added R133: 4.7k, Capacitor_SMD:C_0603_1608Metric_Pad1.08x0.95mm_HandSolder, F.Cu at (165.1, -41.4)
- added R134: 4.7k, Capacitor_SMD:C_0603_1608Metric_Pad1.08x0.95mm_HandSolder, F.Cu at (165.1, -38.9)
- added R135: 4.7k, Capacitor_SMD:C_0603_1608Metric_Pad1.08x0.95mm_HandSolder, F.Cu at (165.1, -36.3)
- added R21: 4.7k, Capacitor_SMD:C_0603_1608Metric_Pad1.08x0.95mm_HandSolder, F.Cu at (121.2, -50.9)
- added R22: 4.7k, Capacitor_SMD:C_0603_1608Metric_Pad1.08x0.95mm_HandSolder, F.Cu at (121.2, -48.4)
- added R23: 4.7k, Capacitor_SMD:C_0603_1608Metric_Pad1.08x0.95mm_HandSolder, F.Cu at (121.2, -45.9)
- added R24: 4.7k, Capacitor_SMD:C_0603_1608Metric_Pad1.08x0.95mm_HandSolder, F.Cu at (121.2, -43.4)
- added R25: 4.7k, Capacitor_SMD:C_0603_1608Metric_Pad1.08x0.95mm_HandSolder, F.Cu at (121.2, -40.9)
- added R26: 4.7k, Capacitor_SMD:C_0603_1608Metric_Pad1.08x0.95mm_HandSolder, F.Cu at (121.2, -38.4)
- added R27: 4.7k, Capacitor_SMD:C_0603_1608Metric_Pad1.08x0.95mm_HandSolder, F.Cu at (121.2, -35.9)
- added R28: 4.7k, Capacitor_SMD:C_0603_1608Metric_Pad1.08x0.95mm_HandSolder, F.Cu at (125.5, -53.4)
- added R29: 10k, Resistor_SMD:R_0603_1608Metric, F.Cu at (129.7, -50.9)
- added R3: 0 ohms, Resistor_SMD:R_0603_1608Metric_Pad0.98x0.95mm_HandSolder, F.Cu at (204.6, 166.4)
- added R30: 0R, Resistor_SMD:R_0603_1608Metric, F.Cu at (129.7, -48.4)
- added R31: 0R, Resistor_SMD:R_0603_1608Metric, F.Cu at (129.7, -45.9)
- added R33: 0R, Resistor_SMD:R_0603_1608Metric, F.Cu at (129.7, -43.4)
- added R34: 0R, Resistor_SMD:R_0603_1608Metric, F.Cu at (129.7, -40.9)
- added R35: 0R, Resistor_SMD:R_0603_1608Metric, F.Cu at (133.7, -53.4)
- added R43: 10k, Capacitor_SMD:C_0603_1608Metric_Pad1.08x0.95mm_HandSolder, F.Cu at (150.6, 213.4)
- added R44: 10k, Capacitor_SMD:C_0603_1608Metric_Pad1.08x0.95mm_HandSolder, F.Cu at (150.6, 215.9)
- added R52: 2.2k, Resistor_SMD:R_0603_1608Metric, F.Cu at (133.7, -50.9)
- added R56: 1k, Resistor_SMD:R_0603_1608Metric, F.Cu at (133.7, -48.4)
- added R57: 1k, Resistor_SMD:R_0603_1608Metric, F.Cu at (133.7, -45.9)
- added R58: 1k, Resistor_SMD:R_0603_1608Metric, F.Cu at (133.7, -43.4)
- added R59: 1k, Resistor_SMD:R_0603_1608Metric, F.Cu at (133.7, -40.9)
- added R60: 10k, Resistor_SMD:R_0603_1608Metric, F.Cu at (137.7, -53.4)
- added R61: 10, Resistor_SMD:R_0603_1608Metric, F.Cu at (137.7, -50.9)
- added R67: 0 ohms, Resistor_SMD:R_0603_1608Metric, F.Cu at (137.7, -48.4)
- added R82: 10k, Capacitor_SMD:C_0603_1608Metric_Pad1.08x0.95mm_HandSolder, F.Cu at (156.1, 233.4)
- added R84: 10k, Capacitor_SMD:C_0603_1608Metric_Pad1.08x0.95mm_HandSolder, F.Cu at (156.1, 236.0)
- added R88: 2.2k, Capacitor_SMD:C_0603_1608Metric_Pad1.08x0.95mm_HandSolder, F.Cu at (112.5, -3.92)
- added R89: 2.2k, Capacitor_SMD:C_0603_1608Metric_Pad1.08x0.95mm_HandSolder, F.Cu at (112.5, -1.41)
- added R90: 2.2k, Capacitor_SMD:C_0603_1608Metric_Pad1.08x0.95mm_HandSolder, F.Cu at (116.8, -8.94)
- added R92: 2.2k, Capacitor_SMD:C_0603_1608Metric_Pad1.08x0.95mm_HandSolder, F.Cu at (116.8, -6.43)
- added R93: 4.7k, Capacitor_SMD:C_0603_1608Metric_Pad1.08x0.95mm_HandSolder, F.Cu at (116.8, -3.92)
- added R94: 4.7k, Capacitor_SMD:C_0603_1608Metric_Pad1.08x0.95mm_HandSolder, F.Cu at (116.8, -1.41)
- added R95: 4.7k, Capacitor_SMD:C_0603_1608Metric_Pad1.08x0.95mm_HandSolder, F.Cu at (121.2, -8.94)
- added R96: 4.7k, Capacitor_SMD:C_0603_1608Metric_Pad1.08x0.95mm_HandSolder, F.Cu at (121.2, -6.43)
- added R97: 4.7k, Capacitor_SMD:C_0603_1608Metric_Pad1.08x0.95mm_HandSolder, F.Cu at (121.2, -3.92)
- added R98: 4.7k, Capacitor_SMD:C_0603_1608Metric_Pad1.08x0.95mm_HandSolder, F.Cu at (121.2, -1.41)
- added R99: 2.2k, Resistor_SMD:R_0603_1608Metric, F.Cu at (159.8, -24.5)
- added TH1: B59985C120A70, TERMISTORES GRACIDA:B59985C0120A070, F.Cu at (194.0, 60.8)
- added U15: LM7705, Package_SO:VSSOP-8_3x3mm_P0.65mm, F.Cu at (177.1, 215.4)
- added U16: MCP1799T-5002H/TT, Package_TO_SOT_SMD:SOT-23, F.Cu at (160.8, 215.4)
- added U17: ILD206T, Package_SO:SOIC-8_3.9x4.9mm_P1.27mm, F.Cu at (114.5, 3.21)
- added U20: 24AA02E-OT, Package_TO_SOT_SMD:SOT-23-5, F.Cu at (160.4, -10.8)
- added U25: ILD206T, Package_SO:SOIC-8_3.9x4.9mm_P1.27mm, F.Cu at (171.5, -44.3)
- added U32: LM7705, Package_SO:VSSOP-8_3x3mm_P0.65mm, F.Cu at (148.5, -4.24)
- added U35: MCP23S17_SS, Package_SO:SSOP-28_5.3x10.2mm_P0.65mm, F.Cu at (130.6, -4.32)
- added U41: TLV2371DBV, Package_TO_SOT_SMD:SOT-23-5, F.Cu at (156.8, 2.40)
- added U42: TLV702475_SOT23-5, Package_TO_SOT_SMD:SOT-23-5, F.Cu at (156.8, -4.22)
- added U5: MCP23S17_SS, Package_SO:SSOP-28_5.3x10.2mm_P0.65mm, F.Cu at (166.8, 224.5)
- added U7: 74LVC1G17, Package_TO_SOT_SMD:SOT-23-5, F.Cu at (146.1, 219.0)
- C103: value 10pF -> 22uF
- C104: value 10pF -> 470nF
- C106: value 0.01uF -> 4.7uF
- C11, C12: footprint Capacitor_THT:C_Rect_L26.5mm_W11.5mm_P22.50mm_MKS4 -> Capacitor_THT:C_Rect_L10.0mm_W3.0mm_P7.50mm_FKS3_FKP3
- C110, C49: value 0.1uF -> 10uF
- C111, C50: value 0.1uF -> 4.7uF
- C117, C118: value 18pF -> 0.1uF
- C40: value 47uF -> 0.1uF
- C45: value 0.1uF -> 470nF
- C63: value 470nF -> 10uF
- C65: value 4.7uF -> 0.01uF
- C71: value 10uF -> 0.1uF
- C72: value 4.7uF -> 10pF
- C73: value 0.1uF -> 10pF
- C86, C87: value 0.1uF -> 18pF
- C89: value 1nF -> 0.1uF
- C91: value 0.1uF -> 4.7uF/10v
- C93: value 0.01uF -> 150uF/10v
- C96: value 0.01uF -> 0.1uF
- D22: value LED -> PMEG2010BER
- D25: value LED -> BZV55B3V3
- D27, D28: value LED -> BZV55B11
- D30: value LED -> BZV55C15
- J11: value RJ45_Wuerth_7499010211A -> 1728840000; footprint Connector_RJ:RJ45_Wuerth_7499010211A_Horizontal -> CONECTORES GRACIDA:16POS-2LINEAS-3.5PITCH
- J15: value 1728840000 -> 8P8C_LED_Shielded; footprint CONECTORES GRACIDA:16POS-2LINEAS-3.5PITCH -> CONECTORES GRACIDA:1728810000
- J6: footprint CONECTORES GRACIDA:16POS-2LINEAS-3.5PITCH -> CONECTORES GRACIDA:1728840000_17-25
- J9: value 1728840000 -> RJ45_Wuerth_7499010211A
- L10, L12: value 10uH -> L_Iron_Small
- L2: value 3.9uH -> SDR0906-3R9ML
- L8: value 0603 -> L_Iron_Small
- Q7: value MMBT3904 -> DMP3099L
- R102: value 10k -> 1K
- R109, R110: value 10k -> 160
- R111, R112: value 10k -> 12k 1%
- R136, R137, R144, R145: value 2.2k -> 4.7k
- R146, R147, R148, R149, R195, R196: value 10k -> 4.7k
- R150, R154, R45, R46: value 4.7k -> 10k
- R151, R152, R153, R155: value 4.7k -> 10
- R156: value 2.2k -> 10
- R157, R158, R164, R175, R65: value 10k -> 10
- R159, R160, R161, R165: value 1K -> 10
- R162, R163: value 0 -> 10
- R166, R167: value 160 -> 10
- R168, R169: value 12k 1% -> 10
- R170: value 12.3k 1% -> 10
- R171, R172, R173, R174: value 49.9R -> 10
- R178: value 470 -> 10k
- R179: value 5.1k 1% -> 0R
- R180, R181: value 0 -> 0R
- R182: value 0 -> 620
- R183: value 2.2k -> 1.5K
- R184, R185, R186, R187, R188, R189, R190, R192: value 2.2k -> 0R
- R191: value 2.2k -> 120 1%
- R193, R194: value 10k -> 0R
- R197: value 4.7k -> 100
- R198, R199: value 4.7k -> 0R
- R200, R201, R202: value 4.7k -> 100K
- R203, R204, R205, R206, R207, R208, R209: value 2.2k -> 100K
- R48: value 4.7k -> 2.2k
- R49, R91: value 10k -> 2.2k
- R50, R51, R53: value 0R -> 2.2k
- R54, R55: value 0R -> 1k
- R71: value 2.2k -> 10k
- R81: value 10 -> 10k
- R87: value 0 ohms -> 2.2k
- U1: value FT900Q -> LTC3646EMSEPBF
- U13: value 74LVC1G17 -> TSB582
- U14: value TSB582 -> ULN2003A; footprint Package_DFN_QFN:DFN-8-1EP_6x5mm_P1.27mm_EP4x4mm -> Package_SO:SOIC-16W_5.3x10.2mm_P1.27mm
- U18: value LM7705 -> ILD206T
- U19: value MCP1799T-5002H/TT -> ILD206T
- U21: value LTC3646EMSEPBF -> FT900Q
- U22: value 24AA02E-OT -> MCP9700Ax-ETT
- U23: value ILD206T -> TPS2024
- U24: value MCP9700Ax-ETT -> ILD206T
- U28, U29: value TLV9301xDBV -> ILD206T
- U30: value LM7705 -> TLV9301xDBV
- U31: value MCP1799T-5002H/TT -> TLV9301xDBV
- U33: value MCP23S17_SS -> MCP1799T-5002H/TT
- U39: value TLV2371DBV -> LTC6820
- U40: value TLV702475_SOT23-5 -> MAX3232
- U43: value ILD206T -> 74LS30
- moved PS2 238.5 mm to (48.9, -29.6)
- moved J9 232.6 mm to (356.0, 184.1)
- moved U1 221.9 mm to (247.0, 62.1), turned to -90 degrees
- moved C13 218.6 mm to (248.7, 56.3)
- moved C14 213.8 mm to (253.5, 67.1), turned to 180 degrees
- moved C17 213.0 mm to (253.5, 65.1), turned to 180 degrees
- moved C1 210.0 mm to (250.5, 64.2)
- moved L3 206.3 mm to (246.5, 75.6), turned to -90 degrees
- moved C5 205.7 mm to (249.9, 67.1), turned to 0 degrees
- moved J15 202.8 mm to (162.5, -60.1)
- moved R10 202.3 mm to (246.9, 56.3)
- moved C10 201.1 mm to (246.4, 67.1), turned to 180 degrees
- moved C2 195.7 mm to (238.0, 63.0)
- moved C4 195.7 mm to (242.3, 63.0)
- moved R11 181.7 mm to (245.0, 56.3)
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Connections:
- net Net-(U14B-IN2-) renamed /Processador/Metal2
- C10 pad 1: Net-(U21-BOOST) -> Net-(U1-BOOST)
- C10 pad 2: Net-(U21-SW) -> Net-(U1-SW)
- C103 pad 1: Net-(C103-Pad1) -> Net-(U32-VOUT)
- C104 pad 1: Net-(C104-Pad1) -> Net-(U32-VOUT)
- C106 pad 1: +3.3v_Fuse -> Net-(U32-CRES)
- C107 pad 1: +1.2Vreg -> -12V_Analog
- C107 pad 2: -12V_Analog -> Net-(C107-Pad2)
- C108 pad 2: Net-(C108-Pad2) -> /Ent Especial/Error_Conn_Entrada_ESP+24v
- C110 pad 1: +1.2Vreg -> Net-(D29-A)
- C111 pad 1: Net-(C111-Pad1) -> Net-(U32-CF+)
- C111 pad 2: -12V_Analog -> Net-(U32-CF-)
- C115 pad 1: +3.3v_Fuse -> Net-(U35-~{RESET})
- C116 pad 1: +3.3v_Fuse -> +3.3v
- C117 pad 1: -12V_Analog -> Net-(U38-C1+)
- C117 pad 2: Net-(U1-XIO) -> Net-(U38-C1-)
- C118 pad 1: Net-(U1-XI/CLKIN) -> +3.3v_Fuse3
- C119 pad 1: -12V_Analog -> +3.3v_Fuse_comm
- C119 pad 2: +5V -> -12V_Analog
- C120 pad 1: +VBUS_OUT -> -12V_Analog
- C120 pad 2: -12V_Analog -> +3.3v_Fuse3
- C121 pad 2: +VBUS_IN -> Net-(U38-VS+)
- C123 pad 1: -12V_Analog -> Net-(U38-C2+)
- C123 pad 2: Net-(C123-Pad2) -> Net-(U38-C2-)
- C125 pad 1: -12V_Analog -> Net-(U40-VS+)
- C125 pad 2: Net-(J12-VBUS) -> -12V_Analog
- C126 pad 1: -12V_Analog -> Net-(U40-VS-)
- C126 pad 2: Net-(C126-Pad2) -> -12V_Analog
- C127 pad 1: -12V_Analog -> Net-(U40-C2+)
- C127 pad 2: /ENTRADAS1/Error_Conn_Entrada_+24v -> Net-(U40-C2-)
- C128 pad 1: -12V_Analog -> +3.3v_Fuse_comm
- C128 pad 2: Net-(C128-Pad2) -> -12V_Analog
- C129 pad 1: -12V_Analog -> Net-(U40-C1+)
- C129 pad 2: Net-(C129-Pad2) -> Net-(U40-C1-)
- C13 pad 2: Net-(U21-VFB) -> Net-(U1-VFB)
- C40 pad 1: +24V -> -12V_Analog
- C40 pad 2: -12V_Analog -> +24V
- C45 pad 1: +3.3v -> Net-(U15-VOUT)
- C49 pad 1: -12V_Analog -> Net-(D21-A)
- C49 pad 2: +24V -> -12V_Analog
- C5 pad 1: Net-(U21-INTVCC) -> Net-(U1-INTVCC)
- C50 pad 1: -12V_Analog -> Net-(U15-CF+)
- C50 pad 2: +24V -> Net-(U15-CF-)
- C51 pad 1: -12V_Analog -> /Error/24v_in1
- C51 pad 2: +24V -> -12V_Analog
- C53 pad 1: -12V_Analog -> Net-(C53-Pad1)
- C53 pad 2: +24V -> -12V_Analog
- C63 pad 1: Net-(U18-VOUT) -> +1.2Vreg
- C65 pad 1: Net-(U18-CRES) -> +3.3v_Fuse
- C71 pad 1: Net-(D31-A) -> Net-(U21-DAC_REFP)
- C72 pad 1: Net-(U18-CF+) -> Net-(C72-Pad1)
- C72 pad 2: Net-(U18-CF-) -> -12V_Analog
- C73 pad 1: /Error/24v_in1 -> Net-(C73-Pad1)
- C77 pad 1: Net-(C77-Pad1) -> -12V_Analog
- C77 pad 2: -12V_Analog -> Net-(C77-Pad2)
- C80 pad 1: -12V_Analog -> Net-(C80-Pad1)
- C80 pad 2: Net-(C80-Pad2) -> -12V_Analog
- C81 pad 1: -12V_Analog -> +3.3v_Fuse
- C81 pad 2: /ENTRADAS/Error_Conn_Entrada_+24v -> -12V_Analog
- C82 pad 1: -12V_Analog -> +3.3v_Fuse
- C82 pad 2: Net-(C82-Pad2) -> -12V_Analog
- C83 pad 1: -12V_Analog -> +3.3V
- C83 pad 2: Net-(C83-Pad2) -> -12V_Analog
- C84 pad 1: Net-(U21-C1-) -> +3.3v_Fuse
- C84 pad 2: Net-(U21-C1+) -> -12V_Analog
- C85 pad 1: -12V_Analog -> +3.3v_Fuse
- C85 pad 2: +3.3V -> -12V_Analog
- C86 pad 1: Net-(U21-C2-) -> -12V_Analog
- C88 pad 2: Net-(U21-V-) -> +5V
- C89 pad 1: Net-(CN1-10) -> +VBUS_OUT
- C90 pad 1: +3.3v_Fuse -> -12V_Analog
- C90 pad 2: -12V_Analog -> +VBUS_IN
- C91 pad 1: DBG_5V -> +VBUS_IN
- C92 pad 1: +1.2Vreg -> -12V_Analog
- C92 pad 2: -12V_Analog -> Net-(C92-Pad2)
- C93 pad 1: +1.2Vreg -> +VBUS_OUT
- C96 pad 1: +3.3v_Fuse -> -12V_Analog
- C96 pad 2: -12V_Analog -> /ENTRADAS1/Error_Conn_Entrada_+24v
- C97 pad 1: +3.3V -> -12V_Analog
- C97 pad 2: -12V_Analog -> Net-(C97-Pad2)
- C98 pad 1: +3.3v_Fuse -> -12V_Analog
- C98 pad 2: -12V_Analog -> /ENTRADAS2/Error_Conn_Entrada_+24v
- D22 pad 1: Net-(D22-K) -> +5V
- D22 pad 2: Net-(D22-A) -> DBG_5V
- D23 pad 2: Net-(D23-A) -> +VBUS_IN
- D24 pad 2: Net-(D24-A) -> +VBUS_OUT
- D25 pad 1: Net-(D25-K) -> /Ent Especial/AN1_POT
- D25 pad 2: Net-(D25-A) -> -12V_Analog
- D27 pad 2: Net-(D27-A) -> -12V_Analog
- D28 pad 2: Net-(D28-A) -> -12V_Analog
- D30 pad 1: Net-(D29-K) -> Net-(D30-K)
- D30 pad 2: Net-(D30-A) -> -12V_Analog
- J11 pad 1: Net-(J11-TD+) -> /ENTRADAS1/Error_Conn_Entrada_+24v
- J11 pad 11: Net-(U1-ENET_LED0/GPIO4) -> -12V_Analog
- J11 pad 12: Net-(J11-Pad12) -> -12V_Analog
- J11 pad 2: Net-(J11-TD-) -> Net-(J11-Pad2)
- J11 pad 3: Net-(J11-RD+) -> /ENTRADAS1/Error_Conn_Entrada_+24v
- J11 pad 4: +3.3V -> /ENTRADAS1/Error_Conn_Entrada_+24v
- J11 pad 5: +3.3V -> Net-(J11-Pad5)
- J11 pad 6: Net-(J11-RD-) -> /ENTRADAS1/Error_Conn_Entrada_+24v
- J11 pad 7: unconnected-(J11-NC-Pad7) -> Net-(J11-Pad7)
- J11 pad 8: -12V_Analog -> /ENTRADAS1/Error_Conn_Entrada_+24v
- J11 pad 9: Net-(J11-Pad9) -> -12V_Analog
- J15 pad 1: (no net) -> Net-(T1-SA)
- J15 pad 10: (no net) -> /Serial_Comm/Led_ctrl/LED1_A
- J15 pad 2: (no net) -> Net-(T1-SB)
- J15 pad 3: (no net) -> Net-(U40-T2OUT)
- J15 pad 4: (no net) -> unconnected-(J15-Pad4)
- J15 pad 5: (no net) -> unconnected-(J15-Pad5)
- J15 pad 6: (no net) -> /Serial_Comm/Led_ctrl/INT
- J15 pad 7: (no net) -> +24V
- J15 pad 8: (no net) -> -12V_Analog
- J15 pad 9: (no net) -> /Serial_Comm/Led_ctrl/LED1_C
- J7 pad 1: (no net) -> /ENTRADAS/Error_Conn_Entrada_+24v
- J7 pad 10: (no net) -> Net-(J7-Pad10)
- J7 pad 11: (no net) -> -12V_Analog
- J7 pad 12: (no net) -> -12V_Analog
- J7 pad 13: (no net) -> Net-(J7-Pad13)
- J7 pad 14: (no net) -> -12V_Analog
- J7 pad 15: (no net) -> Net-(J7-Pad15)
- J7 pad 16: (no net) -> -12V_Analog
- J7 pad 2: (no net) -> Net-(J7-Pad2)
- J7 pad 3: (no net) -> /ENTRADAS/Error_Conn_Entrada_+24v
- J7 pad 4: (no net) -> /ENTRADAS/Error_Conn_Entrada_+24v
- J7 pad 5: (no net) -> Net-(J7-Pad5)
- J7 pad 6: (no net) -> /ENTRADAS/Error_Conn_Entrada_+24v
- J7 pad 7: (no net) -> Net-(J7-Pad7)
- J7 pad 8: (no net) -> /ENTRADAS/Error_Conn_Entrada_+24v
- J7 pad 9: (no net) -> -12V_Analog
- J9 pad 1: (no net) -> Net-(J9-TD+)
- J9 pad 10: (no net) -> Net-(U21-ENET_LED1/GPIO5)
- J9 pad 11: (no net) -> Net-(U21-ENET_LED0/GPIO4)
- J9 pad 12: (no net) -> Net-(J9-Pad12)
- J9 pad 2: (no net) -> Net-(J9-TD-)
- J9 pad 3: (no net) -> Net-(J9-RD+)
- J9 pad 4: (no net) -> +3.3V
- J9 pad 5: (no net) -> +3.3V
- J9 pad 6: (no net) -> Net-(J9-RD-)
- J9 pad 7: (no net) -> unconnected-(J9-NC-Pad7)
- J9 pad 8: (no net) -> -12V_Analog
- J9 pad 9: (no net) -> Net-(J9-Pad9)
- L10 pad 1: /Error/24v_in1 -> -12V_Analog
- L10 pad 2: Net-(C77-Pad1) -> Net-(L10-Pad2)
- L12 pad 1: Net-(C82-Pad2) -> Net-(J10-VBUS)
- L12 pad 2: Net-(C83-Pad2) -> +VBUS_OUT
- L2 pad 2: +24V -> (no net)
- L3 pad 1: Net-(U21-SW) -> Net-(U1-SW)
- L8 pad 1: Net-(U18-VOUT) -> /ENTRADAS/Error_Conn_Entrada_+24v
- L8 pad 2: Net-(U14A-VCC-) -> Net-(C56-Pad2)
- Q10 pad 3: Net-(J6-ICM) -> Net-(J5-FREI)
- Q11 pad 3: Net-(J6-FREI) -> Net-(J5-FUR)
- Q12 pad 3: Net-(J6-FUR) -> Net-(J5-FUL)
- Q7 pad 1: Net-(Q7-B) -> Net-(Q1-C)
- Q7 pad 2: -12V_Analog -> +24V
- Q7 pad 3: Net-(Q13-G) -> Net-(J5-OUT2)
- Q8 pad 3: Net-(J6-OUT2) -> Net-(J5-MZ)
- Q9 pad 3: Net-(J6-MZ) -> Net-(J5-ICM)
- R10 pad 2: Net-(U21-RT) -> Net-(U1-RT)
- R102 pad 1: Net-(U14A-IN1+) -> Net-(U20-SCL)
- R102 pad 2: /Processador/DAC1 -> +3.3V
- R109 pad 1: /Error/24v_in1 -> Net-(J9-Pad9)
- R109 pad 2: Net-(D27-A) -> +3.3V
- R11 pad 1: Net-(U21-INTVCC) -> Net-(U1-INTVCC)
- R11 pad 2: Net-(U21-PGOOD) -> Net-(U1-PGOOD)
- R110 pad 1: /Error/24v_in1 -> Net-(J9-Pad12)
- R110 pad 2: Net-(D28-A) -> +3.3V
- R111 pad 1: /Error/24v_in1 -> Net-(U21-HRREF)
- R111 pad 2: Net-(D29-A) -> -12V_Analog
- R112 pad 1: /Error/24v_in1 -> Net-(U21-DRREF)
- R112 pad 2: Net-(D30-A) -> -12V_Analog
- R136 pad 1: -12V_Analog -> +3.3V
- R136 pad 2: Net-(IC5-A_2) -> /ENTRADAS1/opto_out4
- R137 pad 1: Net-(J8-ST) -> +3.3V
- R137 pad 2: Net-(IC5-A_1) -> /ENTRADAS1/opto_out6
- R138 pad 2: Net-(IC6-A_2) -> Net-(U27-A_1)
- R139 pad 2: Net-(IC6-A_1) -> Net-(U27-A_2)
- R140 pad 2: Net-(U23-A_1) -> Net-(U28-A_1)
- R141 pad 2: Net-(U23-A_2) -> Net-(U28-A_2)
- R142 pad 2: Net-(U26-A_1) -> Net-(U29-A_1)
- R143 pad 2: Net-(U26-A_2) -> Net-(U29-A_2)
- R144 pad 1: Net-(J9-10) -> +3.3V
- R144 pad 2: Net-(U27-A_1) -> /ENTRADAS2/opto_out1
- R145 pad 1: Net-(J9-7) -> +3.3V
- R145 pad 2: Net-(U27-A_2) -> /ENTRADAS2/opto_out3
- R146 pad 1: Net-(IC5-E_1) -> +3.3V
- R146 pad 2: -12V_Analog -> /ENTRADAS2/opto_out2
- R147 pad 1: Net-(IC5-E_2) -> +3.3V
- R147 pad 2: -12V_Analog -> /ENTRADAS2/opto_out5
- R148 pad 1: Net-(IC6-E_1) -> +3.3V
- R148 pad 2: -12V_Analog -> /ENTRADAS2/opto_out4
- R149 pad 1: Net-(IC6-E_2) -> +3.3V
- R149 pad 2: -12V_Analog -> /ENTRADAS2/opto_out6
- R150 pad 1: +3.3V -> -12V_Analog
- R150 pad 2: /ENTRADAS/opto_out1 -> /Ent Especial/AN1_POT
- R151 pad 1: +3.3V -> Net-(R151-Pad1)
- R151 pad 2: /ENTRADAS/opto_out3 -> /Ent Especial/AN1_POT
- R152 pad 1: +3.3V -> Net-(R151-Pad1)
- R152 pad 2: /ENTRADAS/opto_out2 -> Net-(R152-Pad2)
- R153 pad 1: +3.3V -> Net-(R153-Pad1)
- R153 pad 2: /ENTRADAS/opto_out5 -> Net-(R152-Pad2)
- R154 pad 1: +3.3V -> -12V_Analog
- R154 pad 2: /ENTRADAS/opto_out4 -> /Ent Especial/AN0_POT
- R155 pad 1: +3.3V -> Net-(R155-Pad1)
- R155 pad 2: /ENTRADAS/opto_out6 -> /Ent Especial/AN0_POT
- R156 pad 1: Net-(CN1-10) -> Net-(R156-Pad1)
- R156 pad 2: +3.3V -> Net-(R153-Pad1)
- R157 pad 1: +3.3v_Fuse -> Net-(R155-Pad1)
- R157 pad 2: Net-(J10-DET) -> Net-(R157-Pad2)
- R158 pad 1: Net-(U1-STESTRESTN) -> Net-(R158-Pad1)
- R158 pad 2: -12V_Analog -> Net-(U30--)
- R159 pad 1: Net-(U1-I2C1_SCL/GPIO46) -> Net-(R159-Pad1)
- R159 pad 2: +3.3V -> Net-(R157-Pad2)
- R160 pad 1: Net-(U1-I2C1_SDA/GPIO47) -> Net-(D27-K)
- R160 pad 2: +3.3V -> Net-(U30-+)
- R161 pad 1: +VBUS_IN -> Net-(R158-Pad1)
- R161 pad 2: Net-(U1-VBUS_DTC/GPIO3) -> Net-(R156-Pad1)
- R162 pad 1: Net-(C103-Pad1) -> Net-(R162-Pad1)
- R162 pad 2: Net-(U1-RTC_XI/RTC_CLKIN) -> Net-(R158-Pad1)
- R163 pad 1: Net-(C104-Pad1) -> Net-(R163-Pad1)
- R163 pad 2: Net-(U1-RTC_XIO) -> Net-(R159-Pad1)
- R164 pad 1: +3.3v_Fuse -> +12V
- R164 pad 2: Net-(U1-DAC_REFP) -> Net-(R164-Pad2)
- R165 pad 1: +VBUS_OUT -> Net-(R164-Pad2)
- R165 pad 2: Net-(U1-VBUS__DISCHG/_GPIO0) -> Net-(R162-Pad1)
- R166 pad 1: Net-(J11-Pad9) -> Net-(R162-Pad1)
- R166 pad 2: +3.3V -> -12V_Analog
- R167 pad 1: Net-(J11-Pad12) -> Net-(R167-Pad1)
- R167 pad 2: +3.3V -> Net-(U31--)
- R168 pad 1: Net-(U1-HRREF) -> Net-(R162-Pad1)
- R169 pad 1: Net-(U1-DRREF) -> Net-(D28-K)
- R169 pad 2: -12V_Analog -> Net-(U31-+)
- R17 pad 1: Net-(U21-VFB) -> Net-(U1-VFB)
- R170 pad 1: Net-(U1-EREFSET) -> Net-(R167-Pad1)
- R170 pad 2: -12V_Analog -> Net-(R163-Pad1)
- R171 pad 1: Net-(C111-Pad1) -> Net-(R171-Pad1)
- R171 pad 2: Net-(J11-RD-) -> Net-(R167-Pad1)
- R172 pad 1: Net-(C111-Pad1) -> +12V
- R172 pad 2: Net-(J11-RD+) -> Net-(R172-Pad2)
- R173 pad 1: Net-(C108-Pad2) -> Net-(R172-Pad2)
- R173 pad 2: Net-(J11-TD-) -> Net-(R171-Pad1)
- R174 pad 1: Net-(C108-Pad2) -> Net-(R171-Pad1)
- R174 pad 2: Net-(J11-TD+) -> -12V_Analog
- R175 pad 1: /USB/USB_Power_Switcher -> Net-(R171-Pad1)
- R175 pad 2: +3.3V -> -12V_Analog
- R178 pad 1: Net-(D34-K) -> Net-(U35-~{RESET})
- R178 pad 2: -12V_Analog -> +3.3v
- R179 pad 1: Net-(P1-CC) -> +3.3v
- R179 pad 2: -12V_Analog -> Net-(U35-A1)
- R18 pad 2: Net-(U21-VFB) -> Net-(U1-VFB)
- R180 pad 1: -12V_Analog -> +3.3v
- R180 pad 2: Net-(P1-GND-PadA1) -> Net-(U35-A0)
- R181 pad 1: -12V_Analog -> Net-(U35-A0)
- R181 pad 2: Net-(J12-Shield) -> -12V_Analog
- R182 pad 1: -12V_Analog -> /Serial_Comm/600mA
- R182 pad 2: Net-(P1-SHIELD) -> -12V_Analog
- R183 pad 1: -12V_Analog -> /Serial_Comm/+2.0v
- R183 pad 2: Net-(IC10-A_2) -> /Serial_Comm/600mA
- R184 pad 1: Net-(J13-ST) -> Net-(U39-PHA)
- R184 pad 2: Net-(IC10-A_1) -> +3.3v_Fuse3
- R185 pad 1: Net-(J13-AO) -> Net-(U39-POL)
- R185 pad 2: Net-(IC11-A_2) -> +3.3v_Fuse3
- R186 pad 1: Net-(J13-AK) -> Net-(U39-PHA)
- R186 pad 2: Net-(IC11-A_1) -> -12V_Analog
- R187 pad 1: Net-(J15-5) -> Net-(U39-POL)
- R187 pad 2: Net-(U43-A_1) -> -12V_Analog
- R188 pad 1: Net-(J15-2) -> -12V_Analog
- R188 pad 2: Net-(U43-A_2) -> Net-(U39-SLOW)
- R189 pad 2: Net-(U44-A_1) -> +3.3v_Fuse3
- R190 pad 1: Net-(J15-12) -> Net-(U39-SLOW)
- R190 pad 2: Net-(U44-A_2) -> +3.3v_Fuse3
- R191 pad 1: Net-(J15-10) -> Net-(T1-AB)
- R191 pad 2: Net-(U45-A_1) -> Net-(T1-AA)
- R192 pad 1: Net-(J15-7) -> Net-(U40-T2OUT)
- R192 pad 2: Net-(U45-A_2) -> Net-(J14-X8)
- R193 pad 1: Net-(IC10-E_1) -> /Serial_Comm/Led_ctrl/INT
- R193 pad 2: -12V_Analog -> Net-(J14-X9)
- R195 pad 1: Net-(IC11-E_1) -> +3.3v
- R195 pad 2: -12V_Analog -> /Processador/INT_FT812
- R196 pad 1: Net-(IC11-E_2) -> +3.3v
- R196 pad 2: -12V_Analog -> /Processador/INT_FT812
- R197 pad 1: +3.3V -> /Serial_Comm/Led_ctrl/LED1_C
- R197 pad 2: /ENTRADAS1/opto_out1 -> Net-(R197-Pad2)
- R198 pad 1: +3.3V -> Net-(U41--)
- R198 pad 2: /ENTRADAS1/opto_out3 -> Net-(R197-Pad2)
- R199 pad 1: +3.3V -> +24V
- R199 pad 2: /ENTRADAS1/opto_out2 -> Net-(D30-K)
- R200 pad 1: +3.3V -> Net-(U41-+)
- R200 pad 2: /ENTRADAS1/opto_out5 -> /Serial_Comm/Led_ctrl/INT
- R201 pad 1: +3.3V -> Net-(U41--)
- R201 pad 2: /ENTRADAS1/opto_out4 -> /Serial_Comm/Led_ctrl/INT
- R202 pad 1: +3.3V -> +24V
- R202 pad 2: /ENTRADAS1/opto_out6 -> Net-(R202-Pad2)
- R203 pad 1: -12V_Analog -> Net-(R202-Pad2)
- R203 pad 2: Net-(IC15-A_2) -> Net-(U41--)
- R204 pad 1: Net-(J15-ST) -> Net-(R204-Pad1)
- R204 pad 2: Net-(IC15-A_1) -> Net-(U41--)
- R205 pad 1: Net-(J15-AO) -> Net-(R204-Pad1)
- R205 pad 2: Net-(IC16-A_2) -> -12V_Analog
- R206 pad 1: Net-(J15-AK) -> +24V
- R206 pad 2: Net-(IC16-A_1) -> Net-(R206-Pad2)
- R207 pad 1: Net-(J21-5) -> Net-(R206-Pad2)
- R207 pad 2: Net-(U48-A_1) -> Net-(U41-+)
- R208 pad 1: Net-(J21-2) -> Net-(R208-Pad1)
- R208 pad 2: Net-(U48-A_2) -> Net-(U41-+)
- R209 pad 1: Net-(J21-15) -> Net-(R208-Pad1)
- R209 pad 2: Net-(U49-A_1) -> -12V_Analog
- R45 pad 2: /Processador/MO4 -> Net-(D15-K)
- R46 pad 2: /Processador/MO3 -> Net-(D16-K)
- R48 pad 1: -12V_Analog -> Net-(Q1-C)
- R48 pad 2: /Processador/MO1 -> +24V
- R49 pad 1: Net-(U6-~{RESET}) -> Net-(Q2-C)
- R49 pad 2: +3.3v -> +24V
- R50 pad 1: +3.3v -> Net-(Q3-C)
- R50 pad 2: -12V_Analog -> +24V
- R51 pad 1: Net-(U6-A0) -> Net-(Q10-G)
- R51 pad 2: +3.3v -> +24V
- R53 pad 1: -12V_Analog -> Net-(Q12-G)
- R53 pad 2: Net-(U6-A2) -> +24V
- R54 pad 1: Net-(U6-A1) -> -12V_Analog
- R54 pad 2: +3.3v -> Net-(J5-OUT2)
- R55 pad 1: -12V_Analog -> Net-(J5-ICM)
- R55 pad 2: Net-(U6-A0) -> -12V_Analog
- R63 pad 2: Net-(D22-K) -> Net-(J5-DA0)
- R65 pad 1: -12V_Analog -> Net-(U13A-OUT1)
- R65 pad 2: Net-(D24-K) -> Net-(J5-DA0)
- R71 pad 1: Net-(Q11-G) -> Net-(U13B-IN2+)
- R71 pad 2: +24V -> /Processador/DAC0
- R80 pad 1: -12V_Analog -> Net-(U13A-IN1+)
- R80 pad 2: Net-(J6-DA1) -> /Processador/DAC1
- R81 pad 1: Net-(U14B-OUT2) -> /Error/24v_in1
- R81 pad 2: Net-(J6-DA1) -> Net-(D17-A)
- R83 pad 1: -12V_Analog -> /Error/24v_in1
- R83 pad 2: Net-(J6-DA0) -> Net-(D19-A)
- R87 pad 1: Net-(U14A-VCC-) -> Net-(J7-Pad5)
- R87 pad 2: Net-(U14A-EP) -> Net-(U17-A_1)
- R91 pad 1: Net-(U14B-IN2+) -> Net-(J7-Pad15)
- R91 pad 2: /Processador/DAC0 -> Net-(U19-A_1)
- TH2 pad 1: +24V -> Net-(C56-Pad2)
- TH2 pad 2: Net-(C77-Pad1) -> +24V
- TH3 pad 1: Net-(C80-Pad2) -> Net-(C95-Pad2)
- TH4 pad 1: +24V -> Net-(C97-Pad2)
- TH4 pad 2: Net-(C83-Pad2) -> +24V
- TH5 pad 1: Net-(C126-Pad2) -> Net-(C107-Pad2)
- U1 pad 1: /Processador/MO2 -> -12V_Analog
- U1 pad 10: unconnected-(U1-SD_WP/GPIO26-Pad10) -> +24V
- U1 pad 11: /Port Expansor/SCK_SPI -> Net-(U1-SW)
- U1 pad 12: unconnected-(U1-SPIM_SS0/GPIO28-Pad12) -> Net-(U1-BOOST)
- U1 pad 13: /Port Expansor/MOSI_SPI -> Net-(U1-INTVCC)
- U1 pad 14: /Port Expansor/MISO_SPI -> -12V_Analog
- U1 pad 15: unconnected-(U1-SPIM_IO2/GPIO31-Pad15) -> /FUENTES/VRUN_U6
- U1 pad 16: unconnected-(U1-SPIM_IO3/GPIO32-Pad16) -> +24V
- U1 pad 17: /Processador/!CS_Exp -> -12V_Analog
- U1 pad 2: /Processador/MO3 -> Net-(U1-VFB)
- U1 pad 3: Net-(J10-CLK) -> Net-(U1-INTVCC)
- U1 pad 4: Net-(J10-CMD) -> Net-(U1-RT)
- U1 pad 5: Net-(J10-DAT3/CD) -> +10V
- U1 pad 6: Net-(J10-DAT2) -> Net-(U1-PGOOD)
- U1 pad 7: Net-(J10-DAT1) -> -12V_Analog
- U1 pad 8: Net-(J10-DAT0) -> unconnected-(U1-NC-Pad8)
- U1 pad 9: Net-(J10-DET) -> +24V
- U10 pad 2: Net-(U6-GPB4) -> Net-(U5-GPB2)
- U10 pad 5: unconnected-(U10-VCC-Pad5) -> +5V
- U11 pad 2: Net-(U6-GPB2) -> Net-(U5-GPB0)
- U12 pad 2: Net-(U6-GPB0) -> Net-(U5-GPB1)
- U13 pad 1: unconnected-(U13-NC-Pad1) -> Net-(U13A-OUT1)
- U13 pad 2: Net-(U6-GPB1) -> Net-(U13A-IN1-)
- U13 pad 3: -12V_Analog -> Net-(U13A-IN1+)
- U13 pad 4: Net-(Q7-B) -> Net-(U13A-VCC-)
- U13 pad 5: +5V -> Net-(U13B-IN2+)
- U14 pad 1: Net-(U14A-OUT1) -> Net-(U14-I1)
- U14 pad 3: Net-(U14A-IN1+) -> Net-(U14-I3)
- U14 pad 4: Net-(U14A-VCC-) -> Net-(U14-I4)
- U14 pad 5: Net-(U14B-IN2+) -> /Processador/Metal1
- U14 pad 7: Net-(U14B-OUT2) -> Net-(U14-I7)
- U14 pad 8: +12V -> -12V_Analog
- U14 pad 9: Net-(U14A-EP) -> /Error/24v_in2
- U18 pad 1: Net-(U18-CF+) -> Net-(U18-A_1)
- U18 pad 4: Net-(D31-A) -> -12V_Analog
- U18 pad 6: Net-(U18-VOUT) -> /ENTRADAS/opto_out4
- U18 pad 7: Net-(U18-CRES) -> -12V_Analog
- U18 pad 8: Net-(U18-CF-) -> /ENTRADAS/opto_out3
- U19 pad 1: -12V_Analog -> Net-(U19-A_1)
- U19 pad 2: Net-(D31-A) -> -12V_Analog
- U19 pad 3: +12V -> Net-(U19-A_2)
- U21 pad 1: -12V_Analog -> /Processador/MO2
- U21 pad 10: +24V -> unconnected-(U21-SD_WP/GPIO26-Pad10)
- U21 pad 11: Net-(U21-SW) -> /Port Expansor/SCK_SPI
- U21 pad 12: Net-(U21-BOOST) -> unconnected-(U21-SPIM_SS0/GPIO28-Pad12)
- U21 pad 13: Net-(U21-INTVCC) -> /Port Expansor/MOSI_SPI
- U21 pad 14: -12V_Analog -> /Port Expansor/MISO_SPI
- U21 pad 15: /FUENTES/VRUN_U6 -> unconnected-(U21-SPIM_IO2/GPIO31-Pad15)
- U21 pad 16: +24V -> unconnected-(U21-SPIM_IO3/GPIO32-Pad16)
- U21 pad 2: Net-(U21-VFB) -> /Processador/MO3
- U21 pad 3: Net-(U21-INTVCC) -> Net-(J8-CLK)
- U21 pad 4: Net-(U21-RT) -> Net-(J8-CMD)
- U21 pad 5: +10V -> Net-(J8-DAT3/CD)
- U21 pad 6: Net-(U21-PGOOD) -> Net-(J8-DAT2)
- U21 pad 7: -12V_Analog -> Net-(J8-DAT1)
- U21 pad 8: unconnected-(U21-NC-Pad8) -> Net-(J8-DAT0)
- U21 pad 9: +24V -> Net-(J8-DET)
- U22 pad 1: Net-(U1-I2C1_SCL/GPIO46) -> +3.3V
- U22 pad 2: -12V_Analog -> Net-(U21-ADC1/CAM_XCLK/GPIO6)
- U22 pad 3: Net-(U1-I2C1_SDA/GPIO47) -> -12V_Analog
- U22 pad 4: +3.3V -> (no net)
- U22 pad 5: unconnected-(U22-NC-Pad5) -> (no net)
- U23 pad 1: Net-(U23-A_1) -> (no net)
- U23 pad 2: -12V_Analog -> (no net)
- U23 pad 3: Net-(U23-A_2) -> (no net)
- U23 pad 4: -12V_Analog -> (no net)
- U23 pad 5: -12V_Analog -> (no net)
- U23 pad 6: /ENTRADAS/opto_out2 -> (no net)
- U23 pad 7: -12V_Analog -> (no net)
- U23 pad 8: /ENTRADAS/opto_out1 -> (no net)
- U24 pad 1: +3.3V -> Net-(U24-A_1)
- U24 pad 2: Net-(U1-ADC1/CAM_XCLK/GPIO6) -> -12V_Analog
- U24 pad 3: -12V_Analog -> Net-(U24-A_2)
- U26 pad 6: /ENTRADAS/opto_out4 -> /ENTRADAS1/opto_out6
- U26 pad 8: /ENTRADAS/opto_out3 -> /ENTRADAS1/opto_out5
- U27 pad 6: /ENTRADAS/opto_out6 -> /ENTRADAS2/opto_out2
- U27 pad 8: /ENTRADAS/opto_out5 -> /ENTRADAS2/opto_out1
- U28 pad 1: Net-(R224-Pad1) -> Net-(U28-A_1)
- U28 pad 2: Net-(U28-V-) -> -12V_Analog
- U28 pad 3: Net-(U28-+) -> Net-(U28-A_2)
- U28 pad 4: Net-(U28--) -> -12V_Analog
- U28 pad 5: +12V -> -12V_Analog
- U29 pad 1: Net-(R228-Pad1) -> Net-(U29-A_1)
- U29 pad 2: Net-(U28-V-) -> -12V_Analog
- U29 pad 3: Net-(U29-+) -> Net-(U29-A_2)
- U29 pad 4: Net-(U29--) -> -12V_Analog
- U29 pad 5: +12V -> -12V_Analog
- U30 pad 1: Net-(U30-CF+) -> Net-(R151-Pad1)
- U30 pad 2: -12V_Analog -> Net-(U30-V-)
- U30 pad 3: Net-(U30-SD) -> Net-(U30-+)
- U30 pad 4: Net-(D39-A) -> Net-(U30--)
- U30 pad 5: -12V_Analog -> +12V
- U30 pad 6: Net-(U30-VOUT) -> (no net)
- U30 pad 7: Net-(U30-CRES) -> (no net)
- U30 pad 8: Net-(U30-CF-) -> (no net)
- U31 pad 1: -12V_Analog -> Net-(R155-Pad1)
- U31 pad 2: Net-(D39-A) -> Net-(U30-V-)
- U31 pad 3: +12V -> Net-(U31-+)
- U33 pad 1: /ENTRADAS2/opto_out2 -> -12V_Analog
- U33 pad 10: -12V_Analog -> (no net)
- U33 pad 11: /Port Expansor/!CS_SPI -> (no net)
- U33 pad 12: /Port Expansor/SCK_SPI -> (no net)
- U33 pad 13: /Port Expansor/MOSI_SPI -> (no net)
- U33 pad 14: /Port Expansor/MISO_SPI -> (no net)
- U33 pad 15: Net-(U33-A0) -> (no net)
- U33 pad 16: Net-(U33-A1) -> (no net)
- U33 pad 17: -12V_Analog -> (no net)
- U33 pad 18: Net-(U33-~{RESET}) -> (no net)
- U33 pad 19: /Port Expansor/INTB -> (no net)
- U33 pad 2: /ENTRADAS2/opto_out4 -> Net-(D29-A)
- U33 pad 20: /Port Expansor/INTA -> (no net)
- U33 pad 21: /ENTRADAS1/opto_out5 -> (no net)
- U33 pad 22: /ENTRADAS1/opto_out6 -> (no net)
- U33 pad 23: /ENTRADAS/opto_out1 -> (no net)
- U33 pad 24: /ENTRADAS/opto_out3 -> (no net)
- U33 pad 25: /ENTRADAS/opto_out2 -> (no net)
- U33 pad 26: /ENTRADAS/opto_out4 -> (no net)
- U33 pad 27: /ENTRADAS/opto_out5 -> (no net)
- U33 pad 28: /ENTRADAS/opto_out6 -> (no net)
- U33 pad 3: /ENTRADAS2/opto_out5 -> +12V
- U33 pad 4: /ENTRADAS2/opto_out6 -> (no net)
- U33 pad 5: /ENTRADAS1/opto_out1 -> (no net)
- U33 pad 6: /ENTRADAS1/opto_out3 -> (no net)
- U33 pad 7: /ENTRADAS1/opto_out2 -> (no net)
- U33 pad 8: /ENTRADAS1/opto_out4 -> (no net)
- U33 pad 9: +3.3v -> (no net)
- U39 pad 1: Net-(R270-Pad2) -> +3.3v_Fuse3
- U39 pad 2: -12V_Analog -> /Port Expansor/MOSI_SPI
- U39 pad 3: Net-(U39-+) -> /Port Expansor/MISO_SPI
- U39 pad 4: Net-(U39--) -> /Port Expansor/SCK_SPI
- U39 pad 5: Net-(D40-K) -> /Processador/SPIM_SS
- U40 pad 1: unconnected-(U40-IN-Pad1) -> Net-(U40-C1+)
- U40 pad 2: unconnected-(U40-GND-Pad2) -> Net-(U40-VS+)
- U40 pad 3: unconnected-(U40-EN-Pad3) -> Net-(U40-C1-)
- U40 pad 4: unconnected-(U40-NC-Pad4) -> Net-(U40-C2+)
- U40 pad 5: unconnected-(U40-OUT-Pad5) -> Net-(U40-C2-)
- U43 pad 1: Net-(U43-A_1) -> unconnected-(U43-Pad1)
- U43 pad 2: -12V_Analog -> unconnected-(U43-Pad2)
- U43 pad 3: Net-(U43-A_2) -> unconnected-(U43-Pad3)
- U43 pad 4: -12V_Analog -> unconnected-(U43-Pad4)
- U43 pad 5: -12V_Analog -> unconnected-(U43-Pad5)
- U43 pad 6: /ENTRADAS1/opto_out2 -> unconnected-(U43-Pad6)
- U43 pad 7: -12V_Analog -> (no net)
- U43 pad 8: /ENTRADAS1/opto_out1 -> unconnected-(U43-Pad8)
- U8 pad 2: Net-(U6-GPB5) -> Net-(U5-GPB3)
- U9 pad 2: Net-(U6-GPB3) -> Net-(U5-GPB4)
- U9 pad 5: +5V -> unconnected-(U9-VCC-Pad5)
Other:
- board text added: "TestPoint_THTPad_D4.0mm_Drill2.0mm"

Commit message: 08-06-26
Parts:
- J8: footprint CONECTORES GRACIDA:16POS-2LINEAS-3.5PITCH -> Connector_Card:microSD_HC_Hirose_DM3AT-SF-PEJM5
- J9: footprint CONECTORES GRACIDA:16POS-2LINEAS-3.5PITCH -> Connector_RJ:RJ45_Wuerth_7499010211A_Horizontal
- U21: footprint Package_SO:SSOP-16_5.3x6.2mm_P0.65mm -> Package_DFN_QFN:ArtInChip_QFN-100-1EP_12x12mm_P0.4mm_EP7.4x7.4mm_ThermalVias
- U30: footprint Package_SO:VSSOP-8_3x3mm_P0.65mm -> Package_TO_SOT_SMD:SOT-23-5_HandSoldering
- U31: footprint Package_TO_SOT_SMD:SOT-23 -> Package_TO_SOT_SMD:SOT-23-5_HandSoldering
- moved C38 253.6 mm to (238.0, 181.9), turned to -90 degrees
- moved C37 247.5 mm to (238.0, 172.4), turned to -90 degrees
- moved C36 244.5 mm to (226.9, 172.4), turned to -90 degrees
- moved R56 243.5 mm to (236.1, 172.5), turned to -90 degrees
- moved D13 229.4 mm to (303.6, 173.6)
- moved D14 229.4 mm to (303.6, 171.6)
- moved D15 229.4 mm to (303.7, 169.1)
- moved D16 229.4 mm to (303.7, 166.4)
- moved TH5 224.1 mm to (118.0, 132.1), turned to 90 degrees
- moved Q1 223.9 mm to (222.1, 172.2), turned to 90 degrees
- moved J9 223.2 mm to (159.1, 79.0)
- moved TH7 222.4 mm to (118.0, 114.1), turned to 90 degrees
- moved U9 216.2 mm to (233.1, 186.1), turned to -90 degrees
- moved C115 214.4 mm to (270.2, 121.6)
- moved C116 214.4 mm to (270.2, 124.1)
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