File: 01_IO-ASD-PLUS.kicad_pcb (KiCad board)
At the start: 2 copper layers, 180 x 158 mm, 600 parts, among them CN1 10way 1.27mm, IC1 VNI4140K, IC4 VNI4140K, IC5 ILD206T, IC6 ILD206T, IC7 ILD206T, J1 1147330000, J11 1728840000, J12 1728840000, J14 1728810000, J15 8P8C_LED_Shielded, J18 1728810000, J2 1147330000, J3 1147330000, J4 1604470000, J5 1728840000, J6 1728840000, J7 1728840000, J8 Micro_SD_Card_Det1, J9 RJ45_Wuerth_7499010211A, K1 G2RL-1-H, K2 G2RL-1-H, K3 G2RL-1-H, Q1 MMBT3904, Q10 DMP3099L, Q11 DMP3099L, Q12 DMP3099L, Q13 DMP3099L, Q2 MMBT3904, Q3 MMBT3904, Q4 MMBT3904, Q5 MMBT3904, Q6 MMBT3904, Q7 DMP3099L, Q8 DMP3099L, Q9 DMP3099L, U1 LTC3646EMSEPBF, U10 74LVC1G17, U11 74LVC1G17, U12 74LVC1G17, U13 TSB582, U14 ULN2003A, U15 LM7705, U16 MCP1799T-5002H/TT, U17 ILD206T, U18 ILD206T, U19 ILD206T, U2 LTC3646E, U20 24AA02E-OT, U21 FT900Q, U22 MCP9700Ax-ETT, U23 TPS2024, U24 ILD206T, U25 ILD206T, U26 ILD206T, U27 ILD206T, U28 ILD206T, U29 ILD206T, U3 KF33BDT, U30 TLV9301xDBV, U31 TLV9301xDBV, U32 LM7705, U33 MCP1799T-5002H/TT, U35 MCP23S17_SS, U37 LTC6820, U39 LTC6820, U40 MAX3232, U41 TLV2371DBV, U42 TLV702475_SOT23-5, U43 74LS30, U44 ILD206T, U45 ILD206T, U48 ILD206T, U49 ILD206T, U5 MCP23S17_SS, U50 ILD206T, U6 MCP23S17_SS, U7 74LVC1G17, U8 74LVC1G17, U9 74LVC1G17

Commit message: 22-jun-24
Parts:
- moved C39 256.8 mm to (248.9, 181.9), turned to -90 degrees
- moved R57 254.5 mm to (247.0, 182.0), turned to -90 degrees
- moved R59 241.6 mm to (247.1, 172.5), turned to -90 degrees
- moved U10 223.3 mm to (243.9, 186.1), turned to -90 degrees
- moved U12 215.2 mm to (244.1, 176.6), turned to -90 degrees
- moved C41 206.7 mm to (249.0, 172.4), turned to -90 degrees
- moved R51 206.0 mm to (250.9, 186.2), turned to 90 degrees
- moved R52 199.3 mm to (217.0, 130.1)
- moved R58 198.3 mm to (227.0, 131.6)
- moved R53 194.3 mm to (251.0, 176.7), turned to 90 degrees
- moved Q4 189.1 mm to (244.0, 181.7), turned to 90 degrees
- moved Q10 188.1 mm to (248.0, 185.9), turned to 90 degrees
- moved Q12 186.3 mm to (248.1, 176.4), turned to 90 degrees
- moved Q6 179.9 mm to (244.2, 172.2), turned to 90 degrees
- moved U11 176.8 mm to (216.4, 137.0)
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