File: 01_IO-ASD-PLUS.kicad_pcb (KiCad board)
At the start: 2 copper layers, 180 x 158 mm, 600 parts, among them CN1 10way 1.27mm, IC1 VNI4140K, IC4 VNI4140K, IC5 ILD206T, IC6 ILD206T, IC7 ILD206T, J1 1147330000, J11 1728840000, J12 1728840000, J14 1728810000, J15 8P8C_LED_Shielded, J18 1728810000, J2 1147330000, J3 1147330000, J4 1604470000, J5 1728840000, J6 1728840000, J7 1728840000, J8 Micro_SD_Card_Det1, J9 RJ45_Wuerth_7499010211A, K1 G2RL-1-H, K2 G2RL-1-H, K3 G2RL-1-H, Q1 MMBT3904, Q10 DMP3099L, Q11 DMP3099L, Q12 DMP3099L, Q13 DMP3099L, Q2 MMBT3904, Q3 MMBT3904, Q4 MMBT3904, Q5 MMBT3904, Q6 MMBT3904, Q7 DMP3099L, Q8 DMP3099L, Q9 DMP3099L, U1 LTC3646EMSEPBF, U10 74LVC1G17, U11 74LVC1G17, U12 74LVC1G17, U13 TSB582, U14 ULN2003A, U15 LM7705, U16 MCP1799T-5002H/TT, U17 ILD206T, U18 ILD206T, U19 ILD206T, U2 LTC3646E, U20 24AA02E-OT, U21 FT900Q, U22 MCP9700Ax-ETT, U23 TPS2024, U24 ILD206T, U25 ILD206T, U26 ILD206T, U27 ILD206T, U28 ILD206T, U29 ILD206T, U3 KF33BDT, U30 TLV9301xDBV, U31 TLV9301xDBV, U32 LM7705, U33 MCP1799T-5002H/TT, U35 MCP23S17_SS, U37 LTC6820, U39 LTC6820, U40 MAX3232, U41 TLV2371DBV, U42 TLV702475_SOT23-5, U43 74LS30, U44 ILD206T, U45 ILD206T, U48 ILD206T, U49 ILD206T, U5 MCP23S17_SS, U50 ILD206T, U6 MCP23S17_SS, U7 74LVC1G17, U8 74LVC1G17, U9 74LVC1G17

Commit message: 13-jul-26
Parts:
- removed U23: TPS2024, Package_SO:SOIC-8_3.9x4.9mm_P1.27mm
- removed U44, U45, U48, U49, U50: ILD206T, Package_SO:SOIC-8_3.9x4.9mm_P1.27mm
- added C42: 0.1uF, Capacitor_SMD:C_0603_1608Metric, F.Cu at (272.8, 184.6)
- added C44: 22uF, Capacitor_SMD:C_0603_1608Metric, F.Cu at (274.3, 164.1)
- added C46: 0.1uF, Capacitor_SMD:C_0603_1608Metric, F.Cu at (274.3, 167.6)
- added C54: 0.1uF, Capacitor_SMD:C_0603_1608Metric, F.Cu at (284.5, 162.3)
- added C55: 0.1uF, Capacitor_SMD:C_0603_1608Metric, F.Cu at (284.5, 169.3)
- added C64: 1uF, Capacitor_SMD:C_0603_1608Metric_Pad1.08x0.95mm_HandSolder, F.Cu at (279.0, 81.6)
- added R62: 100, Resistor_SMD:R_0603_1608Metric, F.Cu at (276.2, 184.6)
- added R86: 1k, Resistor_SMD:R_0603_1608Metric, F.Cu at (287.0, 165.1)
- C104, C106, C110, C111, C43, C45, C49, C50, C52: footprint Capacitor_SMD:C_0603_1608Metric_Pad1.08x0.95mm_HandSolder -> Capacitor_SMD:C_0603_1608Metric
- C130: value 0.1uF -> C_Small
- C40: footprint Capacitor_Tantalum_SMD:CP_EIA-1608-10_AVX-L_HandSolder -> Capacitor_SMD:C_0603_1608Metric_Pad1.08x0.95mm_HandSolder
- C65, C71, C72: footprint Capacitor_SMD:C_0603_1608Metric -> Capacitor_SMD:C_0603_1608Metric_Pad1.08x0.95mm_HandSolder
- D21: footprint LED_SMD:LED_0402_1005Metric -> LED_SMD:LED_0603_1608Metric
- D22: footprint LED_SMD:LED_0603_1608Metric_Pad1.05x0.95mm_HandSolder -> Diode_SMD:Nexperia_CFP3_SOD-123W
- D25, D27, D28, D30: footprint LED_SMD:LED_0603_1608Metric_Pad1.05x0.95mm_HandSolder -> Diode_SMD:D_MiniMELF
- D29: footprint LED_SMD:LED_0603_1608Metric_Pad1.05x0.95mm_HandSolder -> LED_SMD:LED_0402_1005Metric
- L2: footprint INDUCTORES GRACIDA:INDM4532X320N -> Inductores_GSI:SDR0906-3R9ML
- R109, R110, R111, R112, R150, R151, R152, R153, R154, R155, R183, R184, R185, R186, R187, R188, R189, R190, R191, R192, R193, R194, R195, R196, R197, R198, R199, R200, R201, R202, R203, R204, R205, R206, R207, R208, R209, R48, R63, R65: footprint Capacitor_SMD:C_0603_1608Metric_Pad1.08x0.95mm_HandSolder -> Resistor_SMD:R_0603_1608Metric
- R64: value 10k -> 1k
- R68: value 2.2k -> 100
- R70, R72: value 2.2k -> 10k
- R73: value 2.2k -> 0 ohms
- R75: value 1k -> 2.2k
- R76, R77, R78: value 1k -> 10k
- R79: value 1k -> 0 ohms
- R81, R83, R87, R91: footprint Resistor_SMD:R_0603_1608Metric -> Capacitor_SMD:C_0603_1608Metric_Pad1.08x0.95mm_HandSolder
- R85: value 10 -> 100
- U13: footprint Package_TO_SOT_SMD:SOT-23-5 -> Package_SO:SO-8_3.9x4.9mm_P1.27mm
- U18: footprint Package_SO:VSSOP-8_3x3mm_P0.65mm -> Package_SO:SOIC-8_3.9x4.9mm_P1.27mm
- U19, U24: footprint Package_TO_SOT_SMD:SOT-23 -> Package_SO:SOIC-8_3.9x4.9mm_P1.27mm
- U22: footprint Package_TO_SOT_SMD:SOT-23-5 -> Package_TO_SOT_SMD:SOT-23
- U28, U29: footprint Package_TO_SOT_SMD:SOT-23-5 -> Package_SO:SOIC-8_3.9x4.9mm_P1.27mm
- U33: footprint Package_SO:SSOP-28_5.3x10.2mm_P0.65mm -> Package_TO_SOT_SMD:SOT-23
- U39: footprint Package_TO_SOT_SMD:SOT-23-5 -> Package_SO:MSOP-16-1EP_3x4.039mm_P0.5mm_EP1.651x2.845mm_ThermalVias
- moved R111 299.7 mm to (366.7, 63.5)
- moved R112 299.7 mm to (366.7, 66.0)
- moved L10 294.9 mm to (352.0, 58.5)
- moved C86 282.1 mm to (351.0, 66.5)
- moved C84 282.1 mm to (348.5, 66.5)
- moved C85 282.1 mm to (358.5, 66.5)
- moved C87 282.1 mm to (353.5, 66.5)
- moved R60 278.8 mm to (279.5, 186.6), turned to 180 degrees
- moved R61 274.9 mm to (276.2, 186.6)
- moved R67 272.4 mm to (264.7, 192.6), turned to 180 degrees
- moved R28 266.7 mm to (269.3, 171.2), turned to 90 degrees
- moved R21 266.0 mm to (267.5, 171.2), turned to -90 degrees
- moved C31 263.6 mm to (252.8, 172.3), turned to -90 degrees
- moved C32 262.7 mm to (217.5, 191.7), turned to -90 degrees
- moved R22 262.0 mm to (264.0, 171.2), turned to -90 degrees
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Connections:
- C130 pad 1: Net-(U26-C1-) -> Net-(U13A-VCC-)
- C130 pad 2: Net-(U26-C1+) -> -12V_Analog
- C43 pad 1: Net-(U6-~{RESET}) -> Net-(U13A-VCC-)
- C52 pad 1: -12V_Analog -> Net-(U15-CF+)
- C52 pad 2: +24V -> Net-(U15-CF-)
- J5 pad 10: -12V_Analog -> Net-(J5-DA0)
- J5 pad 11: -12V_Analog -> Net-(J5-DA0)
- J5 pad 12: -12V_Analog -> Net-(J5-DA0)
- J5 pad 13: -12V_Analog -> Net-(J5-DA0)
- J5 pad 14: -12V_Analog -> unconnected-(J5-GND-Pad14)
- J5 pad 15: -12V_Analog -> Net-(U13A-OUT1)
- J5 pad 16: -12V_Analog -> unconnected-(J5-GND-Pad16)
- J5 pad 2: Net-(J5-DA1) -> unconnected-(J5-DA1-Pad2)
- J5 pad 3: Net-(J5-FUR) -> unconnected-(J5-FUR-Pad3)
- J5 pad 4: Net-(J5-FUL) -> unconnected-(J5-FUL-Pad4)
- J5 pad 5: Net-(J5-FREI) -> unconnected-(J5-FREI-Pad5)
- J5 pad 6: Net-(J5-MZ) -> -12V_Analog
- J5 pad 7: Net-(J5-ICM) -> unconnected-(J5-ICM-Pad7)
- J5 pad 8: Net-(J5-OUT2) -> unconnected-(J5-OUT2-Pad8)
- J5 pad 9: -12V_Analog -> Net-(J5-DA0)
- Q10 pad 3: Net-(J5-FREI) -> Net-(Q10-D)
- Q11 pad 3: Net-(J5-FUR) -> Net-(Q11-D)
- Q12 pad 3: Net-(J5-FUL) -> Net-(Q12-D)
- Q7 pad 3: Net-(J5-OUT2) -> Net-(Q7-D)
- Q8 pad 3: Net-(J5-MZ) -> Net-(Q8-D)
- Q9 pad 3: Net-(J5-ICM) -> Net-(Q9-D)
- R54 pad 2: Net-(J5-OUT2) -> Net-(Q7-D)
- R55 pad 1: Net-(J5-ICM) -> Net-(Q9-D)
- R56 pad 2: Net-(J5-MZ) -> Net-(Q8-D)
- R57 pad 2: Net-(J5-FREI) -> Net-(Q10-D)
- R58 pad 2: Net-(J5-FUR) -> Net-(Q11-D)
- R59 pad 2: Net-(J5-FUL) -> Net-(Q12-D)
- R60 pad 2: Net-(J5-DA1) -> Net-(R60-Pad2)
- R61 pad 2: Net-(J5-DA1) -> Net-(R60-Pad2)
- R64 pad 1: -12V_Analog -> Net-(R62-Pad2)
- R64 pad 2: Net-(D23-K) -> Net-(R64-Pad2)
- R66 pad 1: -12V_Analog -> Net-(R64-Pad2)
- R66 pad 2: Net-(D25-K) -> Net-(R66-Pad2)
- R68 pad 1: Net-(Q2-C) -> Net-(R68-Pad1)
- R68 pad 2: +24V -> Net-(U13A-OUT1)
- R69 pad 1: Net-(Q3-C) -> Net-(R69-Pad1)
- R69 pad 2: +24V -> Net-(U13B-IN2-)
- R70 pad 1: Net-(Q10-G) -> Net-(R69-Pad1)
- R70 pad 2: +24V -> Net-(R66-Pad2)
- R72 pad 1: Net-(Q12-G) -> Net-(R72-Pad1)
- R72 pad 2: +24V -> Net-(R69-Pad1)
- R73 pad 1: Net-(Q13-G) -> Net-(R72-Pad1)
- R73 pad 2: +24V -> -12V_Analog
- R74 pad 1: -12V_Analog -> Net-(R74-Pad1)
- R74 pad 2: Net-(J6-OUT2) -> Net-(R68-Pad1)
- R75 pad 1: Net-(J6-ICM) -> Net-(R75-Pad1)
- R75 pad 2: -12V_Analog -> Net-(U13A-IN1-)
- R76 pad 1: -12V_Analog -> Net-(R75-Pad1)
- R76 pad 2: Net-(J6-MZ) -> Net-(R76-Pad2)
- R77 pad 1: -12V_Analog -> Net-(R76-Pad2)
- R77 pad 2: Net-(J6-FREI) -> Net-(R74-Pad1)
- R78 pad 1: -12V_Analog -> Net-(R78-Pad1)
- R78 pad 2: Net-(J6-FUR) -> Net-(R75-Pad1)
- R79 pad 1: -12V_Analog -> Net-(R78-Pad1)
- R79 pad 2: Net-(J6-FUL) -> -12V_Analog
- R85 pad 1: Net-(U14A-OUT1) -> -12V_Analog
- R85 pad 2: Net-(J6-DA0) -> Net-(U15-SD)
- U9 pad 5: unconnected-(U9-VCC-Pad5) -> +5V

Commit message: 13-jul-26_6pm
Parts:
- added J13: 1728810000, CONECTORES GRACIDA:1728810000, F.Cu at (348.9, 127.5)
- added L13: L_Iron_Small, Inductor_SMD:L_0603_1608Metric_Pad1.05x0.95mm_HandSolder, F.Cu at (122.9, 140.6)
- added L14: L_Iron_Small, Inductor_SMD:L_0603_1608Metric_Pad1.05x0.95mm_HandSolder, F.Cu at (122.0, 172.7)
- added L16: L_Iron_Small, Inductor_SMD:L_0603_1608Metric_Pad1.05x0.95mm_HandSolder, F.Cu at (122.3, 124.3)
- added U34: MCP23S17_SS, Package_SO:SSOP-28_5.3x10.2mm_P0.65mm, F.Cu at (350.1, 146.4)
- added U36: LTC6820, Package_SO:MSOP-16-1EP_3x4.039mm_P0.5mm_EP1.651x2.845mm_ThermalVias, F.Cu at (348.9, 135.7)
- added U38: TLV2371DBV, Package_TO_SOT_SMD:SOT-23-5, F.Cu at (359.9, 142.9)
- J14: value 1728810000 -> 8P8C_LED_Shielded
- R68: value 100 -> 2.2k
- R69: value 2.2k -> 10k
- R70: value 10k -> 100
- R73: value 0 ohms -> 1k
- R74: value 1k -> 0 ohms
- R79: value 0 ohms -> 10k
- R80: value 10k -> 0 ohms
- U35: value MCP23S17_SS -> MAX3232
- U37: value LTC6820 -> MAX3232
- U39: value LTC6820 -> TLV702475_SOT23-5
- U40: value MAX3232 -> 74LS30
- moved C97 237.6 mm to (122.8, 166.6)
- moved C108 202.8 mm to (125.8, 124.3), turned to 90 degrees
- moved R166 172.3 mm to (147.3, 109.5), turned to 90 degrees
- moved R160 163.9 mm to (156.0, 103.8), turned to 180 degrees
- moved C95 159.4 mm to (122.0, 143.1), turned to 90 degrees
- moved R150 154.7 mm to (171.5, 103.3)
- moved R159 152.6 mm to (182.2, 108.1)
- moved R163 145.1 mm to (183.3, 103.1)
- moved R151 139.7 mm to (175.2, 102.1)
- moved R152 139.7 mm to (175.2, 104.6)
- moved R153 139.7 mm to (175.2, 107.1)
- moved R156 138.7 mm to (179.3, 101.1)
- moved R155 132.6 mm to (182.1, 105.6)
- moved R161 132.1 mm to (168.5, 103.6), turned to 90 degrees
- moved C101 131.2 mm to (184.8, 100.6)
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Connections:
- C115 pad 1: Net-(U35-~{RESET}) -> Net-(U34-~{RESET})
- C117 pad 1: Net-(U38-C1+) -> Net-(U35-C1+)
- C117 pad 2: Net-(U38-C1-) -> Net-(U35-C1-)
- C121 pad 2: Net-(U38-VS+) -> Net-(U35-VS+)
- C122 pad 2: Net-(U38-VS-) -> Net-(U35-VS-)
- C123 pad 1: Net-(U38-C2+) -> Net-(U35-C2+)
- C123 pad 2: Net-(U38-C2-) -> Net-(U35-C2-)
- C125 pad 1: Net-(U40-VS+) -> Net-(U37-VS+)
- C126 pad 1: Net-(U40-VS-) -> Net-(U37-VS-)
- C127 pad 1: Net-(U40-C2+) -> Net-(U37-C2+)
- C127 pad 2: Net-(U40-C2-) -> Net-(U37-C2-)
- C129 pad 1: Net-(U40-C1+) -> Net-(U37-C1+)
- C129 pad 2: Net-(U40-C1-) -> Net-(U37-C1-)
- J14 pad 1: Net-(J14-X0) -> Net-(T1-SA)
- J14 pad 10: Net-(J14-X9) -> /Serial_Comm/Led_ctrl/LED1_A
- J14 pad 2: -12V_Analog -> Net-(T1-SB)
- J14 pad 3: Net-(J14-X1) -> Net-(U37-T2OUT)
- J14 pad 4: Net-(J14-X6) -> unconnected-(J14-Pad4)
- J14 pad 5: Net-(J14-X2) -> unconnected-(J14-Pad5)
- J14 pad 6: Net-(J14-X7) -> /Serial_Comm/Led_ctrl/INT
- J14 pad 7: Net-(J14-X3) -> +24V
- J14 pad 8: Net-(J14-X8) -> -12V_Analog
- J14 pad 9: -12V_Analog -> /Serial_Comm/Led_ctrl/LED1_C
- L17 pad 1: Net-(U39-IM) -> Net-(U36-IM)
- L17 pad 4: Net-(U39-IP) -> Net-(U36-IP)
- R178 pad 1: Net-(U35-~{RESET}) -> Net-(U34-~{RESET})
- R179 pad 2: Net-(U35-A1) -> Net-(U34-A1)
- R180 pad 2: Net-(U35-A0) -> Net-(U34-A0)
- R181 pad 1: Net-(U35-A0) -> Net-(U34-A0)
- R184 pad 1: Net-(U39-PHA) -> Net-(U36-PHA)
- R185 pad 1: Net-(U39-POL) -> Net-(U36-POL)
- R186 pad 1: Net-(U39-PHA) -> Net-(U36-PHA)
- R187 pad 1: Net-(U39-POL) -> Net-(U36-POL)
- R188 pad 2: Net-(U39-SLOW) -> Net-(U36-SLOW)
- R189 pad 1: Net-(U39-MSTR) -> Net-(U36-MSTR)
- R190 pad 1: Net-(U39-SLOW) -> Net-(U36-SLOW)
- R192 pad 1: Net-(U40-T2OUT) -> Net-(U37-T2OUT)
- R192 pad 2: Net-(J14-X8) -> Net-(J13-X8)
- R193 pad 2: Net-(J14-X9) -> Net-(J13-X9)
- R198 pad 1: Net-(U41--) -> Net-(U38--)
- R200 pad 1: Net-(U41-+) -> Net-(U38-+)
- R201 pad 1: Net-(U41--) -> Net-(U38--)
- R203 pad 2: Net-(U41--) -> Net-(U38--)
- R204 pad 2: Net-(U41--) -> Net-(U38--)
- R207 pad 2: Net-(U41-+) -> Net-(U38-+)
- R208 pad 2: Net-(U41-+) -> Net-(U38-+)
- R55 pad 1: Net-(Q9-D) -> -12V_Analog
- R55 pad 2: -12V_Analog -> Net-(Q8-D)
- R56 pad 1: -12V_Analog -> Net-(Q9-D)
- R56 pad 2: Net-(Q8-D) -> -12V_Analog
- R68 pad 2: Net-(U13A-OUT1) -> Net-(U13B-IN2-)
- R69 pad 1: Net-(R69-Pad1) -> Net-(R68-Pad1)
- R69 pad 2: Net-(U13B-IN2-) -> Net-(R66-Pad2)
- R70 pad 1: Net-(R69-Pad1) -> Net-(R70-Pad1)
- R70 pad 2: Net-(R66-Pad2) -> Net-(U13A-OUT1)
- R72 pad 2: Net-(R69-Pad1) -> Net-(R68-Pad1)
- R73 pad 1: Net-(R72-Pad1) -> Net-(R73-Pad1)
- R73 pad 2: -12V_Analog -> Net-(R70-Pad1)
- R74 pad 1: Net-(R74-Pad1) -> Net-(R72-Pad1)
- R74 pad 2: Net-(R68-Pad1) -> -12V_Analog
- R77 pad 2: Net-(R74-Pad1) -> Net-(R73-Pad1)
- R79 pad 1: Net-(R78-Pad1) -> Net-(U13A-IN1+)
- R79 pad 2: -12V_Analog -> /Processador/DAC1
- R80 pad 1: Net-(U13A-IN1+) -> Net-(R78-Pad1)
- R80 pad 2: /Processador/DAC1 -> -12V_Analog
- U35 pad 1: /ENTRADAS2/opto_out2 -> Net-(U35-C1+)
- U35 pad 10: -12V_Analog -> /Processador/UART0_TXD
- U35 pad 11: /Port Expansor/!CS_SPI -> /Processador/UART1_TXD
- U35 pad 12: /Port Expansor/SCK_SPI -> /Processador/UART1_RXD
- U35 pad 13: /Port Expansor/MOSI_SPI -> Net-(J13-X2)
- U35 pad 14: /Port Expansor/MISO_SPI -> Net-(J13-X0)
- U35 pad 15: Net-(U35-A0) -> -12V_Analog
- U35 pad 16: Net-(U35-A1) -> +3.3v_Fuse_comm
- U35 pad 17: -12V_Analog -> (no net)
- U35 pad 18: Net-(U35-~{RESET}) -> (no net)
- U35 pad 19: /Port Expansor/INTB -> (no net)
- U35 pad 2: /ENTRADAS2/opto_out4 -> Net-(U35-VS+)
- U35 pad 20: /Port Expansor/INTA -> (no net)
- U35 pad 21: /ENTRADAS1/opto_out5 -> (no net)
- U35 pad 22: /ENTRADAS1/opto_out6 -> (no net)
- U35 pad 23: /ENTRADAS/opto_out1 -> (no net)
- U35 pad 24: /ENTRADAS/opto_out3 -> (no net)
- U35 pad 25: /ENTRADAS/opto_out2 -> (no net)
- U35 pad 26: /ENTRADAS/opto_out4 -> (no net)
- U35 pad 27: /ENTRADAS/opto_out5 -> (no net)
- U35 pad 28: /ENTRADAS/opto_out6 -> (no net)
- U35 pad 3: /ENTRADAS2/opto_out5 -> Net-(U35-C1-)
- U35 pad 4: /ENTRADAS2/opto_out6 -> Net-(U35-C2+)
- U35 pad 5: /ENTRADAS1/opto_out1 -> Net-(U35-C2-)
- U35 pad 6: /ENTRADAS1/opto_out3 -> Net-(U35-VS-)
- U35 pad 7: /ENTRADAS1/opto_out2 -> Net-(J13-X1)
- U35 pad 8: /ENTRADAS1/opto_out4 -> Net-(J13-X3)
- U35 pad 9: +3.3v -> /Processador/UART0_RXD
- U37 pad 1: +3.3v_Fuse3 -> Net-(U37-C1+)
- U37 pad 10: Net-(U37-IM) -> /Processador/INT_FT812
- U37 pad 11: Net-(U37-IP) -> /Processador/BUSY_DISPLAY
- U37 pad 12: Net-(U37-MSTR) -> /Processador/INT_FT812
- U37 pad 13: Net-(U37-SLOW) -> /Serial_Comm/Led_ctrl/INT
- U37 pad 14: -12V_Analog -> Net-(J13-X7)
- U37 pad 15: /Serial_Comm/600mA -> -12V_Analog
- U37 pad 16: /Serial_Comm/+2.0v -> +3.3v_Fuse_comm
- U37 pad 2: /Port Expansor/MOSI_SPI -> Net-(U37-VS+)
- U37 pad 3: /Port Expansor/MISO_SPI -> Net-(U37-C1-)
- U37 pad 4: /Port Expansor/SCK_SPI -> Net-(U37-C2+)
- U37 pad 5: /Processador/SPIM_SS -> Net-(U37-C2-)
- U37 pad 6: +3.3v_Fuse3 -> Net-(U37-VS-)
- U37 pad 7: Net-(U37-POL) -> Net-(U37-T2OUT)
- U37 pad 8: Net-(U37-PHA) -> Net-(J13-X6)
- U37 pad 9: +3.3v_Fuse3 -> /Processador/METAL_INTERRUPCION
- U39 pad 1: +3.3v_Fuse3 -> unconnected-(U39-IN-Pad1)
- U39 pad 10: Net-(U39-IM) -> (no net)
- U39 pad 11: Net-(U39-IP) -> (no net)
- U39 pad 12: Net-(U39-MSTR) -> (no net)
- U39 pad 13: Net-(U39-SLOW) -> (no net)
- U39 pad 14: -12V_Analog -> (no net)
- U39 pad 15: /Serial_Comm/600mA -> (no net)
- U39 pad 16: /Serial_Comm/+2.0v -> (no net)
- U39 pad 2: /Port Expansor/MOSI_SPI -> unconnected-(U39-GND-Pad2)
- U39 pad 3: /Port Expansor/MISO_SPI -> unconnected-(U39-EN-Pad3)
- U39 pad 4: /Port Expansor/SCK_SPI -> unconnected-(U39-NC-Pad4)
- U39 pad 5: /Processador/SPIM_SS -> unconnected-(U39-OUT-Pad5)
- U39 pad 6: +3.3v_Fuse3 -> (no net)
- U39 pad 7: Net-(U39-POL) -> (no net)
- U39 pad 8: Net-(U39-PHA) -> (no net)
- U39 pad 9: +3.3v_Fuse3 -> (no net)
- U40 pad 1: Net-(U40-C1+) -> unconnected-(U40-Pad1)
- U40 pad 2: Net-(U40-VS+) -> unconnected-(U40-Pad2)
- U40 pad 3: Net-(U40-C1-) -> unconnected-(U40-Pad3)
- U40 pad 4: Net-(U40-C2+) -> unconnected-(U40-Pad4)
- U40 pad 5: Net-(U40-C2-) -> unconnected-(U40-Pad5)

Commit message: 14-JUL-26
Parts:
- added C99: 0.1uF, Capacitor_SMD:C_0603_1608Metric_Pad1.08x0.95mm_HandSolder, F.Cu at (156.5, 100.8)
- C130: value C_Small -> 0.1uF
- R64, R66: footprint Capacitor_SMD:C_0603_1608Metric_Pad1.08x0.95mm_HandSolder -> Resistor_SMD:R_0603_1608Metric
- U39: footprint Package_SO:MSOP-16-1EP_3x4.039mm_P0.5mm_EP1.651x2.845mm_ThermalVias -> Package_TO_SOT_SMD:SOT-23-5
- moved R167 154.2 mm to (164.3, 103.3)
- moved R172 151.8 mm to (164.3, 105.1), turned to 180 degrees
- moved R171 151.1 mm to (164.3, 101.6), turned to 180 degrees
- moved R173 146.3 mm to (164.3, 99.8)
- moved D28 107.3 mm to (168.5, 100.6), turned to 180 degrees
- moved R157 38.9 mm to (204.4, 106.3)
- moved U31 25.1 mm to (168.5, 103.8), turned to 180 degrees
- moved R156 20.1 mm to (159.3, 102.6)
- moved R151 19.6 mm to (156.0, 106.1)
- moved R152 19.5 mm to (156.0, 107.8)
- moved R153 15.9 mm to (159.3, 107.8), turned to 180 degrees
- moved D25 14.5 mm to (151.8, 107.1), turned to 180 degrees
- moved R150 12.6 mm to (159.3, 106.1), turned to 180 degrees
- moved R161 9.28 mm to (159.3, 104.3), turned to 0 degrees
- moved C101 7.50 mm to (177.3, 100.8)
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Connections:
- C130 pad 1: Net-(U13A-VCC-) -> -12V_Analog
- C130 pad 2: -12V_Analog -> +12V
