File: 01_IO-ASD-PLUS.kicad_pcb (KiCad board)
At the start: 2 copper layers, 180 x 158 mm, 610 parts, among them CN1 10way 1.27mm, IC1 VNI4140K, IC4 VNI4140K, IC5 ILD206T, IC6 ILD206T, IC7 ILD206T, J1 1147330000, J11 1728840000, J12 1728840000, J13 1728810000, J14 8P8C_LED_Shielded, J15 8P8C_LED_Shielded, J18 1728810000, J2 1147330000, J3 1147330000, J4 1604470000, J5 1728840000, J6 1728840000, J7 1728840000, J8 Micro_SD_Card_Det1, J9 RJ45_Wuerth_7499010211A, K1 G2RL-1-H, K2 G2RL-1-H, K3 G2RL-1-H, Q1 MMBT3904, Q10 DMP3099L, Q11 DMP3099L, Q12 DMP3099L, Q13 DMP3099L, Q2 MMBT3904, Q3 MMBT3904, Q4 MMBT3904, Q5 MMBT3904, Q6 MMBT3904, Q7 DMP3099L, Q8 DMP3099L, Q9 DMP3099L, U1 LTC3646EMSEPBF, U10 74LVC1G17, U11 74LVC1G17, U12 74LVC1G17, U13 TSB582, U14 ULN2003A, U15 LM7705, U16 MCP1799T-5002H/TT, U17 ILD206T, U18 ILD206T, U19 ILD206T, U2 LTC3646E, U20 24AA02E-OT, U21 FT900Q, U22 MCP9700Ax-ETT, U24 ILD206T, U25 ILD206T, U26 ILD206T, U27 ILD206T, U28 ILD206T, U29 ILD206T, U3 KF33BDT, U30 TLV9301xDBV, U31 TLV9301xDBV, U32 LM7705, U33 MCP1799T-5002H/TT, U34 MCP23S17_SS, U35 MAX3232, U36 LTC6820, U37 MAX3232, U38 TLV2371DBV, U39 TLV702475_SOT23-5, U40 74LS30, U41 TLV2371DBV, U42 TLV702475_SOT23-5, U43 74LS30, U5 MCP23S17_SS, U6 MCP23S17_SS, U7 74LVC1G17, U8 74LVC1G17, U9 74LVC1G17

Commit message: 17-07-26
Parts:
- C109: value 1uF -> 0.1uF
- C112: value 0.1uF -> 0.1uf
- D29: footprint LED_SMD:LED_0402_1005Metric -> LED_SMD:LED_0603_1608Metric_Pad1.05x0.95mm_HandSolder
- R176: value 10k -> 100
- R177: value 470 -> 1k
- moved R37 188.6 mm to (23.3, 220.1)
- moved R38 188.6 mm to (27.5, 220.6)
- moved R39 188.6 mm to (27.8, 223.8)
- moved R40 188.6 mm to (19.9, 221.8)
- moved R47 188.6 mm to (23.8, 222.6)
- moved U6 188.6 mm to (23.3, 230.6)
- moved R174 149.3 mm to (164.3, 106.6)
- moved C111 143.7 mm to (185.0, 101.1)
- moved C114 142.3 mm to (190.0, 105.7)
- moved R154 138.6 mm to (176.1, 106.1), turned to 180 degrees
- moved C106 133.6 mm to (190.0, 100.9)
- moved C112 133.1 mm to (185.0, 99.4)
- moved C104 132.4 mm to (190.0, 102.5)
- moved C103 131.3 mm to (190.0, 104.1)
- moved R170 128.8 mm to (176.1, 104.3)
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Connections:
- C105 pad 1: Net-(BT1-+) -> Net-(U32-CRES)
- C109 pad 1: +1.2Vreg -> Net-(D29-A)
- C112 pad 1: +3.3v_Fuse -> Net-(U32-CF+)
- C112 pad 2: -12V_Analog -> Net-(U32-CF-)
- C113 pad 1: +3.3v_Fuse -> Net-(D29-A)
- C114 pad 1: +3.3V -> +12V
- R176 pad 1: /USB/USB_Current_Status -> Net-(U32-SD)
- R176 pad 2: +3.3V -> -12V_Analog
- R177 pad 1: Net-(D33-K) -> -12V_Analog
- R177 pad 2: -12V_Analog -> Net-(D29-K)

Commit message: 21-JUL-26
Parts:
- removed IC4: VNI4140K, Package_SO:ST_PowerSSO-24_SlugDown_ThermalVias
- removed IC5, IC6, IC7: ILD206T, SOIC:SOIC 8
- removed PS2: MGFW402412, Fuentes_GSI:MGFW400512
- removed Q13: DMP3099L, Package_TO_SOT_SMD:SOT-23
- added C68: 10uF, Capacitor_SMD:C_0603_1608Metric_Pad1.08x0.95mm_HandSolder, F.Cu at (311.8, 60.3)
- added J10: USB_Type A_ Receptacle, Connector_USB:USB_A_Molex_105057_Vertical, F.Cu at (286.4, 102.3)
- added L11: L_Iron_Small, Inductor_SMD:L_0603_1608Metric_Pad1.05x0.95mm_HandSolder, F.Cu at (171.8, 63.1)
- added P1: USB_C_Plug_USB2.0, CONECTORES GRACIDA:USB4145030070C, F.Cu at (178.3, 69.9)
- added U23: TPS2024, Package_SO:SOIC-8_3.9x4.9mm_P1.27mm, F.Cu at (279.8, 105.1)
- moved C89 224.4 mm to (281.4, 109.7)
- moved C93 221.9 mm to (275.8, 104.5), turned to 90 degrees
- moved D24 214.0 mm to (277.8, 111.5)
- moved C88 200.4 mm to (281.6, 100.5), turned to 180 degrees
- moved R121 198.0 mm to (281.4, 111.3)
- moved R119 197.8 mm to (277.8, 109.7), turned to 180 degrees
- moved R118 193.5 mm to (278.2, 100.5), turned to 180 degrees
- moved R124 185.0 mm to (281.7, 98.9), turned to 180 degrees
- moved R131 153.3 mm to (182.8, 134.8), turned to -90 degrees
- moved R135 148.8 mm to (190.2, 138.3), turned to 90 degrees
- moved U26 146.9 mm to (186.6, 136.5), turned to 90 degrees
- moved R130 145.5 mm to (182.8, 138.3), turned to -90 degrees
- moved U25 143.5 mm to (186.6, 127.5), turned to 90 degrees
- moved R128 141.8 mm to (182.8, 129.3), turned to -90 degrees
- moved R133 141.6 mm to (190.2, 125.7), turned to 90 degrees
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Connections:
- C58 pad 1: Net-(CN1-10) -> Net-(U21-RESETN)
- CN1 pad 1: (no net) -> Net-(U21-SPIS0_CLK/GPIO36)
- CN1 pad 10: (no net) -> Net-(U21-RESETN)
- CN1 pad 2: (no net) -> Net-(U21-SPIS0_SS/GPIO37)
- CN1 pad 3: (no net) -> Net-(U21-SPIS0_MOSI/GPIO38)
- CN1 pad 4: (no net) -> Net-(U21-SPIS0_MISO/GPIO39)
- CN1 pad 5: (no net) -> unconnected-(CN1-Pad5)
- CN1 pad 6: (no net) -> unconnected-(CN1-Pad6)
- CN1 pad 7: (no net) -> -12V_Analog
- CN1 pad 8: (no net) -> Net-(U21-DEBUG)
- CN1 pad 9: (no net) -> DBG_5V
- R99 pad 1: Net-(CN1-10) -> Net-(U21-RESETN)
- U21 pad 20: Net-(CN1-1) -> Net-(U21-SPIS0_CLK/GPIO36)
- U21 pad 21: Net-(CN1-2) -> Net-(U21-SPIS0_SS/GPIO37)
- U21 pad 22: Net-(CN1-3) -> Net-(U21-SPIS0_MOSI/GPIO38)
- U21 pad 23: Net-(CN1-4) -> Net-(U21-SPIS0_MISO/GPIO39)
- U21 pad 34: Net-(CN1-10) -> Net-(U21-RESETN)
- U21 pad 36: Net-(CN1-8) -> Net-(U21-DEBUG)

Commit message: 24/07/2026
Parts:
- removed C130, C131, C132, C133, C134, C135, C136, C137, C138, C139, C140, C141, C142, C143, C152, C153, C160, C161, C162, C163, C164, C165, C166, C167, C168, C169, C170, C171, C172, C173, C174: 0.1uF, Capacitor_SMD:C_0603_1608Metric_Pad1.08x0.95mm_HandSolder
- removed C149: 470nF, Capacitor_SMD:C_0603_1608Metric
- removed C151, C156: 4.7uF, Capacitor_SMD:C_0603_1608Metric
- removed C155: 10uF, Capacitor_SMD:C_0603_1608Metric
- removed D32: PMEG2010BER, Diode_SMD:Nexperia_CFP3_SOD-123W
- removed D33, D34: LED, LED_SMD:LED_0603_1608Metric_Pad1.05x0.95mm_HandSolder
- removed D35, D36: BZV55B3V3, Diode_SMD:D_MiniMELF
- removed D37, D38: BZV55B11, Diode_SMD:D_MiniMELF
- removed D39: LED, LED_SMD:LED_0402_1005Metric
- removed D40: BZV55C15, Diode_SMD:D_MiniMELF
- removed J15: 8P8C_LED_Shielded, CONECTORES GRACIDA:1728810000
- removed L18, L20: 10uH, Inductor_SMD:L_0603_1608Metric_Pad1.05x0.95mm_HandSolder
- removed L21: 0603, Inductor_SMD:L_0603_1608Metric_Pad1.05x0.95mm_HandSolder
- removed L23: 200uH, Inductores_GSI:DLW43_MUR
- removed L25: SDR0906-3R9ML, Inductores_GSI:SDR0906-3R9ML
- removed R210, R211, R212: 2.2k, Capacitor_SMD:C_0603_1608Metric_Pad1.08x0.95mm_HandSolder
- removed R213, R214, R215, R216: 10k, Capacitor_SMD:C_0603_1608Metric_Pad1.08x0.95mm_HandSolder
- removed R217, R218, R219, R220, R221, R222, R37, R38, R39, R40, R47: 4.7k, Capacitor_SMD:C_0603_1608Metric_Pad1.08x0.95mm_HandSolder
- removed R223, R227, R251: 10k, Resistor_SMD:R_0603_1608Metric
- removed R224, R225, R226, R228, R229, R230, R231, R232, R233, R234, R235, R236, R237, R238, R239, R240, R241, R242, R243, R244, R245, R246, R247, R248: 10, Resistor_SMD:R_0603_1608Metric
- removed R252, R253, R254, R257, R258, R259, R260, R261, R262, R263, R265, R266, R267, R271, R272: 0R, Resistor_SMD:R_0603_1608Metric
- removed R255: 620, Resistor_SMD:R_0603_1608Metric
- removed R256: 1.5K, Resistor_SMD:R_0603_1608Metric
- removed R264: 120 1%, Resistor_SMD:R_0603_1608Metric
- removed R268, R269: 4.7k, Resistor_SMD:R_0603_1608Metric
- removed R270: 100, Resistor_SMD:R_0603_1608Metric
- removed R273, R274, R275, R276, R277, R278, R279, R280, R281, R282: 100K, Resistor_SMD:R_0603_1608Metric
- removed U41: TLV2371DBV, Package_TO_SOT_SMD:SOT-23-5
- removed U42: TLV702475_SOT23-5, Package_TO_SOT_SMD:SOT-23-5
- removed U43: 74LS30, Package_SO:SOIC-8_3.9x4.9mm_P1.27mm
- removed U6: MCP23S17_SS, Package_SO:SSOP-28_5.3x10.2mm_P0.65mm
- added PS2: MGFW402412, Fuentes_GSI:MGFW400512, F.Cu at (60.2, 67.6)
- added T1: Transformer_1P_1S, TRANSFORMADORES GRACIDA:TRANFORMADOR_1001C, F.Cu at (242.1, 165.2)
- J14: footprint CONECTORES GRACIDA:1728810000 -> CONECTORES GRACIDA:WE-RJ45LAN
- moved R181 298.2 mm to (20.9, 183.1)
- moved R190 284.4 mm to (25.0, 178.3)
- moved R185 282.5 mm to (27.8, 192.4)
- moved R184 280.1 mm to (27.5, 185.3)
- moved R31 224.9 mm to (21.3, 190.9)
- moved R30 224.9 mm to (21.3, 188.4)
- moved J13 223.9 mm to (125.2, 117.6)
- moved U40 207.5 mm to (349.3, 196.4)
- moved C122 204.8 mm to (205.1, 176.4), turned to 90 degrees
- moved L17 201.0 mm to (231.6, 162.1), turned to 180 degrees
- moved C94 196.1 mm to (283.2, 96.7)
- moved C124 190.5 mm to (222.6, 158.2)
- moved C126 160.9 mm to (184.0, 159.6), turned to 180 degrees
- moved R192 159.3 mm to (184.1, 161.2), turned to 180 degrees
- moved C78 159.1 mm to (202.9, 102.0)
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Connections:
- J5 pad 7: unconnected-(J5-ICM-Pad7) -> Net-(J5-ICM)
- J5 pad 8: unconnected-(J5-OUT2-Pad8) -> Net-(J5-ICM)
- L17 pad 1: Net-(U36-IM) -> Net-(T1-AB)
- L17 pad 2: Net-(T1-AA) -> Net-(U36-IM)
- L17 pad 3: Net-(T1-AB) -> Net-(U36-IP)
- L17 pad 4: Net-(U36-IP) -> Net-(T1-AA)
- R185 pad 1: Net-(U36-POL) -> unconnected-(R185-Pad1)
- R70 pad 2: Net-(U13A-OUT1) -> Net-(J5-ICM)
