File: Procesador.kicad_sch (KiCad schematic)
At the start: 62 parts, among them CN7 10way 1.27mm, J11 Micro_SD_Card_Det1, J15 RJ45_Wuerth_7499010211A, SW1 Reset, U1 FT900L-C-T, U31 MCP9700Ax-ETT, U6 24AA02E-OT, Y1 Crystal, Y2 Crystal

Commit message: 22 mayo 26 actualizacion
se actualizo la PCB para la rama laptop Antigua
Parts:
- removed U1: FT900L-C-T, footprints:LQFP_100_14X14X1P4_BRI, symbol MICROS_DIGITAL_GSI:FT900L-C-T
- added U1: FT900Q, footprints:LQFP_100_14X14X1P4_BRI, symbol MICROS_DIGITAL_GSI_v2:FT900Q
- renumbered C86 to C100, C103 to C101, C106 to C102, C94 to C103, C95 to C104, C102 to C105, C96 to C106, C97 to C107, C119 to C108, C98 to C109, C99 to C110, C118 to C111, C100 to C112, C101 to C113, C117 to C114, C104 to C115, C105 to C116, C107 to C117, C108 to C118, C83 to C89, C84 to C90, C85 to C91, C87 to C92, C88 to C93, C89 to C94, C90 to C95, C91 to C96, C116 to C97, C92 to C98, C93 to C99, CN7 to CN1, J11 to J10, J15 to J11, L15 to L13, R141 to R156, R142 to R157, R143 to R158, R160 to R159, R161 to R160, R146 to R161, R144 to R162, R145 to R163, R151 to R164, R148 to R165, R163 to R166, R162 to R167, R147 to R168, R149 to R169, R150 to R170, R164 to R171, R165 to R172, R166 to R173, R167 to R174, U6 to U22, U31 to U24
Connections:
- net !CS_Exp: now also U1.17 (SPIM_SS1/GPIO33)
- net !CS_J5_J6: now also U1.18 (SPIM_SS2/GPIO34)
- net +1.2Vreg: now also U1.32 (FSOURCE), U1.63 (VOUT1), U1.67 (VCC1V2), U1.77 (VOUT2); no longer C106.1
- net +3.3v_Fuse: now also C106.1, U1.33 (VPP), U1.46 (VCCIO3V3), U1.64 (VCCIO3V3), U1.68 (VUSB3V3), U1.76 (VETH3V3), U1.79 (VETH3V3), U1.95 (VCC3V3A)
- net ADC2: now also U1.88 (ADC2/CAM_PCLK/GPIO7)
- net ADC3: now also U1.89 (ADC3/CAM_VD/GPIO8)
- net BUSY_DISPLAY: now also U1.44 (UART0_RI/UART1_CTS/PWM7/GPIO55)
- net D+_H_P: now also U1.73 (H_DP)
- net D-_H_N: now also U1.72 (H_DM)
- net DAC0: now also U1.98 (DAC0/CAM_D3/GPIO14)
- net DAC1: now also U1.97 (DAC1/CAM_D4/GPIO13)
- net GND: now also U1.45 (GND)
- net INTA_J5_J6: now also U1.48 (PWM1/GPIO57)
- net INT_FT812: now also U1.40 (UART0_CTS/GPIO51)
- net METAL_INTERRUPCION: now also U1.43 (UART0_DCD/UART1_RTS/PWM6/GPIO54)
- net MO1: now also U1.47 (PWM0/GPIO56)
- net MO2: now also U1.1 (CAN1_TXD/CAM_D0/GPIO17)
- net MO3: now also U1.2 (CAN1_RXD/GPIO18)
- net MO4: now also U1.93 (ADC7/CAM_D5/GPIO12)
- net Metal1: now also U1.99 (CAN0_TXD/CAM_D2/GPIO15)
- net Metal2: now also U1.100 (CAN0_RXD/CAM_D1/GPIO16)
- net PD_N: now also U1.49 (PWM2/GPIO58)
- net SPIM_MISO: now also U1.14 (SPIM_MISO/GPIO30)
- net SPIM_MOSI: now also U1.13 (SPIM_MOSI/GPIO29)
- net SPIM_SCLK: now also U1.11 (SPIM_CLK/GPIO27)
- net SPIM_SS: now also U1.19 (SPIM_SS3/GPIO35)
- net UART0_RXD: now also U1.38 (UART0_RXD/GPIO49)
- net UART0_TXD: now also U1.37 (UART0_TXD/GPIO48)
- net UART1_RXD: now also U1.42 (UART0_DSR/UART1_RXD/PWM5/GPIO53)
- net UART1_TXD: now also U1.41 (UART0_DTR/UART1_TXD/PWM4/GPIO52)
- net USB_Current_Status: now also U1.58 (OC_N/GPIO1)
- net USB_D+_Device: now also U1.70 (D_DP)
- net USB_D-_Device: now also U1.69 (D_DM)
- net USB_Power_Switcher: now also U1.59 (PSW_N/GPIO2)
- net at C89.1, CN1. (9), R156.1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: now also U1.34 (RESETN)
- net at J11.1 (TD+), R174.2: now also U1.82 (TXOP)
- net at C118.1, Y2.2: now also U1.65 (XI/CLKIN)
- net at BT1.1 (+), C105.1: now also U1.86 (VDDBAT)
- net at C117.2, Y2.1: now also U1.66 (XIO)
- net at R170.1: now also U1.78 (EREFSET)
- net at R159.1, U22.1 (SCL): now also U1.30 (I2C1_SCL/GPIO46)
- net at J10.9 (DET), R157.2: now also U1.9 (SD_CD/GPIO25)
- net at R160.1, U22.3 (SDA): now also U1.31 (I2C1_SDA/GPIO47)
- net at J11.10: now also U1.62 (ENET_LED1/GPIO5)
- net at J11.11: now also U1.61 (ENET_LED0/GPIO4)
- net at J11.2 (TD-), R173.2: now also U1.83 (TXON)
- net at J11.3 (RD+), R172.2: now also U1.80 (RXIP)
- net at J11.6 (RD-), R171.2: now also U1.81 (RXIN)
- net at R161.2: now also U1.60 (VBUS_DTC/GPIO3)
- net at C102.1, R164.2: now also U1.96 (DAC_REFP)
- net at U24.2 (V_{OUT}): now also U1.87 (ADC1/CAM_XCLK/GPIO6)
- net at R168.1: now also U1.75 (HRREF)
- net at L14.2: now also U1.74 (AGND)
- net at R162.2: now also U1.85 (RTC_XI/RTC_CLKIN)
- net at J10.1 (DAT2): now also U1.6 (SD_DATA2/GPIO22)
- net at J10.2 (DAT3/CD): now also U1.5 (SD_DATA3/GPIO21)
- net at J10.3 (CMD): now also U1.4 (SD_CMD/GPIO20)
- net at J10.5 (CLK): now also U1.3 (SD_CLK/GPIO19)
- net at J10.7 (DAT0): now also U1.8 (SD_DATA0/GPIO24)
- net at J10.8 (DAT1): now also U1.7 (SD_DATA1/GPIO23)
- net at R169.1: now also U1.71 (DRREF)
- net at R158.1: now also U1.35 (STESTRESTN)
- net at R165.2: now also U1.57 (VBUS__DISCHG/_GPIO0)
- net at R163.2: now also U1.84 (RTC_XIO)
- net at L13.2: now also U1.94 (AGND)
- new net: CN1. (9), U1.20 (SPIS0_CLK/GPIO36)
- new net: CN1. (9), U1.21 (SPIS0_SS/GPIO37)
- new net: CN1. (9), U1.22 (SPIS0_MOSI/GPIO38)
- new net: CN1. (9), U1.23 (SPIS0_MISO/GPIO39)
- new net: CN1. (9), U1.36 (DEBUG)

Commit message: 05/06/26
Parts:
- renumbered C89 to C58, C90 to C59, C91 to C60, C92 to C61, C93 to C62, C94 to C63, C95 to C64, C96 to C65, C97 to C66, C98 to C67, C99 to C68, C100 to C69, C101 to C70, C102 to C71, C103 to C72, C104 to C73, C105 to C74, C106 to C75, C107 to C76, C108 to C77, C109 to C78, C110 to C79, C111 to C80, C112 to C81, C113 to C82, C114 to C83, C115 to C84, C116 to C85, C117 to C86, C118 to C87, D32 to D22, J10 to J8, J11 to J9, L14 to L10, L13 to L9, R157 to R100, R158 to R101, R159 to R102, R160 to R103, R161 to R104, R162 to R105, R163 to R106, R164 to R107, R165 to R108, R166 to R109, R167 to R110, R168 to R111, R169 to R112, R170 to R113, R171 to R114, R172 to R115, R173 to R116, R174 to R117, R156 to R99, U22 to U20, U1 to U21, U24 to U22

Commit message: 08-06-26
Parts:
- J8: footprint (none) -> Connector_Card:microSD_HC_Hirose_DM3AT-SF-PEJM5
- U21: footprint footprints:LQFP_100_14X14X1P4_BRI -> Package_DFN_QFN:ArtInChip_QFN-100-1EP_12x12mm_P0.4mm_EP7.4x7.4mm_ThermalVias
Changed lines of the file:
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@@
 			)
 		)
-		(property "Footprint" "footprints:LQFP_100_14X14X1P4_BRI"
+		(property "Footprint" "Package_DFN_QFN:ArtInChip_QFN-100-1EP_12x12mm_P0.4mm_EP7.4x7.4mm_ThermalVias"
 			(at 106.68 22.86 0)
 			(effects
@@
 			)
 		)
-		(property "Footprint" ""
+		(property "Footprint" "Connector_Card:microSD_HC_Hirose_DM3AT-SF-PEJM5"
 			(at -17.78 19.05 0)
 			(effects
